File: PTN-PumpControlBoard.kicad_pcb (KiCad board)
At the start: 2 copper layers, 94.4 x 64.2 mm, 58 parts, among them J1 CAN_OUT, J2 CAN_IN, J3 PPTC032LFBN-RC, J4 PPTC032LFBN-RC, J5 PPTC032LFBN-RC, U1 PeripheralSOM, U2 EMC2305-1-AP-TR, U3 TLV6001DCK, U4 TLV6001DCK, U5 TLV6001DCK, U6 TLV6001DCK

Commit message: making in prettyyy (kinda)
Parts:
- moved H4 0.57 mm to (191.0, 120.8)
- moved H1 0.57 mm to (103.4, 63.4)
- moved H3 0.57 mm to (103.4, 120.8)
- moved H2 0.45 mm to (191.0, 63.4)
Routing:
- net /FAN2_TACH: track 65.5 -> 70.1 mm
Other:
- outline, holes or cut-outs redrawn
- board text added: "- +"
- board text added: "- F +"
- board text added: "- F P +"
- board text added: "- P T +"
- board text added: "L H - +"
Changed lines of the file:
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@@
 	(footprint "MountingHole:MountingHole_3.2mm_M3"
 		(layer "F.Cu")
-		(at 103.8 120.4)
+		(at 103.4 120.8)
 		(descr "Mounting Hole 3.2mm, no annular, M3")
 		(tags "mounting hole 3.2mm no annular m3")
@@
 		(at 114.47 83.26 -90)
 		(property "Reference" "J3"
-			(at -1.016 -3.937 90)
+			(at -4.86 0.07 180)
 			(layer "F.SilkS")
 			(effects
@@
 	(footprint "MountingHole:MountingHole_3.2mm_M3"
 		(layer "F.Cu")
-		(at 190.6 120.4)
+		(at 191 120.8)
 		(descr "Mounting Hole 3.2mm, no annular, M3")
 		(tags "mounting hole 3.2mm no annular m3")
@@
 	(footprint "MountingHole:MountingHole_3.2mm_M3"
 		(layer "F.Cu")
-		(at 190.6 63.6)
+		(at 191 63.4)
 		(descr "Mounting Hole 3.2mm, no annular, M3")
 		(tags "mounting hole 3.2mm no annular m3")
@@
 	(footprint "MountingHole:MountingHole_3.2mm_M3"
 		(layer "F.Cu")
-		(at 103.8 63.8)
+		(at 103.4 63.4)
 		(descr "Mounting Hole 3.2mm, no annular, M3")
 		(tags "mounting hole 3.2mm no annular m3")
@@
 		(embedded_fonts no)
 	)
-	(gr_rect
-		(start 100 60)
-		(end 194.4 124.2)
+	(gr_arc
+		(start 191.2 60)
+		(mid 193.462742 60.937258)
+		(end 194.4 63.2)
 		(stroke
 			(width 0.05)
 			(type default)
 		)
-		(fill no)
 		(layer "Edge.Cuts")
 	)
+	(gr_line
+		(start 103.2 60)
+		(end 191.2 60)
+		(stroke
+			(width 0.05)
+			(type default)
+		)
+		(layer "Edge.Cuts")
+	)
+	(gr_line
+		(start 100 121)
+		(end 100 63.2)
+		(stroke
+			(width 0.05)
+			(type default)
+		)
+		(layer "Edge.Cuts")
+	)
+	(gr_arc
+		(start 103.2 124.2)
+		(mid 100.937258 123.262742)
+		(end 100 121)
+		(stroke
+			(width 0.05)
+			(type default)
+		)
+		(layer "Edge.Cuts")
+	)
+	(gr_line
+		(start 194.4 63.2)
+		(end 194.4 121)
+		(stroke
+			(width 0.05)
+			(type default)
+		)
+		(layer "Edge.Cuts")
+	)
+	(gr_arc
+		(start 100 63.2)
+		(mid 100.937258 60.937258)
+		(end 103.2 60)
+		(stroke
+			(width 0.05)
+			(type default)
+		)
+		(layer "Edge.Cuts")
+	)
+	(gr_line
+		(start 191.2 124.2)
+		(end 103.2 124.2)
+		(stroke
+			(width 0.05)
+			(type default)
+		)
+		(layer "Edge.Cuts")
+	)
+	(gr_arc
+		(start 194.4 121)
+		(mid 193.462742 123.262742)
+		(end 191.2 124.2)
+		(stroke
+			(width 0.05)
+			(type default)
+		)
+		(layer "Edge.Cuts")
+	)
+	(gr_text "-  +"
+		(at 149.2 122.6 0)
+		(layer "F.SilkS")
+		(effects
+			(font
+				(size 1 1)
+				(thickness 0.1)
+			)
+			(justify left bottom)
+		)
+	)
+	(gr_text "-  F  +"
+		(at 101 103.6 270)
+		(layer "F.SilkS")
+		(effects
+			(font
+				(size 1 1)
+				(thickness 0.1)
+			)
+			(justify left bottom)
+		)
+	)
+	(gr_text "L  H  -  +"
+		(at 115 122.8 0)
+		(layer "F.SilkS")
+		(effects
+			(font
+				(size 1 1)
+				(thickness 0.1)
+			)
+			(justify left bottom)
+		)
+	)
+	(gr_text "-  P  T  +"
+		(at 192 94.4 90)
+		(layer "F.SilkS")
+		(effects
+			(font
+				(size 1 1)
+				(thickness 0.1)
+			)
+			(justify left bottom)
+		)
+	)
+	(gr_text "-  +"
+		(at 191.4 104.2 90)
+		(layer "F.SilkS")
+		(effects
+			(font
+				(size 1 1)
+				(thickness 0.1)
+			)
+			(justify left bottom)
+		)
+	)
+	(gr_text "-  +"
+		(at 191.4 115.2 90)
+		(layer "F.SilkS")
+		(effects
+			(font
+				(size 1 1)
+				(thickness 0.1)
+			)
+			(justify left bottom)
+		)
+	)
+	(gr_text "-  F  P  +"
+		(at 100.8 75.6 270)
+		(layer "F.SilkS")
+		(effects
+			(font
+				(size 1 1)
+				(thickness 0.1)
+			)
+			(justify left bottom)
+		)
+	)
+	(gr_text "L  H  -  +"
+		(at 130.6 122.8 0)
+		(layer "F.SilkS")
+		(effects
+			(font
+				(size 1 1)
+				(thickness 0.1)
+			)
+			(justify left bottom)
+		)
+	)
+	(gr_text "-  P  T  +"
+		(at 191.8 79.2 90)
+		(layer "F.SilkS")
+		(effects
+			(font
+				(size 1 1)
+				(thickness 0.1)
+			)
+			(justify left bottom)
+		)
+	)
 	(segment
 		(start 152.425 84.825)
@@
 	)
 	(segment
-		(start 175.501 95.101)
-		(end 188.56426 95.101)
+		(start 191.4 90.2)
+		(end 189.5 88.3)
 		(width 0.2)
 		(layer "B.Cu")
@@
 	)
 	(segment
-		(start 167.74 90.88)
-		(end 171.96 95.1)
+		(start 176.2 95.8)
+		(end 172.66 95.8)
 		(width 0.2)
 		(layer "B.Cu")
@@
 	)
 	(segment
-		(start 172.6 92.2)
-		(end 175.5 95.1)
+		(start 189.5 88.3)
+		(end 188.4875 88.3)
 		(width 0.2)
 		(layer "B.Cu")
@@
 	)
 	(segment
-		(start 175 76.974202)
-		(end 186.325798 88.3)
+		(start 175.5 95.1)
+		(end 176.2 95.8)
 		(width 0.2)
 		(layer "B.Cu")
@@
 	)
 	(segment
-		(start 171.96 95.1)
+		(start 172.6 92.2)
 		(end 175.5 95.1)
 		(width 0.2)
@@
 	)
 	(segment
-		(start 189.8885 93.77676)
-		(end 189.8885 89.701)
+		(start 175 76.974202)
+		(end 186.325798 88.3)
 		(width 0.2)
 		(layer "B.Cu")
@@
 	)
 	(segment
-		(start 188.56426 95.101)
-		(end 189.8885 93.77676)
+		(start 176.2 95.8)
+		(end 190 95.8)
 		(width 0.2)
 		(layer "B.Cu")
@@
 	)
 	(segment
-		(start 189.8885 89.701)
-		(end 188.4875 88.3)
+		(start 190 95.8)
+		(end 191.4 94.4)
 		(width 0.2)
 		(layer "B.Cu")
@@
 	)
 	(segment
-		(start 175.5 95.1)
-		(end 175.501 95.101)
+		(start 167.74 90.88)
+		(end 172.66 95.8)
+		(width 0.2)
+		(layer "B.Cu")
+		(net 10)
+	)
+	(segment
+		(start 191.4 94.4)
+		(end 191.4 90.2)
 		(width 0.2)
 		(layer "B.Cu")
@@
 		(min_thickness 0.25)
 		(filled_areas_thickness no)
-		(fill yes
+		(fill
 			(thermal_gap 0.5)
 			(thermal_bridge_width 0.5)
@@
 		(min_thickness 0.25)
 		(filled_areas_thickness no)
-		(fill yes
+		(fill
 			(thermal_gap 0.5)
 			(thermal_bridge_width 0.5)
@@
 		(min_thickness 0.25)
 		(filled_areas_thickness no)
-		(fill yes
+		(fill
 			(thermal_gap 0.5)
 			(thermal_bridge_width 0.5)
@@
 		(min_thickness 0.25)
 		(filled_areas_thickness no)
-		(fill yes
+		(fill
 			(thermal_gap 0.5)
 			(thermal_bridge_width 0.5)
@@
 		(min_thickness 0.25)
 		(filled_areas_thickness no)
-		(fill yes
+		(fill
 			(thermal_gap 0.5)
 			(thermal_bridge_width 0.5)
@@
 		(min_thickness 0.25)
 		(filled_areas_thickness no)
-		(fill yes
+		(fill
 			(thermal_gap 0.5)
 			(thermal_bridge_width 0.5)
