File: PTN-PumpControlBoard.kicad_pcb (KiCad board)
At the start: 2 copper layers, 94.4 x 64.2 mm, 58 parts, among them J1 CAN_OUT, J2 CAN_IN, J3 PPTC032LFBN-RC, J4 PPTC032LFBN-RC, J5 PPTC032LFBN-RC, U1 PeripheralSOM, U2 EMC2305-1-AP-TR, U3 TLV6001DCK, U4 TLV6001DCK, U5 TLV6001DCK, U6 TLV6001DCK

Commit message: added +24V and GND flat test points
Parts:
- added +24V1: Pad_TP, UTSVT_Special:TestPoint_HEX_3mmID, F.Cu at (177.2, 68.0)
- added GND3: Pad_TP, UTSVT_Special:TestPoint_HEX_3mmID, F.Cu at (172.4, 68.0)
Routing:
- net GND: vias 8 -> 9
Changed lines of the file:
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@@
 		)
 	)
+	(footprint "UTSVT_Special:TestPoint_HEX_3mmID"
+		(layer "F.Cu")
+		(at 177.2 68 90)
+		(property "Reference" "+24V1"
+			(at 2.2 0 0)
+			(unlocked yes)
+			(layer "F.SilkS")
+			(effects
+				(font
+					(size 1 1)
+					(thickness 0.15)
+				)
+			)
+		)
+		(property "Value" "Pad_TP"
+			(at 0 1 90)
+			(unlocked yes)
+			(layer "F.Fab")
+			(effects
+				(font
+					(size 1 1)
+					(thickness 0.15)
+				)
+			)
+		)
+		(property "Datasheet" ""
+			(at 0 0 90)
+			(layer "F.Fab")
+			(hide yes)
+			(effects
+				(font
+					(size 1.27 1.27)
+					(thickness 0.15)
+				)
+			)
+		)
+		(property "Description" "test point"
+			(at 0 0 90)
+			(layer "F.Fab")
+			(hide yes)
+			(effects
+				(font
+					(size 1.27 1.27)
+					(thickness 0.15)
+				)
+			)
+		)
+		(property ki_fp_filters "Pin* Test*")
+		(sheetname "/")
+		(sheetfile "PTN-PumpControlBoard.kicad_sch")
+		(attr smd)
+		(fp_text user "${REFERENCE}"
+			(at 0 2.5 90)
+			(unlocked yes)
+			(layer "F.Fab")
+			(effects
+				(font
+					(size 1 1)
+					(thickness 0.15)
+				)
+			)
+		)
+		(pad "1" connect custom
+			(at 0 0 90)
+			(size 3 3)
+			(layers "F.Cu" "F.Mask")
+			(net 5 "+24V")
+			(pinfunction "1")
+			(pintype "passive")
+			(options
+				(clearance outline)
+				(anchor circle)
+			)
+			(primitives
+				(gr_poly
+					(pts
+						(xy 0 -1.732051) (xy 1.5 -0.866025) (xy 1.5 0.866025) (xy 0 1.732051) (xy -1.5 0.866025) (xy -1.5 -0.866025)
+					)
+					(width 0)
+					(fill yes)
+				)
+			)
+		)
+		(embedded_fonts no)
+	)
 	(footprint "TestPoint:TestPoint_Keystone_5010-5014_Multipurpose"
 		(layer "F.Cu")
@@
 		)
 	)
+	(footprint "UTSVT_Special:TestPoint_HEX_3mmID"
+		(layer "F.Cu")
+		(at 172.4 68 90)
+		(property "Reference" "GND3"
+			(at 2.2 0 0)
+			(unlocked yes)
+			(layer "F.SilkS")
+			(effects
+				(font
+					(size 1 1)
+					(thickness 0.15)
+				)
+			)
+		)
+		(property "Value" "Pad_TP"
+			(at 0 1 90)
+			(unlocked yes)
+			(layer "F.Fab")
+			(effects
+				(font
+					(size 1 1)
+					(thickness 0.15)
+				)
+			)
+		)
+		(property "Datasheet" ""
+			(at 0 0 90)
+			(layer "F.Fab")
+			(hide yes)
+			(effects
+				(font
+					(size 1.27 1.27)
+					(thickness 0.15)
+				)
+			)
+		)
+		(property "Description" "test point"
+			(at 0 0 90)
+			(layer "F.Fab")
+			(hide yes)
+			(effects
+				(font
+					(size 1.27 1.27)
+					(thickness 0.15)
+				)
+			)
+		)
+		(property ki_fp_filters "Pin* Test*")
+		(sheetname "/")
+		(sheetfile "PTN-PumpControlBoard.kicad_sch")
+		(attr smd)
+		(fp_text user "${REFERENCE}"
+			(at 0 2.5 90)
+			(unlocked yes)
+			(layer "F.Fab")
+			(effects
+				(font
+					(size 1 1)
+					(thickness 0.15)
+				)
+			)
+		)
+		(pad "1" connect custom
+			(at 0 0 90)
+			(size 3 3)
+			(layers "F.Cu" "F.Mask")
+			(net 2 "GND")
+			(pinfunction "1")
+			(pintype "passive")
+			(options
+				(clearance outline)
+				(anchor circle)
+			)
+			(primitives
+				(gr_poly
+					(pts
+						(xy 0 -1.732051) (xy 1.5 -0.866025) (xy 1.5 0.866025) (xy 0 1.732051) (xy -1.5 0.866025) (xy -1.5 -0.866025)
+					)
+					(width 0)
+					(fill yes)
+				)
+			)
+		)
+		(embedded_fonts no)
+	)
 	(footprint "Resistor_SMD:R_0805_2012Metric"
 		(layer "F.Cu")
@@
 	)
 	(via
+		(at 172.4 68)
+		(size 0.9)
+		(drill 0.5)
+		(layers "F.Cu" "B.Cu")
+		(net 2)
+	)
+	(via
 		(at 172.4 85.2)
 		(size 0.9)
@@
 		(min_thickness 0.25)
 		(filled_areas_thickness no)
-		(fill
+		(fill yes
 			(thermal_gap 0.5)
 			(thermal_bridge_width 0.5)
@@
 		(min_thickness 0.25)
 		(filled_areas_thickness no)
-		(fill
+		(fill yes
 			(thermal_gap 0.5)
 			(thermal_bridge_width 0.5)
@@
 		(min_thickness 0.25)
 		(filled_areas_thickness no)
-		(fill
+		(fill yes
 			(thermal_gap 0.5)
 			(thermal_bridge_width 0.5)
@@
 		(min_thickness 0.25)
 		(filled_areas_thickness no)
-		(fill
+		(fill yes
 			(thermal_gap 0.5)
 			(thermal_bridge_width 0.5)
@@
 		(min_thickness 0.25)
 		(filled_areas_thickness no)
-		(fill
+		(fill yes
 			(thermal_gap 0.5)
 			(thermal_bridge_width 0.5)
@@
 		(min_thickness 0.25)
 		(filled_areas_thickness no)
-		(fill
+		(fill yes
 			(thermal_gap 0.5)
 			(thermal_bridge_width 0.5)

Commit message: Fixed fan schematic based on review feedback
Parts:
- removed FL_OUT1, FL_TP1, F_PWM1, F_TACH1, F_TACH2, GND1, GND2, P_FG1, P_PWM1: Scope_TP, TestPoint:TestPoint_Keystone_5010-5014_Multipurpose
- removed F_PWM2: Scope_T1, TestPoint:TestPoint_Keystone_5010-5014_Multipurpose
- removed J3, J5: PPTC032LFBN-RC, Headers:SULLINS_PPTC032LFBN-RC
- removed R1, R2, R3: 10k, Resistor_SMD:R_0805_2012Metric
- removed R4: 15k, Resistor_SMD:R_0805_2012Metric
- removed TH1: Thermistor_PTC, Resistor_SMD:R_0603_1608Metric
- added C3: 1uF, Capacitor_SMD:C_0805_2012Metric, F.Cu at (222.9, 80.7)
- added C4: 1uF, Capacitor_SMD:C_0805_2012Metric, F.Cu at (222.9, 83.7)
- added J12: SFH11-PBPC-D05-ST-BK, Headers:CONN_SFH11-xxxC-D05-ST-XX_SUL, F.Cu at (227.9, 111.5)
- added R18: 10k, Resistor_SMD:R_0805_2012Metric, F.Cu at (171.7, 83.0)
- added R19: 10k, Resistor_SMD:R_0805_2012Metric, F.Cu at (216.5, 83.7)
- added R20: 10k, Resistor_SMD:R_0805_2012Metric, F.Cu at (216.5, 86.6)
- added R21: 10k, Resistor_SMD:R_0805_2012Metric, F.Cu at (216.5, 89.5)
- added R22: 10k, Resistor_SMD:R_0805_2012Metric, F.Cu at (216.5, 92.5)
- added R23: 33k, Resistor_SMD:R_0805_2012Metric, F.Cu at (216.5, 95.5)
- added R24: 33k, Resistor_SMD:R_0805_2012Metric, F.Cu at (216.5, 98.4)
- D1: value D_Zener -> VSSAF522-M3/H; footprint Diode_SMD:D_SOD-323F -> UTSVT_Passive:DO-221AC
- R5, R6: value 1k -> 5k
- moved U2 9.97 mm to (175.6, 79.6)
- moved C1 3.10 mm to (174.8, 84.6)
- moved C2 3.10 mm to (177.0, 84.6)
Connections:
- D1 pad 1: Net-(D1-K) -> +24V
- FLOW1 pad 2: /FlowrateSensor/FLOW_OUT -> GND
- FLOW1 pad 3: GND -> /FlowrateSensor/FLOW_OUT
- J4 pad 3: /~{SMBALERT} -> unconnected-(J4-Pad3)
- U2 pad 1: /FAN_SCL -> /FAN_SDA
- U2 pad 11: Net-(U2-CLK) -> /Fans/CLK
- U2 pad 2: /FAN_SDA -> /FAN_SCL
- U2 pad 4: unconnected-(U2-ADDR_SEL-Pad4) -> /Fans/ADDR_SEL
- U2 pad 5: /FAN2_PWM -> /FAN1_PWM
- U2 pad 7: /FAN1_PWM -> /FAN2_PWM
- U3 pad 2: AGND -> Net-(U3-V-)
- U3 pad 5: VDDA -> Net-(U3-V+)
Routing:
- net /FAN2_PWM: track 56.2 -> 32.0 mm, vias 1 -> 0
- net /FAN2_TACH: track 70.1 -> 46.8 mm, vias 1 -> 0
- net /FAN1_PWM: track 41.3 -> 20.6 mm
- net /FAN1_TACH: track 45.0 -> 26.9 mm, vias 2 -> 1
- net Net-(U3-V-): track 0.00 -> 4.37 mm, vias 0 -> 1
- net AGND: track 10.6 -> 6.25 mm, vias 4 -> 3
- net VDDA: track 12.4 -> 10.0 mm
- net Net-(U3-V+): track 0.00 -> 2.39 mm
- net Net-(U2-CLK): track 2.37 -> 0.00 mm
- net /Fans/CLK: track 0.00 -> 2.37 mm
- net +24V: track 4.46 -> 6.42 mm, vias 0 -> 1
- net Net-(D1-K): track 1.59 -> 0.00 mm
- net GND: track 16.7 -> 16.4 mm, vias 9 -> 8
- net (no net): track 0.00 -> 0.21 mm, vias 0 -> 1

Commit message: set up layout
Parts:
- removed GND3: Pad_TP, UTSVT_Special:TestPoint_HEX_3mmID
- removed J12: SFH11-PBPC-D05-ST-BK, Headers:CONN_SFH11-xxxC-D05-ST-XX_SUL
- removed U3, U4, U5, U6: TLV6001DCK, Package_TO_SOT_SMD:SOT-353_SC-70-5
- added C10: 15uF, Capacitor_SMD:C_0805_2012Metric, F.Cu at (201.2, 105.4)
- added C11: .1uF, Capacitor_SMD:C_0805_2012Metric, F.Cu at (201.2, 108.4)
- added C12: .1uF, Capacitor_SMD:C_0805_2012Metric, F.Cu at (201.2, 111.4)
- added C13: 1uF, Capacitor_SMD:C_0805_2012Metric, F.Cu at (103.8, 90.6)
- added C14: 15uF, Capacitor_SMD:C_0805_2012Metric, F.Cu at (103.8, 93.6)
- added C15: .1uF, Capacitor_SMD:C_0805_2012Metric, F.Cu at (103.8, 96.6)
- added C16: .1uF, Capacitor_SMD:C_0805_2012Metric, F.Cu at (103.8, 99.6)
- added C5: 1uF, Capacitor_SMD:C_0805_2012Metric, F.Cu at (196.9, 106.8)
- added C6: 15uF, Capacitor_SMD:C_0805_2012Metric, F.Cu at (196.9, 109.8)
- added C7: .1uF, Capacitor_SMD:C_0805_2012Metric, F.Cu at (196.8, 112.2)
- added C8: .1uF, Capacitor_SMD:C_0805_2012Metric, F.Cu at (201.2, 99.4)
- added C9: 1uF, Capacitor_SMD:C_0805_2012Metric, F.Cu at (201.2, 102.4)
- added D2: TVS, Diode_SMD:D_0603_1608Metric, F.Cu at (147.0, 82.8)
- added D3: TVS, Diode_SMD:D_0603_1608Metric, F.Cu at (147.0, 85.4)
- added D4: TVS, Diode_SMD:D_0603_1608Metric, F.Cu at (147.0, 88.0)
- added D5: TVS, Diode_SMD:D_0603_1608Metric, F.Cu at (147.0, 90.6)
- added D6: TVS, Diode_SMD:D_0603_1608Metric, F.Cu at (147.0, 93.2)
- added D7: VSSAF522-M3/H, UTSVT_Passive:MMDL101T1G, F.Cu at (180.3, 73.0)
- added D8: VSSAF522-M3/H, UTSVT_Passive:MMDL101T1G, F.Cu at (180.3, 75.8)
- added GND1: Pad_TP, UTSVT_Special:TestPoint_HEX_3mmID, F.Cu at (116.0, 64.0)
- added IC1: TLV9002QDRQ1, OpAmp:SOIC127P600X175-8N, F.Cu at (178.8, 96.6)
- added IC2: TLV9002QDRQ1, OpAmp:SOIC127P600X175-8N, F.Cu at (178.8, 103.2)
- added IC3: TLV9002QDRQ1, OpAmp:SOIC127P600X175-8N, F.Cu at (111.5, 112.3)
- added J3: SFH11-PBPC-D05-ST-BK, UTSVT_Connectors:CONN_SFH11-xxxC-D05-ST-XX_SUL, F.Cu at (162.0, 107.2)
- added PS1: TSR_1-24120SM, TSR_1-24120SM:TSR124120SM, F.Cu at (115.8, 94.8)
- added Q1: BUK7M27-80EX, Package_TO_SOT_SMD:LFPAK33, F.Cu at (167.4, 68.2)
- added Q2: BUK7M27-80EX, Package_TO_SOT_SMD:LFPAK33, F.Cu at (167.3, 73.6)
- added Q3: BUK7M27-80EX, Package_TO_SOT_SMD:LFPAK33, F.Cu at (113.3, 106.2)
- added R1: 5k, Resistor_SMD:R_0603_1608Metric, F.Cu at (172.0, 66.9)
- added R16: 15k, Resistor_SMD:R_0603_1608Metric, F.Cu at (184.2, 118.8)
- added R17: 0, Resistor_SMD:R_0603_1608Metric, F.Cu at (184.2, 121.3)
- added R2: 5k, Resistor_SMD:R_0603_1608Metric, F.Cu at (172.0, 69.4)
- added R25: 0, Resistor_SMD:R_0603_1608Metric, F.Cu at (97.8, 101.7)
- added R26: 10k, Resistor_SMD:R_0603_1608Metric, F.Cu at (97.8, 104.2)
- added R27: 15k, Resistor_SMD:R_0603_1608Metric, F.Cu at (97.8, 106.7)
- added R28: 0, Resistor_SMD:R_0603_1608Metric, F.Cu at (97.8, 109.2)
- added R29: 1k, Resistor_SMD:R_0603_1608Metric, F.Cu at (97.8, 111.7)
- added R3: 10k, Resistor_SMD:R_0603_1608Metric, F.Cu at (172.0, 71.9)
- added R30: 0, Resistor_SMD:R_0603_1608Metric, F.Cu at (97.8, 114.2)
- added R31: 10k, Resistor_SMD:R_0603_1608Metric, F.Cu at (108.4, 75.2)
- added R4: 33k, Resistor_SMD:R_0603_1608Metric, F.Cu at (172.0, 74.4)
- added T_TP4: Pad_TP, UTSVT_Special:TestPoint_HEX_3mmID, F.Cu at (105.0, 116.0)
- C4: value 1uF -> 15uF
- D1: value VSSAF522-M3/H -> TVS; footprint UTSVT_Passive:DO-221AC -> Diode_SMD:D_0603_1608Metric
- FAN1, FAN2: value Conn_01x04 -> Conn_01x03; footprint Connector_Molex:Molex_Nano-Fit_105309-xx04_1x04_P2.50mm_Vertical -> Connector_Molex:Molex_Nano-Fit_105309-xx03_1x03_P2.50mm_Vertical
- J1: value CAN_OUT -> CAN_IN; footprint Connector_Molex:Molex_Nano-Fit_105309-xx04_1x04_P2.50mm_Vertical -> UTSVT_Connectors:Molex_Nano-Fit_105309-xx04_1x04_P2.50mm_Vertical
- J2: value CAN_IN -> CAN_OUT; footprint Connector_Molex:Molex_Nano-Fit_105309-xx04_1x04_P2.50mm_Vertical -> UTSVT_Connectors:Molex_Nano-Fit_105309-xx04_1x04_P2.50mm_Vertical
- J4: value PPTC032LFBN-RC -> SFH11-PBPC-D05-ST-BK; footprint Headers:SULLINS_PPTC032LFBN-RC -> UTSVT_Connectors:CONN_SFH11-xxxC-D05-ST-XX_SUL
- R10: value 0 -> 10k; footprint Resistor_SMD:R_0805_2012Metric -> Resistor_SMD:R_0603_1608Metric
- R11: value 0 -> 15k; footprint Resistor_SMD:R_0805_2012Metric -> Resistor_SMD:R_0603_1608Metric
- R12, R20: footprint Resistor_SMD:R_0805_2012Metric -> Resistor_SMD:R_0603_1608Metric
- R13: value 100 -> 1k; footprint Resistor_SMD:R_0805_2012Metric -> Resistor_SMD:R_0603_1608Metric
- R14: value 1.4k -> 0; footprint Resistor_SMD:R_0805_2012Metric -> Resistor_SMD:R_0603_1608Metric
- R15, R8, R9: value 1k -> 10k; footprint Resistor_SMD:R_0805_2012Metric -> Resistor_SMD:R_0603_1608Metric
- R18: value 10k -> 1k; footprint Resistor_SMD:R_0805_2012Metric -> Resistor_SMD:R_0603_1608Metric
- R19, R22: value 10k -> 0; footprint Resistor_SMD:R_0805_2012Metric -> Resistor_SMD:R_0603_1608Metric
- R21: value 10k -> 15k; footprint Resistor_SMD:R_0805_2012Metric -> Resistor_SMD:R_0603_1608Metric
- R23: value 33k -> 1k; footprint Resistor_SMD:R_0805_2012Metric -> Resistor_SMD:R_0603_1608Metric
- R24: value 33k -> 0; footprint Resistor_SMD:R_0805_2012Metric -> Resistor_SMD:R_0603_1608Metric
- R5, R6: value 5k -> 10k; footprint Resistor_SMD:R_0805_2012Metric -> Resistor_SMD:R_0603_1608Metric
- R7: value 1k -> 33k; footprint Resistor_SMD:R_0805_2012Metric -> Resistor_SMD:R_0603_1608Metric
- moved R15 77.1 mm to (172.6, 118.6)
- moved +24V1 66.9 mm to (110.4, 64.4)
- moved R13 62.6 mm to (176.1, 116.8)
- moved R14 62.6 mm to (176.0, 113.2)
- moved J4 54.0 mm to (120.4, 72.8)
- moved D1 51.9 mm to (147.0, 79.5), turned to 0 degrees
- moved R9 51.7 mm to (179.4, 66.8)
- moved R19 44.1 mm to (180.0, 108.4)
- moved R20 44.1 mm to (180.0, 111.3)
- moved R21 44.1 mm to (180.0, 114.3)
- moved R22 44.1 mm to (180.0, 117.2)
- moved R23 44.1 mm to (180.0, 120.2)
- moved R24 44.1 mm to (180.0, 123.2)
- moved R18 38.8 mm to (173.2, 121.8)
- moved R8 35.6 mm to (175.6, 74.4)
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Connections:
- C3 pad 1: VDDA -> /TempSensors/IN1+
- C3 pad 2: Net-(U3-V+) -> AGND
- C4 pad 1: Net-(U3-V-) -> /TEMP1
- D1 pad 1: +24V -> GND
- D1 pad 2: GND -> /PUMP_PWM
- FAN1 pad 3: /FAN1_PWM -> Net-(FAN1-Pin_3)
- FAN2 pad 3: /FAN2_PWM -> Net-(FAN2-Pin_3)
- FLOW1 pad 1: +24V -> +12V
- J1 pad 2: GNDPWR -> GND
- J2 pad 2: GNDPWR -> GND
- J4 pad 1: /TEMP3 -> /FLOW
- J4 pad 2: /TEMP2 -> /PUMP_FG
- J4 pad 3: unconnected-(J4-Pad3) -> /PUMP_PWM
- J4 pad 4: /TEMP1 -> unconnected-(J4-Pad4)
- R10 pad 1: /TEMP1 -> VDDA
- R10 pad 2: Net-(U3--) -> Net-(TEMP1-Pin_1)
- R11 pad 1: /TEMP2 -> Net-(TEMP1-Pin_1)
- R11 pad 2: Net-(U4--) -> /TempSensors/IN1+
- R12 pad 1: /TEMP3 -> /TempSensors/OUT1
- R12 pad 2: Net-(U5--) -> /TempSensors/IN1-
- R13 pad 1: Net-(U6--) -> /TempSensors/OUT1
- R13 pad 2: GND -> /TEMP1
- R14 pad 1: /FLOW -> /TempSensors/IN1-
- R14 pad 2: Net-(U6--) -> AGND
- R15 pad 1: +3.3V -> VDDA
- R15 pad 2: /PUMP_FG -> Net-(TEMP3-Pin_1)
- R18 pad 1: /FAN_SDA -> /TempSensors/OUT2
- R18 pad 2: +3.3V -> /TEMP2
- R19 pad 1: /FAN_SCL -> /TempSensors/IN2-
- R19 pad 2: +3.3V -> AGND
- R20 pad 1: /FAN1_PWM -> VDDA
- R20 pad 2: +3.3V -> Net-(TEMP2-Pin_1)
- R21 pad 1: /~{SMBALERT} -> Net-(TEMP2-Pin_1)
- R21 pad 2: +3.3V -> /TempSensors/IN3+
- R22 pad 1: /FAN2_PWM -> /TempSensors/OUT3
- R22 pad 2: +3.3V -> /TempSensors/IN3-
- R23 pad 1: /Fans/ADDR_SEL -> /TempSensors/OUT3
- R23 pad 2: +3.3V -> /TEMP3
- R24 pad 1: /Fans/CLK -> /TempSensors/IN3-
- R24 pad 2: +3.3V -> AGND
- R5 pad 1: +3.3V -> /FAN_SCL
- R5 pad 2: /FAN1_TACH -> +3.3V
- R6 pad 1: +3.3V -> /~{SMBALERT}
- R6 pad 2: /FAN2_TACH -> +3.3V
- R7 pad 1: VDDA -> /Fans/CLK
- R7 pad 2: Net-(TEMP1-Pin_1) -> +3.3V
- R8 pad 1: VDDA -> /FAN1_PWM
- R8 pad 2: Net-(TEMP2-Pin_1) -> +3.3V
- R9 pad 1: VDDA -> /FAN2_PWM
- R9 pad 2: Net-(TEMP3-Pin_1) -> +3.3V
- T_TP1 pad 1: /TEMP1 -> /TempSensors/OUT1
- T_TP2 pad 1: /TEMP2 -> /TempSensors/OUT3
- T_TP3 pad 1: /TEMP3 -> /TempSensors/OUT2
Routing:
- net /PUMP_PWM: track 74.0 -> 0.00 mm, vias 1 -> 0
- net /PUMP_FG: track 72.5 -> 0.00 mm, vias 1 -> 0
- net /FLOW: track 70.4 -> 0.00 mm, vias 2 -> 0
- net /CAN_L: track 61.1 -> 0.00 mm, vias 1 -> 0
- net /CAN_H: track 60.2 -> 0.00 mm, vias 1 -> 0
- net /TEMP1: track 59.1 -> 0.00 mm, vias 2 -> 0
- net /TEMP2: track 51.3 -> 0.00 mm
- net /FAN2_TACH: track 46.8 -> 0.00 mm
- net /~{SMBALERT}: track 41.9 -> 0.00 mm, vias 2 -> 0
- net /TEMP3: track 33.3 -> 0.00 mm
- net /FAN2_PWM: track 32.0 -> 0.00 mm
- net /FAN1_TACH: track 26.9 -> 0.00 mm, vias 1 -> 0
- net Net-(TEMP2-Pin_1): track 26.7 -> 0.00 mm
- net /FAN1_PWM: track 20.6 -> 0.00 mm, vias 2 -> 0
- net /FlowrateSensor/FLOW_OUT: track 20.2 -> 0.00 mm
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- removed copper zone on F.Cu, net +3.3V
- removed copper zone on B.Cu, net AGND
- removed copper zone on B.Cu, net GNDPWR
- removed copper zone on F.Cu, net VDDA

Commit message: review notes
Parts:
- C3, C4, C5, C6, C7, C8, IC1, R10, R11, R12, R13, R14, R15, R16, R17, R18, R19: moved to B.Cu
- moved C12 43.7 mm to (158.5, 120.9)
- moved J3 42.6 mm to (165.2, 64.7), turned to 0 degrees
- moved C11 41.0 mm to (162.1, 120.9), turned to 180 degrees
- moved C9 37.1 mm to (165.8, 113.7)
- moved C10 37.1 mm to (165.8, 116.7)
- moved R2 26.0 mm to (184.6, 92.2)
- moved T_OUT1 25.8 mm to (197.0, 99.6)
- moved T_TP1 25.6 mm to (196.8, 103.8)
- moved T_TP2 25.4 mm to (196.4, 115.2)
- moved T_OUT2 25.4 mm to (196.4, 111.2)
- moved C4 23.3 mm to (174.4, 96.6), turned to 180 degrees
- moved IC2 23.1 mm to (160.3, 117.0)
- moved C8 22.0 mm to (180.2, 105.8), turned to -90 degrees
- moved C5 20.9 mm to (180.8, 120.0)
- moved R9 20.0 mm to (182.0, 86.6), turned to -90 degrees
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Connections:
- C12 pad 1: Net-(C12-Pad1) -> /TempSensors/V2-
- C15 pad 1: Net-(C15-Pad1) -> /FlowrateSensor/V3-
- C8 pad 1: Net-(C8-Pad1) -> /TempSensors/V1-
- D7 pad 1: GND -> /Fans/NET1
- D8 pad 1: GND -> /Fans/NET2
- FAN1 pad 3: Net-(FAN1-Pin_3) -> /Fans/NET1
- FAN2 pad 3: Net-(FAN2-Pin_3) -> /Fans/NET2
- IC1 pad 4: AGND -> /TempSensors/V1-
- IC2 pad 4: AGND -> /TempSensors/V2-
- IC3 pad 4: GND -> /FlowrateSensor/V3-
- J3 pad 1: /FAN1_PWM -> /FAN1_TACH
- J3 pad 10: /~{SMBALERT} -> GND
- J3 pad 2: /FAN1_TACH -> /FAN2_TACH
- J3 pad 3: /FAN2_PWM -> /TEMP1
- J3 pad 4: /FAN2_TACH -> /TEMP2
- J3 pad 5: /TEMP1 -> /TEMP3
- J3 pad 6: /TEMP2 -> /FAN_SCL
- J3 pad 7: /TEMP3 -> /FAN_SDA
- J3 pad 8: /FAN_SCL -> /~{SMBALERT}
- J3 pad 9: /FAN_SDA -> GND
- J4 pad 10: unconnected-(J4-Pad10) -> GND
- J4 pad 3: /PUMP_PWM -> unconnected-(J4-Pad3)
- J4 pad 9: unconnected-(J4-Pad9) -> GND
- Q1 pad 5: Net-(FAN1-Pin_3) -> /Fans/NET1
- Q2 pad 5: Net-(FAN2-Pin_3) -> /Fans/NET2
- U2 pad 5: /FAN1_PWM -> /FAN2_PWM
- U2 pad 6: /FAN1_TACH -> /FAN2_TACH
- U2 pad 7: /FAN2_PWM -> /FAN1_PWM
- U2 pad 8: /FAN2_TACH -> /FAN1_TACH
Routing:
- net Net-(TEMP1-Pin_1): track 0.00 -> 12.0 mm
- net /TempSensors/OUT1: track 0.00 -> 7.19 mm
- net /TempSensors/IN1+: track 0.00 -> 5.72 mm
- net /PUMP_FG: track 0.00 -> 4.34 mm
- net /Fans/NET1: track 0.00 -> 3.65 mm
- net /Fans/NET2: track 0.00 -> 3.59 mm
- net /TempSensors/IN1-: track 0.20 -> 3.57 mm
- net /TempSensors/V1-: track 0.00 -> 2.07 mm
- net /TEMP1: track 0.00 -> 1.83 mm
Other:
- board text added: "F - +"
- board text removed: "- F +"
- board text removed: "- P T +"

Commit message: cube sux
Parts:
- removed IC3: TLV9002QDRQ1, OpAmp:SOIC127P600X175-8N
- removed PS1: TSR_1-24120SM, TSR_1-24120SM:TSR124120SM
- removed T_TP4: Pad_TP, UTSVT_Special:TestPoint_HEX_3mmID
- added +5V1: Pad_TP, UTSVT_Special:TestPoint_HEX_3mmID, F.Cu at (224.2, 100.7)
- added 5V_IN1: Conn_01x02, UTSVT_Connectors:Molex_Nano-Fit_105309-xx02_1x02_P2.50mm_Vertical, F.Cu at (53.6, 99.8)
- added C17: 0.1uF, Capacitor_SMD:C_0603_1608Metric_Pad1.08x0.95mm_HandSolder, F.Cu at (224.4, 91.3)
- added C18: 10uF, Capacitor_SMD:C_0805_2012Metric_Pad1.18x1.45mm_HandSolder, F.Cu at (227.5, 105.6)
- added C19: 10uF, Capacitor_SMD:C_0805_2012Metric_Pad1.18x1.45mm_HandSolder, F.Cu at (227.5, 108.6)
- added C20: 10uF, Capacitor_SMD:C_0805_2012Metric_Pad1.18x1.45mm_HandSolder, F.Cu at (227.5, 111.6)
- added C21: 10uF, Capacitor_SMD:C_0805_2012Metric_Pad1.18x1.45mm_HandSolder, F.Cu at (234.3, 101.6)
- added C22: 1uF, Capacitor_SMD:C_0603_1608Metric_Pad1.08x0.95mm_HandSolder, F.Cu at (234.1, 91.3)
- added C23: 100nF, Capacitor_SMD:C_0603_1608Metric_Pad1.08x0.95mm_HandSolder, F.Cu at (234.1, 93.8)
- added C24: 1uF, Capacitor_SMD:C_0603_1608Metric_Pad1.08x0.95mm_HandSolder, F.Cu at (234.1, 96.4)
- added C25: 10uF, Capacitor_SMD:C_0805_2012Metric_Pad1.18x1.45mm_HandSolder, F.Cu at (234.3, 104.6)
- added D10: VSSAF522-M3/H, UTSVT_Passive:MMDL101T1G, F.Cu at (252.9, 55.5)
- added D11: MBR230S1F, Diode_SMD:D_SOD-123F, F.Cu at (225.0, 96.8)
- added D12: TVS, Diode_SMD:D_SOD-323_HandSoldering, F.Cu at (244.8, 101.6)
- added D13: TVS, Diode_SMD:D_SOD-123F, F.Cu at (239.5, 101.8)
- added J5: SFH11-PBPC-D05-ST-BK, UTSVT_Connectors:CONN_SFH11-xxxC-D05-ST-XX_SUL, F.Cu at (213.9, 82.0)
- added L1: 100uH, Inductor_SMD:L_Coilcraft_MSS1246-XXX, F.Cu at (215.2, 97.2)
- added LOGO1: Dr. Hallock, UTSVT_Logos:Hallock_Image_Small, F.Cu at (218.1, 66.2)
- added LOGO2: LHRS, UTSVT_Logos:LHRs_LOGO, F.Cu at (237.0, 56.0)
- added Q5: PSMN8R5-40MSDX, Package_TO_SOT_SMD:LFPAK33, F.Cu at (252.8, 59.3)
- added R32: ROSC, Resistor_SMD:R_0603_1608Metric_Pad0.98x0.95mm_HandSolder, F.Cu at (224.4, 93.8)
- added R33: 10k, Resistor_SMD:R_0603_1608Metric, F.Cu at (248.1, 55.4)
- added R34: 100, Resistor_SMD:R_0603_1608Metric, F.Cu at (248.1, 57.9)
- added R35: 100k, Resistor_SMD:R_0603_1608Metric, F.Cu at (248.1, 60.4)
- added R36: 10k, Resistor_SMD:R_0603_1608Metric, F.Cu at (248.1, 62.9)
- added R37: 24m, Resistor_SMD:R_0603_1608Metric_Pad0.98x0.95mm_HandSolder, F.Cu at (234.1, 98.9)
- added R38: 10k, Resistor_SMD:R_0603_1608Metric_Pad0.98x0.95mm_HandSolder, F.Cu at (238.4, 91.3)
- added R39: 45.3k, Resistor_SMD:R_0603_1608Metric_Pad0.98x0.95mm_HandSolder, F.Cu at (238.4, 93.8)
- added R40: 590, Resistor_SMD:R_0603_1608Metric_Pad0.98x0.95mm_HandSolder, F.Cu at (238.4, 96.4)
- added R41: 2.1k, Resistor_SMD:R_0603_1608Metric_Pad0.98x0.95mm_HandSolder, F.Cu at (238.4, 98.9)
- added R42: 402k, Resistor_SMD:R_0603_1608Metric_Pad0.98x0.95mm_HandSolder, F.Cu at (242.8, 91.3)
- added R43: 10k, Resistor_SMD:R_0603_1608Metric_Pad0.98x0.95mm_HandSolder, F.Cu at (242.8, 93.8)
- added R44: 10k, Resistor_SMD:R_0603_1608Metric_Pad0.98x0.95mm_HandSolder, F.Cu at (242.8, 96.4)
- added R45: 100k, Resistor_SMD:R_0603_1608Metric_Pad0.98x0.95mm_HandSolder, F.Cu at (242.8, 98.9)
- added U6: TPS5405DR, UTSVT_Power:TPS5405DR, F.Cu at (220.8, 107.3)
- C13: value 1uF -> 10uF; footprint Capacitor_SMD:C_0805_2012Metric -> Capacitor_SMD:C_0805_2012Metric_Pad1.18x1.45mm_HandSolder
- C14: value 15uF -> 1uF; footprint Capacitor_SMD:C_0805_2012Metric -> Capacitor_SMD:C_0603_1608Metric_Pad1.08x0.95mm_HandSolder
- C15: value .1uF -> 10nF; footprint Capacitor_SMD:C_0805_2012Metric -> Capacitor_SMD:C_0603_1608Metric_Pad1.08x0.95mm_HandSolder
- C16: value .1uF -> 3.3nF; footprint Capacitor_SMD:C_0805_2012Metric -> Capacitor_SMD:C_0603_1608Metric_Pad1.08x0.95mm_HandSolder
- J1: value CAN_IN -> 53307-2471; footprint UTSVT_Connectors:Molex_Nano-Fit_105309-xx04_1x04_P2.50mm_Vertical -> UTSVT_Connectors:PeripheralSOM
- J2: value CAN_OUT -> CAN_IN
- J3: value SFH11-PBPC-D05-ST-BK -> CAN_OUT; footprint UTSVT_Connectors:CONN_SFH11-xxxC-D05-ST-XX_SUL -> UTSVT_Connectors:Molex_Nano-Fit_105309-xx04_1x04_P2.50mm_Vertical
- Q1, Q2, Q3: value BUK7M27-80EX -> PSMN8R5-40MSDX
- R10: value 10k -> 33k; moved to F.Cu
- R11: value 15k -> 33k; moved to F.Cu
- R12, R17, R22: value 0 -> 10k
- R13, R18, R23: value 1k -> 15k
- R15, R20: value 10k -> 1k
- R16, R21, R27: value 15k -> 0
- R2: value 5k -> 100k
- R25: value 0 -> 1k
- R26: value 10k -> 0
- R28: value 0 -> 100k
- R29: value 1k -> 10k
- R3: value 10k -> 5k
- R31: value 10k -> 16k; footprint Resistor_SMD:R_0603_1608Metric -> Resistor_SMD:R_0603_1608Metric_Pad0.98x0.95mm_HandSolder
- R4: value 33k -> 100k
- R7: value 33k -> 10k
- U1: value PeripheralSOM -> LM76202QPWPRQ1; footprint UTSVT_Special:PeripheralSOM -> UTSVT_Power:LM76202QPWPRQ1
- moved D8 89.7 mm to (103.3, 72.8), turned to -90 degrees
- moved D7 89.0 mm to (103.5, 87.9), turned to -90 degrees
- moved FAN1 83.8 mm to (106.7, 90.7), turned to 180 degrees
- moved FAN2 82.7 mm to (106.4, 75.5), turned to 180 degrees
- moved R1 77.2 mm to (110.5, 92.1), turned to 180 degrees
- moved Q2 72.3 mm to (111.4, 78.5), turned to 180 degrees
- moved Q1 72.3 mm to (111.4, 82.8), turned to 180 degrees
- moved R2 70.5 mm to (114.7, 82.7), turned to -90 degrees
- moved J3 69.8 mm to (122.7, 119.9), turned to -90 degrees
- moved R9 66.1 mm to (116.3, 79.3), turned to 90 degrees
- moved R8 65.0 mm to (116.3, 82.7), turned to -90 degrees
- moved R10 64.7 mm to (119.1, 76.7), turned to 90 degrees
- moved R4 63.1 mm to (114.7, 79.3), turned to 90 degrees
- moved R3 60.9 mm to (110.3, 69.1)
- moved R11 59.3 mm to (120.1, 85.3), turned to -90 degrees
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Connections:
- C13 pad 1: /FlowrateSensor/IN4+ -> +24V
- C14 pad 1: /FLOW -> Net-(U6-VIN)
- C15 pad 1: /FlowrateSensor/V3- -> Net-(U6-SS)
- C16 pad 1: +3.3V -> Net-(U6-COMP)
- C16 pad 2: GND -> Net-(C16-Pad2)
- FLOW1 pad 1: +12V -> +5V
- J1 pad 1: +24V -> GND
- J1 pad 2: GND -> +3.3V
- J1 pad 3: /CAN_H -> GND
- J1 pad 4: /CAN_L -> /FAN_SDA
- J2 pad 1: +24V -> +24V_IN
- J3 pad 1: /FAN1_TACH -> +24V
- J3 pad 2: /FAN2_TACH -> GND
- J3 pad 3: /TEMP1 -> /CAN_H
- J3 pad 4: /TEMP2 -> /CAN_L
- J4 pad 1: /FLOW -> /FAN1_TACH
- J4 pad 2: /PUMP_FG -> /FAN2_TACH
- J4 pad 3: unconnected-(J4-Pad3) -> /FAN1_PWM
- J4 pad 4: unconnected-(J4-Pad4) -> /FAN2_PWM
- J4 pad 6: unconnected-(J4-Pad6) -> /FAN_SCL
- J4 pad 7: unconnected-(J4-Pad7) -> /FAN_SDA
- J4 pad 8: unconnected-(J4-Pad8) -> /~{SMBALERT}
- Q3 pad 5: Net-(Q3-D) -> /FLOW
- R10 pad 1: VDDA -> /Fans/ADDR_SEL
- R10 pad 2: Net-(TEMP1-Pin_1) -> +3.3V
- R11 pad 1: Net-(TEMP1-Pin_1) -> /Fans/CLK
- R11 pad 2: /TempSensors/IN1+ -> +3.3V
- R12 pad 1: /TempSensors/OUT1 -> VDDA
- R12 pad 2: /TempSensors/IN1- -> Net-(TEMP1-Pin_1)
- R13 pad 1: /TempSensors/OUT1 -> Net-(TEMP1-Pin_1)
- R13 pad 2: /TEMP1 -> /TempSensors/IN1+
- R14 pad 1: /TempSensors/IN1- -> /TempSensors/OUT1
- R14 pad 2: AGND -> /TempSensors/IN1-
- R15 pad 1: VDDA -> /TempSensors/OUT1
- R15 pad 2: Net-(TEMP3-Pin_1) -> /TEMP1
- R16 pad 1: Net-(TEMP3-Pin_1) -> /TempSensors/IN1-
- R16 pad 2: /TempSensors/IN2+ -> AGND
- R17 pad 1: /TempSensors/OUT2 -> VDDA
- R17 pad 2: /TempSensors/IN2- -> Net-(TEMP3-Pin_1)
- R18 pad 1: /TempSensors/OUT2 -> Net-(TEMP3-Pin_1)
- R18 pad 2: /TEMP2 -> /TempSensors/IN2+
- R19 pad 1: /TempSensors/IN2- -> /TempSensors/OUT2
- R19 pad 2: AGND -> /TempSensors/IN2-
- R2 pad 1: +3.3V -> /FAN1_PWM
- R2 pad 2: /FAN2_TACH -> GND
- R20 pad 1: VDDA -> /TempSensors/OUT2
- R20 pad 2: Net-(TEMP2-Pin_1) -> /TEMP2
- R21 pad 1: Net-(TEMP2-Pin_1) -> /TempSensors/IN2-
- R21 pad 2: /TempSensors/IN3+ -> AGND
- R22 pad 1: /TempSensors/OUT3 -> VDDA
- R22 pad 2: /TempSensors/IN3- -> Net-(TEMP2-Pin_1)
- R23 pad 1: /TempSensors/OUT3 -> Net-(TEMP2-Pin_1)
- R23 pad 2: /TEMP3 -> /TempSensors/IN3+
- R24 pad 1: /TempSensors/IN3- -> /TempSensors/OUT3
- R24 pad 2: AGND -> /TempSensors/IN3-
- R25 pad 1: /FlowrateSensor/FLOW_OUT -> /TempSensors/OUT3
- R25 pad 2: Net-(Q3-G) -> /TEMP3
- R26 pad 1: Net-(Q3-D) -> /TempSensors/IN3-
- R26 pad 2: +3.3V -> AGND
- R27 pad 1: Net-(Q3-D) -> /FlowrateSensor/FLOW_OUT
- R27 pad 2: /FlowrateSensor/IN4+ -> Net-(Q3-G)
- R28 pad 1: /FlowrateSensor/OUT4 -> Net-(Q3-G)
- R28 pad 2: /FlowrateSensor/IN4- -> GND
- R29 pad 1: /FlowrateSensor/OUT4 -> /FLOW
- R29 pad 2: /FLOW -> +3.3V
- R3 pad 1: /FAN_SDA -> +3.3V
- R3 pad 2: +3.3V -> /FAN2_TACH
- R30 pad 1: /FlowrateSensor/IN4- -> +24V
- R30 pad 2: GND -> Net-(U6-VIN)
- R31 pad 1: +3.3V -> Net-(C16-Pad2)
- R31 pad 2: /PUMP_FG -> GND
- R4 pad 1: /Fans/ADDR_SEL -> /FAN2_PWM
- R4 pad 2: +3.3V -> GND
- R5 pad 1: /FAN_SCL -> /FAN_SDA
- R6 pad 1: /~{SMBALERT} -> /FAN_SCL
- R7 pad 1: /Fans/CLK -> /~{SMBALERT}
- U1 pad 1: /~{SMBALERT} -> +24V_IN
- U1 pad 10: VDDA -> /PowerProtection/IMON
- U1 pad 11: GND -> /PowerProtection/ILIM
- U1 pad 12: AGND -> Net-(U1-DVDT)
- U1 pad 13: /PUMP_PWM -> unconnected-(U1-NC_2-Pad13)
- U1 pad 14: unconnected-(U1-I2C1_SCL-Pad14) -> /FAULT
- U1 pad 15: unconnected-(U1-SPI1_MISO-Pad15) -> +24V
- U1 pad 16: unconnected-(U1-I2C1_SDA-Pad16) -> +24V
- U1 pad 17: unconnected-(U1-SPI1_MOSI-Pad17) -> /PowerProtection/RTN
- U1 pad 2: +3.3V -> +24V_IN
- U1 pad 3: /PUMP_FG -> /PowerProtection/UVLO
- U1 pad 4: GND -> unconnected-(U1-NC_1-Pad4)
- U1 pad 5: unconnected-(U1-SPI2_SCK-Pad5) -> /PowerProtection/OVP
- U1 pad 6: /FAN_SDA -> /PowerProtection/MODE
- U1 pad 7: unconnected-(U1-SPI2_NSS-Pad7) -> /PowerProtection/SHDN
- U1 pad 8: /FAN_SCL -> /PowerProtection/RTN
- U1 pad 9: +3.3V -> GND
Routing:
- net /FAN2_TACH: track 0.00 -> 23.7 mm
- net /FAN1_TACH: track 0.00 -> 20.5 mm
- net /Fans/NET2: track 3.59 -> 18.6 mm
- net /FAN2_PWM: track 0.00 -> 7.02 mm
- net /FAN1_PWM: track 0.00 -> 5.65 mm
- net /Fans/NET1: track 3.65 -> 9.10 mm
- net /FAN_SCL: track 0.00 -> 3.82 mm
- net /FAN_SDA: track 0.00 -> 2.15 mm
- net /Fans/ADDR_SEL: track 0.00 -> 1.74 mm
- net /Fans/CLK: track 0.00 -> 1.64 mm
- net /~{SMBALERT}: track 0.00 -> 1.60 mm
