File: PTN-PumpControlBoard.kicad_pcb (KiCad board)
At the start: 2 copper layers, 94.4 x 64.2 mm, 121 parts, among them IC1 TLV9002QDRQ1, IC2 TLV9002QDRQ1, J1 53307-2471, J2 CAN_IN, J3 CAN_OUT, J4 SFH11-PBPC-D05-ST-BK, J5 SFH11-PBPC-D05-ST-BK, Q1 PSMN8R5-40MSDX, Q2 PSMN8R5-40MSDX, Q3 PSMN8R5-40MSDX, Q5 PSMN8R5-40MSDX, U1 LM76202QPWPRQ1, U2 EMC2305-1-AP-TR, U6 TPS5405DR

Commit message: fan and temp subcircuits
Parts:
- removed T_OUT2, T_OUT3, T_TP2, T_TP3: Pad_TP, UTSVT_Special:TestPoint_HEX_3mmID
- C10, C11, C12, C9, IC2, R20, R21, R22, R23, R24, R25, R26: moved to B.Cu
- moved 5V_IN1 113.7 mm to (165.3, 120.8), turned to 0 degrees
- moved FLOW1 113.4 mm to (165.0, 108.0), turned to 0 degrees
- moved PUMP1 113.4 mm to (164.8, 92.5), turned to 0 degrees
- moved R31 109.7 mm to (160.8, 100.3), turned to 0 degrees
- moved J5 101.2 mm to (122.7, 125.8)
- moved T_OUT1 84.4 mm to (112.6, 97.8)
- moved T_TP1 84.2 mm to (112.6, 102.8)
- moved TEMP2 84.0 mm to (104.2, 108.8), turned to 180 degrees
- moved TEMP1 83.8 mm to (104.4, 99.0), turned to 180 degrees
- moved J4 78.4 mm to (122.9, 117.5), turned to 0 degrees
- moved R16 74.4 mm to (119.2, 85.4), turned to 180 degrees
- moved L1 71.9 mm to (147.8, 122.2), turned to 180 degrees
- moved J3 67.9 mm to (164.8, 66.7), turned to 0 degrees
- moved C6 66.2 mm to (116.9, 99.6)
- moved R15 65.0 mm to (116.6, 90.0)
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Connections:
- J1 pad 11: /TEMP2 -> /TEMP1
- J1 pad 9: /TEMP1 -> /TEMP2
- R17 pad 2: Net-(TEMP3-Pin_1) -> Net-(TEMP2-Pin_1)
- R18 pad 1: Net-(TEMP3-Pin_1) -> Net-(TEMP2-Pin_1)
- R22 pad 2: Net-(TEMP2-Pin_1) -> Net-(TEMP3-Pin_1)
- R23 pad 1: Net-(TEMP2-Pin_1) -> Net-(TEMP3-Pin_1)
Routing:
- net Net-(TEMP2-Pin_1): track 0.00 -> 24.0 mm, vias 0 -> 1
- net Net-(TEMP1-Pin_1): track 12.0 -> 35.4 mm
- net /TempSensors/OUT1: track 7.19 -> 23.0 mm, vias 0 -> 1
- net Net-(TEMP3-Pin_1): track 1.76 -> 9.05 mm
- net /TempSensors/IN2+: track 0.00 -> 6.07 mm
- net /TempSensors/OUT2: track 0.00 -> 5.37 mm
- net /Fans/NET1: track 9.10 -> 14.3 mm
- net /TempSensors/IN2-: track 0.00 -> 5.08 mm
- net /TempSensors/IN3+: track 0.00 -> 3.90 mm
- net /TempSensors/OUT3: track 0.00 -> 3.88 mm
- net /TempSensors/IN3-: track 0.00 -> 3.87 mm
- net /FAN1_TACH: track 20.5 -> 24.4 mm
- net /Fans/NET2: track 18.6 -> 15.2 mm
- net /TEMP3: track 0.00 -> 3.32 mm
- net /FAN2_TACH: track 23.7 -> 21.4 mm
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Other:
- board size 94.4 x 64.2 mm -> 88.6 x 72.2 mm

Commit message: flowrate subcircuit
Parts:
- C13, C14, C15, C16, C17, C18, C19, C20, D11, Q3, R27, R28, R29, R30, R31, R32, U6: moved to B.Cu
- moved U1 122.9 mm to (260.5, 95.6)
- moved Q5 102.9 mm to (155.4, 92.4)
- moved R35 97.1 mm to (158.6, 98.0)
- moved R34 96.9 mm to (158.6, 95.0)
- moved Q3 96.5 mm to (157.9, 113.3), turned to -90 degrees
- moved R33 94.6 mm to (160.6, 91.4)
- moved R36 94.5 mm to (157.4, 89.4)
- moved D10 93.1 mm to (169.2, 96.4), turned to 90 degrees
- moved C14 91.9 mm to (153.8, 127.9), turned to 180 degrees
- moved C13 91.1 mm to (151.0, 129.1), turned to 90 degrees
- moved R27 87.9 mm to (161.4, 114.4), turned to 180 degrees
- moved C18 86.3 mm to (142.2, 118.8), turned to 90 degrees
- moved +5V1 86.0 mm to (143.2, 129.4)
- moved R28 85.6 mm to (159.2, 109.4), turned to 90 degrees
- moved C15 85.0 mm to (148.4, 125.7), turned to 180 degrees
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Routing:
- net +5V: track 0.00 -> 45.7 mm, vias 0 -> 1
- net /TempSensors/OUT1: track 23.0 -> 10.5 mm
- net Net-(D11-K): track 0.00 -> 6.15 mm, vias 0 -> 2
- net Net-(Q3-G): track 0.00 -> 4.99 mm
- net /FLOW: track 0.00 -> 4.53 mm
- net /FlowrateSensor/ROSC: track 0.00 -> 4.36 mm
- net /PUMP_FG: track 4.34 -> 0.00 mm
- net Net-(U6-VIN): track 0.00 -> 3.99 mm
- net Net-(U6-BOOT): track 0.00 -> 3.58 mm
- net /FlowrateSensor/FLOW_OUT: track 0.00 -> 3.37 mm
- net Net-(U6-COMP): track 0.00 -> 2.33 mm
- net Net-(U6-SS): track 0.00 -> 2.14 mm
- net Net-(C16-Pad2): track 0.00 -> 2.02 mm
- net Net-(TEMP1-Pin_1): track 35.4 -> 34.8 mm
- net Net-(TEMP2-Pin_1): track 24.0 -> 24.2 mm, vias 1 -> 0
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
Commit message: all subcircuits other than rpp
Parts:
- moved D1 141.9 mm to (257.0, 144.9)
- moved D2 141.9 mm to (257.0, 148.2)
- moved D3 141.9 mm to (257.0, 150.8)
- moved D4 141.9 mm to (257.0, 153.4)
- moved D5 141.9 mm to (257.0, 156.0)
- moved D6 141.9 mm to (257.0, 158.6)
- moved G*** 71.2 mm to (248.2, 115.6)
- moved LOGO2 11.7 mm to (242.2, 66.4)
- moved Q5 8.77 mm to (157.3, 101.0), turned to 180 degrees
- moved R36 8.25 mm to (155.6, 97.5), turned to -90 degrees
- moved J4 5.06 mm to (123.3, 117.5)
- moved R34 2.43 mm to (158.8, 97.4), turned to -90 degrees
- moved R35 1.54 mm to (157.2, 97.4), turned to 90 degrees
- moved J1 0.95 mm to (135.8, 110.6)
- moved R33 0.82 mm to (160.8, 92.2), turned to 180 degrees
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Connections:
- PUMP1 pad 2: /PUMP_PWM -> /PUMP_FG
- PUMP1 pad 3: /PUMP_FG -> /PUMP_PWM
Routing:
- net /FAN_SCL: track 3.82 -> 47.9 mm
- net /PUMP_PWM: track 0.00 -> 42.7 mm
- net /FAN_SDA: track 2.15 -> 43.7 mm
- net /PUMP_FG: track 0.00 -> 38.6 mm
- net /TEMP1: track 2.04 -> 38.4 mm
- net /~{SMBALERT}: track 1.60 -> 37.9 mm, vias 0 -> 2
- net /TEMP2: track 1.90 -> 28.4 mm
- net /FLOW: track 4.53 -> 27.8 mm, vias 0 -> 1
- net /TEMP3: track 3.32 -> 26.0 mm, vias 0 -> 1
- net /CAN_H: track 0.00 -> 14.7 mm
- net /CAN_L: track 0.00 -> 14.5 mm
- net Net-(Q5-G): track 0.00 -> 3.38 mm
- net /Pump/PWM: track 0.00 -> 1.78 mm
