File: PTN-PumpControlBoard.kicad_pcb (KiCad board)
At the start: 2 copper layers, 53.1 x 81.9 mm, 114 parts, among them IC1 LM74502HDDFR, IC2 LM74502HDDFR, J1 PWR_CAN, J2 Pump_Temp, J3 Flow_Fan, J4 53307-2471, J5 SFH11-PBPC-D05-ST-BK, Q1 IRLML0030TRPBF, Q2 IRLML0030TRPBF, Q3 NVMFWS1D7N04XMT1G, Q4 NVMFWS1D7N04XMT1G, Q5 NVMFWS1D7N04XMT1G, Q6 NVMFWS1D7N04XMT1G, U1 EMC2305-1-AP-TR, U2 TLV9002QDRQ1, U3 LMR33630ADDA

Commit message: lookin cute
Parts:
- TP4: value 12V_OUT -> 12V
- moved D22 9.28 mm to (181.1, 119.4)
- moved R46 9.28 mm to (181.1, 117.8)
- moved TP2 9.27 mm to (177.7, 118.7)
Connections:
- J4 pad 14: /FLOW_LED -> /FAN_CHIP
- J4 pad 17: /LED1 -> /TEMP_LED
- J4 pad 18: /FAN_CHIP -> /FLOW_LED
- J4 pad 19: /TEMP_LED -> /LED1
Routing:
- net /PUMP_TACH: track 20.8 -> 108.4 mm
- net /PUMP_PWM: track 12.2 -> 85.7 mm
- net +3.3V: track 28.3 -> 91.5 mm, vias 0 -> 4
- net /PWM_PSOM: track 0.00 -> 59.3 mm, vias 0 -> 2
- net /TACH_PSOM: track 0.00 -> 46.3 mm, vias 0 -> 2
- net /Fans+Pump/PUMP_PWM_CHIP: track 0.00 -> 41.5 mm, vias 0 -> 2
- net /Fans+Pump/PUMP_TACH_CHIP: track 0.00 -> 36.1 mm, vias 0 -> 2
- net /LED1: track 0.00 -> 33.6 mm
- net /TEMP_LED: track 0.00 -> 29.8 mm
- net +12V: track 65.3 -> 93.9 mm
- net /FLOW_LED: track 0.00 -> 28.0 mm, vias 0 -> 2
- net /FAN_CHIP: track 0.00 -> 26.2 mm, vias 0 -> 2
- net /FAN1_PWM: track 23.2 -> 47.2 mm
- net /FAN1_TACH: track 19.9 -> 42.3 mm
- net /PUMP_LED: track 0.00 -> 21.3 mm
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
Commit message: pls don't crash on me again
Parts:
- D1, D13, D14, D2, D4: moved to B.Cu
- moved D2 49.1 mm to (172.4, 111.3), turned to 180 degrees
- moved D3 46.7 mm to (173.3, 118.4)
- moved D1 45.0 mm to (167.7, 98.9), turned to 0 degrees
- moved LOGO2 35.1 mm to (176.7, 58.2)
- moved D14 34.7 mm to (187.4, 96.0), turned to 180 degrees
- moved D5 29.4 mm to (155.6, 96.5)
- moved D13 26.7 mm to (185.2, 113.5), turned to -90 degrees
- moved D4 25.7 mm to (157.4, 112.8), turned to 0 degrees
- moved D6 23.0 mm to (155.6, 101.5)
- moved TP3 1.50 mm to (168.0, 55.5)
- moved TP1 1.32 mm to (186.1, 55.2)
- moved TP5 0.61 mm to (189.6, 55.2)
Connections:
- D1 pad 2: /PUMP_PWM -> /PWM_PSOM
- D2 pad 2: /PUMP_TACH -> /TACH_PSOM
Routing:
- net /FLOW1: track 38.7 -> 50.9 mm, vias 1 -> 3
- net /TEMP2: track 48.9 -> 58.2 mm, vias 2 -> 3
- net Net-(IC2-GATE): track 14.8 -> 6.45 mm
- net /FLOW2: track 34.0 -> 39.9 mm, vias 2 -> 3
- net /TEMP1: track 44.3 -> 48.3 mm, vias 2 -> 3
- net /PWM_PSOM: track 59.3 -> 62.0 mm
- net /TACH_PSOM: track 46.3 -> 48.8 mm
- net +24V: track 83.5 -> 85.4 mm, vias 4 -> 5
- net +12V: track 93.9 -> 95.7 mm
- net /FAN_SDA: track 35.9 -> 34.4 mm, vias 5 -> 4
- net /Power/12V_BUCKED: track 12.1 -> 10.7 mm
- net GND: track 42.3 -> 41.3 mm, vias 51 -> 56
- net /TEMP_IN2: track 38.1 -> 37.6 mm
Other:
- board text added: "SURABHI K LHRS 2025 PUMP CONTROLLER"
- board text removed: "PUMP CONTROLLER SURABHI K LHRS 2025"

Commit message: drc passingggg
Parts:
- moved LOGO1 70.6 mm to (159.5, 57.9)
- moved D2 0.69 mm to (172.8, 110.7)
- moved C11 0.67 mm to (155.1, 69.4)
- moved C12 0.67 mm to (155.1, 67.8)
- moved D1 0.21 mm to (167.6, 98.7)
Routing:
- net GND: track 41.3 -> 74.8 mm, vias 56 -> 82
- net +24V: track 85.4 -> 110.6 mm
- net Net-(IC2-GATE): track 6.45 -> 15.7 mm
- net /PUMP_TACH: track 108.4 -> 111.5 mm
- net /PUMP_PWM: track 85.7 -> 88.5 mm
- net +12V: track 95.7 -> 94.5 mm, vias 2 -> 4
- net /FLOW1: track 50.9 -> 51.2 mm, vias 3 -> 5
Other:
- board text added: "TEMP TPs"

Commit message: rounded corners and nanofit connectors
Parts:
- moved C10 32.5 mm to (131.8, 64.2)
- moved C11 32.5 mm to (122.7, 71.5)
- moved C12 32.5 mm to (122.7, 69.9)
- moved C13 32.5 mm to (125.0, 54.9)
- moved C14 32.5 mm to (125.0, 56.6)
- moved C15 32.5 mm to (125.0, 58.3)
- moved C16 32.5 mm to (125.0, 60.0)
- moved C18 32.5 mm to (131.8, 67.7)
- moved C19 32.5 mm to (119.1, 87.8)
- moved C2 32.5 mm to (138.2, 105.5)
- moved C20 32.5 mm to (129.1, 87.7)
- moved C3 32.5 mm to (138.9, 89.2)
- moved C5 32.5 mm to (143.4, 80.1)
- moved C6 32.5 mm to (142.8, 68.7)
- moved C8 32.5 mm to (138.0, 65.9)
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Other:
- outline, holes or cut-outs redrawn
