File: PTN-PumpControlBoard.kicad_sch (KiCad schematic)
At the start: 10 parts, among them J1 PeripheralCANConnector, U1 EMC2305-1-AP-TR, U2 PeripheralSOM, U3 ST7735R

Commit message: Initial layout with 1 pump, 2 temp, 1 flow all on front side
Connections:
- net FAN_SPEED: now also U2.15 (SPI1_MISO); no longer U2.3 (SPI2_MISO)
- net FLOW: now also U2.13 (SPI1_SCK); no longer U2.1 (SPI2_MOSI)
- net LCD_RESET: now also U2.3 (SPI2_MISO); no longer U2.15 (SPI1_MISO)
- net LCD_TFT_~{CS}: now also U2.7 (SPI2_NSS); no longer U2.19 (SPI1_NSS)
- net MOSI: now also U2.1 (SPI2_MOSI); no longer U2.17 (SPI1_MOSI)
- net PUMP_PG: now also U2.16 (I2C1_SDA); no longer U2.14 (I2C1_SCL)
- net PUMP_PWM: now also U2.14 (I2C1_SCL); no longer U2.16 (I2C1_SDA)
- net PUMP_SPEED: now also U2.17 (SPI1_MOSI); no longer U2.5 (SPI2_SCK)
- net SCLK: now also U2.5 (SPI2_SCK); no longer U2.13 (SPI1_SCK)
- net SYST_MODE: now also U2.19 (SPI1_NSS); no longer U2.7 (SPI2_NSS)
Changed lines of the file:
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@@
+		)
+	)
+	(label "PUMP_PG"
+		(at 135.89 49.53 0)
+		(fields_autoplaced yes)
+		(effects
+			(font
+				(size 1.27 1.27)
+			)
+			(justify left bottom)
+		)
+	)
+	(label "MOSI"
+		(at 135.89 77.47 0)
+		(fields_autoplaced yes)
+		(effects
+			(font
+				(size 1.27 1.27)
+			)
+			(justify left bottom)
 		)
 	)
@@
 		)
 	)
-	(label "PUMP_SPEED"
-		(at 135.89 74.93 0)
-		(fields_autoplaced yes)
-		(effects
-			(font
-				(size 1.27 1.27)
-			)
-			(justify left bottom)
-		)
-	)
 	(label "FAN2_PWM"
 		(at 172.72 46.99 0)
@@
 		)
 	)
-	(label "SCLK"
-		(at 135.89 63.5 0)
-		(fields_autoplaced yes)
-		(effects
-			(font
-				(size 1.27 1.27)
-			)
-			(justify left bottom)
-		)
-	)
 	(label "FAN2_PWM"
 		(at 25.4 113.03 180)
@@
 		)
 	)
-	(label "PUMP_PG"
-		(at 135.89 46.99 0)
+	(label "SCLK"
+		(at 135.89 74.93 0)
 		(fields_autoplaced yes)
 		(effects
@@
 		)
 	)
+	(label "LCD_TFT_~{CS}"
+		(at 135.89 72.39 0)
+		(fields_autoplaced yes)
+		(effects
+			(font
+				(size 1.27 1.27)
+			)
+			(justify left bottom)
+		)
+	)
+	(label "LCD_RESET"
+		(at 135.89 80.01 0)
+		(fields_autoplaced yes)
+		(effects
+			(font
+				(size 1.27 1.27)
+			)
+			(justify left bottom)
+		)
+	)
 	(label "SYST_MODE"
-		(at 135.89 72.39 0)
+		(at 135.89 60.96 0)
+		(fields_autoplaced yes)
+		(effects
+			(font
+				(size 1.27 1.27)
+			)
+			(justify left bottom)
+		)
+	)
+	(label "PUMP_PWM"
+		(at 135.89 46.99 0)
 		(fields_autoplaced yes)
 		(effects
@@
 		)
 	)
+	(label "FAN_SPEED"
+		(at 135.89 68.58 0)
+		(fields_autoplaced yes)
+		(effects
+			(font
+				(size 1.27 1.27)
+			)
+			(justify left bottom)
+		)
+	)
 	(label "FAN_SCL"
 		(at 205.74 27.94 180)
@@
 		)
 	)
+	(label "PUMP_SPEED"
+		(at 135.89 66.04 0)
+		(fields_autoplaced yes)
+		(effects
+			(font
+				(size 1.27 1.27)
+			)
+			(justify left bottom)
+		)
+	)
 	(label "MOSI"
 		(at 115.57 135.89 0)
@@
 	)
 	(label "FLOW"
-		(at 135.89 77.47 0)
-		(fields_autoplaced yes)
-		(effects
-			(font
-				(size 1.27 1.27)
-			)
-			(justify left bottom)
-		)
-	)
-	(label "FLOW"
 		(at 63.5 67.31 0)
 		(fields_autoplaced yes)
@@
 		)
 	)
-	(label "LCD_TFT_~{CS}"
-		(at 135.89 60.96 0)
-		(fields_autoplaced yes)
-		(effects
-			(font
-				(size 1.27 1.27)
-			)
-			(justify left bottom)
-		)
-	)
-	(label "PUMP_PWM"
-		(at 135.89 49.53 0)
-		(fields_autoplaced yes)
-		(effects
-			(font
-				(size 1.27 1.27)
-			)
-			(justify left bottom)
-		)
-	)
 	(label "FAN_SDA"
 		(at 205.74 30.48 180)
@@
 		)
 	)
-	(label "LCD_RESET"
-		(at 135.89 68.58 0)
-		(fields_autoplaced yes)
-		(effects
-			(font
-				(size 1.27 1.27)
-			)
-			(justify left bottom)
-		)
-	)
 	(label "SYST_MODE"
 		(at 63.5 29.21 0)
@@
 		)
 	)
-	(label "MOSI"
-		(at 135.89 66.04 0)
-		(fields_autoplaced yes)
-		(effects
-			(font
-				(size 1.27 1.27)
-			)
-			(justify left bottom)
-		)
-	)
 	(label "FAN_SCL"
 		(at 135.89 53.34 0)
@@
 		)
 	)
+	(label "FLOW"
+		(at 135.89 63.5 0)
+		(fields_autoplaced yes)
+		(effects
+			(font
+				(size 1.27 1.27)
+			)
+			(justify left bottom)
+		)
+	)
 	(label "FAN1_TACH"
 		(at 205.74 40.64 180)
@@
 		)
 	)
-	(label "FAN_SPEED"
-		(at 135.89 80.01 0)
-		(fields_autoplaced yes)
-		(effects
-			(font
-				(size 1.27 1.27)
-			)
-			(justify left bottom)
-		)
-	)

Commit message: schematic with 12V components, unigain buffers & extra temp sensor
Parts:
- removed U3: ST7735R, LCD:adafruit_st7735r, symbol Misc:ST7735
- added H1, H2, H3, H4: MountingHole, MountingHole:MountingHole_3.2mm_M3, symbol Mechanical:MountingHole
- added J2: CAN_OUT, Connector_Molex:Molex_Nano-Fit_105309-xx04_1x04_P2.50mm_Vertical, symbol utsvt-connectors:PeripheralCANConnector
- J1: value PeripheralCANConnector -> CAN_IN; footprint UTSVT_Connectors:Molex_MicroFit3.0_1x4xP3.00mm_PolarizingPeg_Vertical -> Connector_Molex:Molex_Nano-Fit_105309-xx04_1x04_P2.50mm_Vertical
Connections:
- net CAN_H: now also J2.3 (CAN_H)
- net CAN_L: now also J2.4 (CAN_L)
- net FAN1_PWM: now also U1.7 (PWM2); no longer U1.5 (PWM1)
- net FAN2_PWM: now also U1.5 (PWM1); no longer U1.7 (PWM2)
- net GNDPWR: now also J2.2 (GNDPWR)
- net +12V renamed +24V
- net +24V: now also J2.1 (24V)
- net FAN_SPEED: no longer names the net of U2.15 (SPI1_MISO)
- net LCD_RESET: no longer names the net of U2.3 (SPI2_MISO)
- net LCD_TFT_~{CS}: no longer names the net of U2.7 (SPI2_NSS)
- net MOSI: no longer names the net of U2.1 (SPI2_MOSI)
- net PUMP_SPEED: no longer names the net of U2.17 (SPI1_MOSI)
- net SCLK: no longer names the net of U2.5 (SPI2_SCK)
- net SYST_MODE: no longer names the net of U2.19 (SPI1_NSS)
- no-connect marks 9 -> 7
Other:
- removed sheet Switches
- sheet Fans ports: added TACH1, TACH2; removed TACH1_OUT, TACH2_OUT
- sheet Pump ports: added Shunt_A, Shunt_B; removed none
- note added: "3 ADC pins for thermistors pls"
- note removed: "can this be a gpio?"
- moved on the sheet: C1, C2, J1, R1, R2, R3, R4, U1, U2

Commit message: repicked parts to be 24V tolerant and changed corresponding circuitry
Parts:
- added D1: D_Zener, Diode_SMD:D_SOD-323F, symbol Device:D_Zener
- added TH1: Thermistor_PTC, Resistor_SMD:R_0603_1608Metric, symbol Device:Thermistor_PTC
- renumbered H3 to H2, H2 to H3, R2 to R1, R1 to R2, U2 to U1, U1 to U2
Connections:
- net +24V: now also TH1.1
- net FLOW: now also U1.19 (SPI1_NSS); no longer U1.13 (SPI1_SCK)
- net GND: now also D1.2 (A)
- net PUMP_PWM: now also U1.13 (SPI1_SCK); no longer U1.14 (I2C1_SCL)
- net PUMP_FG: now reaches U1.17 (SPI1_MOSI)
- net PUMP_PG: no longer names the net of U1.16 (I2C1_SDA)
- new net: D1.1 (K), TH1.2
- no-connect marks 7 -> 14
Other:
- sheet Pump ports: added FG; removed PG, Shunt_A, Shunt_B
- note added: "flow sensor only rated for 24V so this makes the board safe for 22-26V"

Commit message: reworked layout with 24V components but no testpoints & headers
Parts:
- J1: value CAN_IN -> CAN_OUT
- J2: value CAN_OUT -> CAN_IN
Connections:
- net PUMP_FG: now also U1.7 (SPI2_NSS); no longer U1.17 (SPI1_MOSI)
- net ~{SMBALERT}: now also U1.1 (SPI2_MOSI)
- no-connect marks 14 -> 13
Changed lines of the file:
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@@
 		)
 	)
-	(text_box "TODO/QUESTIONS:\n\n- is it ok to just change labels on psom? or new footprint?\n- low pass on sensors?"
+	(text_box "TODO/QUESTIONS:\n\n- is it ok to just change labels on psom? or new footprint?\n- low pass on sensors?\n- reverse polarity protection?"
 		(exclude_from_sim no)
-		(at 234.95 127 0)
+		(at 15.24 156.21 0)
 		(size 43.18 32.385)
 		(margins 0.9525 0.9525 0.9525 0.9525)
@@
 	)
 	(no_connect
+		(at 133.35 72.39)
+	)
+	(no_connect
 		(at 120.65 130.81)
-	)
-	(no_connect
-		(at 133.35 83.82)
-	)
-	(no_connect
-		(at 133.35 78.74)
 	)
 	(no_connect
@@
 	(wire
 		(pts
-			(xy 133.35 72.39) (xy 137.16 72.39)
+			(xy 133.35 83.82) (xy 137.16 83.82)
 		)
 		(stroke
@@
 	(wire
 		(pts
+			(xy 133.35 78.74) (xy 137.16 78.74)
+		)
+		(stroke
+			(width 0)
+			(type default)
+		)
+	)
+	(wire
+		(pts
 			(xy 36.83 121.92) (xy 36.83 124.46)
 		)
@@
 			(width 0)
 			(type default)
+		)
+	)
+	(label "~{SMBALERT}"
+		(at 137.16 83.82 0)
+		(effects
+			(font
+				(size 1.27 1.27)
+			)
+			(justify left bottom)
 		)
 	)
@@
 	)
 	(label "PUMP_FG"
-		(at 137.16 72.39 0)
+		(at 137.16 78.74 0)
 		(effects
 			(font
@@
 			)
 		)
-		(property "Value" "CAN_OUT"
+		(property "Value" "CAN_IN"
 			(at 170.18 54.61 0)
 			(effects
@@
 			)
 		)
-		(property "Value" "CAN_IN"
+		(property "Value" "CAN_OUT"
 			(at 170.18 25.4 0)
 			(effects

Commit message: added test points and headers, AGND and 12V not fully connected
Parts:
- added J3, J4: SFH11-PBPC-D05-ST-BK, Headers:CONN_SFH11-xxxC-D05-ST-XX_SUL, symbol UTSVT_Connectors:SFH11-PBPC-D05-ST-BK
- added LOGO1: Logo_Placeholder, symbol utsvt-misc:Logo_Placeholder
- renumbered C2 to C1, C1 to C2, H3 to H2, H2 to H3
Connections:
- net FAN1_PWM: now also J3.10
- net FAN1_TACH: now also J3.9
- net FAN2_PWM: now also J3.6
- net FAN2_TACH: now also J3.8
- net FAN_SCL: now also J3.5
- net FAN_SDA: now also J3.7
- net FLOW: now also J4.2
- net PUMP_FG: now also U1.3 (SPI2_MISO), J4.3; no longer U1.7 (SPI2_NSS)
- net PUMP_PWM: now also J4.1
- net TEMP1: now also J3.4
- net TEMP2: now also J3.2
- net TEMP3: now also J3.1
- net ~{SMBALERT}: now also J3.3
- no-connect marks 13 -> 20

Commit message: filled zones finally workinggggg
Parts:
- removed J3, J4: SFH11-PBPC-D05-ST-BK, Headers:CONN_SFH11-xxxC-D05-ST-XX_SUL, symbol UTSVT_Connectors:SFH11-PBPC-D05-ST-BK
- removed LOGO1: Logo_Placeholder, symbol utsvt-misc:Logo_Placeholder
- added J3, J4, J5: PPTC032LFBN-RC, Headers:SULLINS_PPTC032LFBN-RC, symbol PPTC032LFBN-RC-6_pin:PPTC032LFBN-RC
Connections:
- net FAN1_PWM: now also J5.4
- net FAN1_TACH: now also J5.6
- net FAN2_PWM: now also J5.1
- net FAN2_TACH: now also J5.2
- net FAN_SCL: now also J5.3
- net FAN_SDA: now also J5.5
- net FLOW: now also J3.2
- net PUMP_FG: now also J3.3
- net PUMP_PWM: now also J3.1
- net TEMP1: now also J4.4
- net TEMP2: now also J4.2
- net TEMP3: now also J4.1
- net ~{SMBALERT}: now also J4.3
- no-connect marks 20 -> 18

Commit message: added +24V and GND flat test points
Parts:
- added +24V, GND: Pad_TP, UTSVT_Special:TestPoint_HEX_3mmID, symbol Connector:TestPoint
Connections:
- net +24V: now also +24V.1
- net GND: now also GND.1

Commit message: updated pump datasheet
Parts:
- renumbered +24V to +24V1, GND to GND3
Changed lines of the file:
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@@
 		(dnp no)
 		(fields_autoplaced yes)
-		(property "Reference" "+24V"
+		(property "Reference" "+24V1"
 			(at 243.84 90.1699 90)
 			(effects
@@
 			(project "PTN-PumpControlBoard"
 				(path "/591f46f8-eb1d-42dc-a4cb-8182eac4ef58"
-					(reference "+24V")
+					(reference "+24V1")
 					(unit 1)
 				)
@@
 		(dnp no)
 		(fields_autoplaced yes)
-		(property "Reference" "GND"
+		(property "Reference" "GND3"
 			(at 243.84 96.5199 90)
 			(effects
@@
 			(project "PTN-PumpControlBoard"
 				(path "/591f46f8-eb1d-42dc-a4cb-8182eac4ef58"
-					(reference "GND")
-					(unit 1)
-				)
+					(reference "GND3")
+					(unit 1)
+				)
