File: PTN-PumpControlBoard.kicad_sch (KiCad schematic)
At the start: 19 parts, among them J1 53307-2471, J2 CAN_IN, J3 CAN_OUT, J4 SFH11-PBPC-D05-ST-BK, J5 SFH11-PBPC-D05-ST-BK

Commit message: cube sux
Connections:
- net FAULT: now also J1.17 (SPI1_MOSI); no longer J1.19 (SPI1_NSS)
- net FLOW: now also J1.15 (ADC1_IN11); no longer J1.12 (SPI2_NSS)
- net IMON: now also J1.19 (SPI1_NSS); no longer J1.23 (SPI1_SCK)
- net PUMP_FG: now also J1.23 (SPI1_SCK); no longer J1.14 (SPI2_MISO)
- net PUMP_PWM: now also J1.21 (SPI1_MISO); no longer J1.18 (SPI2_SCK)
- net ~{SMBALERT}: now also J1.12 (SPI2_NSS); no longer J1.16 (SPI2_MOSI)
Other:
- note added: "pa12"
- note added: "pa2"
- note added: "pa4"
- note added: "pa5"
- note added: "pa6"
- note added: "pb0"
- note added: "pb10"
- note added: "pb12"
- note added: "pb3"
- note added: "pb6"
- note added: "pb7"

Commit message: fan and temp subcircuits
Connections:
- net TEMP1: now also J1.11 (ADC1_IN9); no longer J1.9 (ADC1_IN7)
- net TEMP2: now also J1.9 (ADC1_IN7); no longer J1.11 (ADC1_IN9)
Changed lines of the file:
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@@
+		)
+	)
+	(label "TEMP1"
+		(at 135.89 58.42 0)
+		(effects
+			(font
+				(size 1.27 1.27)
+			)
+			(justify left bottom)
 		)
 	)
@@
 			)
 			(justify right bottom)
-		)
-	)
-	(label "TEMP2"
-		(at 135.89 58.42 0)
-		(effects
-			(font
-				(size 1.27 1.27)
-			)
-			(justify left bottom)
 		)
 	)
@@
 		)
 	)
-	(label "TEMP1"
+	(label "TEMP2"
 		(at 135.89 55.88 0)
 		(effects

Commit message: everything done other than the routing for logic analyzers
Connections:
- net FAULT: no longer names the net of J1.17 (SPI1_MOSI)
- net IMON: no longer names the net of J1.19 (SPI1_NSS)
- no-connect marks 11 -> 13
Other:
- sheet PowerProtection ports: added none; removed 24V_Ext, Fault, IMON_OUT
- note removed: "pa12"
- note removed: "pb0"

Commit message: doneee (hopefully)
Parts:
- LOGO1: footprint UTSVT_Logos:Hallock_Image_Small -> UTSVT_Logos:Hallock_Image_Tiny
Connections:
- net FAN1_PWM: now also J4.7; no longer J4.3
- net FAN2_PWM: now also J4.3; no longer J4.4
- net FAN2_TACH: now also J4.8; no longer J4.2
- net FAN_SCL: now also J5.5; no longer J4.6
- net FAN_SDA: now also J5.3; no longer J4.7
- net FLOW: now also J5.8; no longer J5.1
- net PUMP_FG: now also J5.4; no longer J5.2
- net PUMP_PWM: now also J5.6
- net TEMP1: now also J4.2; no longer J5.3
- net TEMP2: now also J4.4; no longer J5.4
- net TEMP3: now also J4.6; no longer J5.5
- net ~{SMBALERT}: now also J5.7; no longer J4.8
Changed lines of the file:
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@@
 		)
 	)
-	(text_box "QUESTIONS:\n\nTODO:\n~ cube mx ss\n~ make rpp circuit look nice\n~ steal psom buck calcs\n~ buck test points\n~ fan pwm in logic analyzer\n~ switch to pmos - scrapped\n~ temp range/voltage range\n~ bypass connector for buck\n~ pmos for pump pwm pin\n~ new pmos\nX 3.3V header?"
+	(text_box "QUESTIONS:\n\nTODO:\n~ cube mx ss\n~ make rpp circuit look nice\n~ steal psom buck calcs\n~ buck test points\n~ fan pwm in logic analyzer\n~ switch to pmos - scrapped\n~ temp range/voltage range\n~ bypass connector for buck\n~ pmos for pump pwm pin\n~ new pmos\n~ 3.3V header?"
 		(exclude_from_sim no)
 		(at 16.51 142.24 0)
@@
 	)
 	(no_connect
+		(at 234.95 67.31)
+	)
+	(no_connect
+		(at 234.95 69.85)
+	)
+	(no_connect
 		(at 95.25 74.93)
 	)
@@
 	)
 	(no_connect
-		(at 234.95 85.09)
+		(at 234.95 40.64)
 	)
 	(no_connect
@@
 	)
 	(no_connect
-		(at 234.95 80.01)
-	)
-	(no_connect
-		(at 234.95 82.55)
-	)
-	(no_connect
 		(at 95.25 69.85)
 	)
@@
 		)
 	)
+	(label "TEMP2"
+		(at 234.95 38.1 180)
+		(effects
+			(font
+				(size 1.27 1.27)
+			)
+			(justify right bottom)
+		)
+	)
 	(label "CAN_L"
 		(at 201.93 33.02 0)
@@
 		)
 	)
-	(label "PUMP_FG"
-		(at 234.95 69.85 180)
+	(label "FAN_SDA"
+		(at 26.67 30.48 180)
 		(effects
 			(font
@@
 		)
 	)
-	(label "FAN_SDA"
-		(at 26.67 30.48 180)
+	(label "FAN1_TACH"
+		(at 234.95 30.48 180)
 		(effects
 			(font
@@
 		)
 	)
+	(label "FLOW"
+		(at 234.95 85.09 180)
+		(effects
+			(font
+				(size 1.27 1.27)
+			)
+			(justify right bottom)
+		)
+	)
 	(label "TEMP3"
 		(at 64.77 55.88 0)
@@
 		)
 	)
-	(label "FAN1_TACH"
-		(at 234.95 30.48 180)
+	(label "FAN1_PWM"
+		(at 234.95 45.72 180)
 		(effects
 			(font
@@
 		)
 	)
-	(label "FAN_SCL"
-		(at 234.95 43.18 180)
-		(effects
-			(font
-				(size 1.27 1.27)
-			)
-			(justify right bottom)
-		)
-	)
 	(label "FLOW"
 		(at 118.11 113.03 0)
@@
 		)
 	)
-	(label "~{SMBALERT}"
-		(at 234.95 48.26 180)
-		(effects
-			(font
-				(size 1.27 1.27)
-			)
-			(justify right bottom)
-		)
-	)
 	(label "PUMP_FG"
 		(at 135.89 82.55 0)
@@
 		)
 	)
-	(label "FAN2_TACH"
-		(at 234.95 33.02 180)
+	(label "FAN_SCL"
+		(at 234.95 77.47 180)
 		(effects
 			(font
@@
 		)
 	)
-	(label "FAN2_PWM"
-		(at 234.95 38.1 180)
+	(label "TEMP1"
+		(at 234.95 33.02 180)
 		(effects
 			(font
@@
 	)
 	(label "PUMP_PWM"
-		(at 26.67 95.25 180)
+		(at 234.95 80.01 180)
 		(effects
 			(font
@@
 		)
 	)
-	(label "FLOW"
-		(at 234.95 67.31 180)
+	(label "PUMP_PWM"
+		(at 26.67 95.25 180)
 		(effects
 			(font
@@
 		)
 	)
-	(label "FAN1_PWM"
-		(at 64.77 27.94 0)
-		(effects
-			(font
-				(size 1.27 1.27)
-			)
-			(justify left bottom)
-		)
-	)
-	(label "FAN1_PWM"
+	(label "FAN2_PWM"
 		(at 234.95 35.56 180)
 		(effects
@@
 		)
 	)
-	(label "TEMP2"
-		(at 234.95 74.93 180)
+	(label "FAN1_PWM"
+		(at 64.77 27.94 0)
 		(effects
 			(font
 				(size 1.27 1.27)
 			)
-			(justify right bottom)
+			(justify left bottom)
 		)
 	)
-	(label "FAN_SDA"
-		(at 234.95 45.72 180)
+	(label "TEMP3"
+		(at 234.95 43.18 180)
 		(effects
 			(font
@@
 		)
 	)
+	(label "FAN_SDA"
+		(at 234.95 72.39 180)
+		(effects
+			(font
+				(size 1.27 1.27)
+			)
+			(justify right bottom)
+		)
+	)
 	(label "TEMP2"
 		(at 135.89 55.88 0)
@@
 		)
 	)
-	(label "TEMP1"
-		(at 234.95 72.39 180)
+	(label "FAN2_TACH"
+		(at 234.95 48.26 180)
+		(effects
+			(font
+				(size 1.27 1.27)
+			)
+			(justify right bottom)
+		)
+	)
+	(label "~{SMBALERT}"
+		(at 234.95 82.55 180)
 		(effects
 			(font
@@
 		)
 	)
-	(label "TEMP3"
-		(at 234.95 77.47 180)
+	(label "PUMP_FG"
+		(at 234.95 74.93 180)
 		(effects
 			(font
@@
 			)
 		)
-		(property "Footprint" "UTSVT_Logos:Hallock_Image_Small"
+		(property "Footprint" "UTSVT_Logos:Hallock_Image_Tiny"
 			(at 184.15 112.395 0)
 			(effects

Commit message: datasheets disappeared for some reason
Changed lines of the file:
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@@
 		)
 	)
-	(text_box "QUESTIONS:\n\nTODO:\n~ cube mx ss\n~ make rpp circuit look nice\n~ steal psom buck calcs\n~ buck test points\n~ fan pwm in logic analyzer\n~ switch to pmos - scrapped\n~ temp range/voltage range\n~ bypass connector for buck\n~ pmos for pump pwm pin\n~ new pmos\n~ 3.3V header?"
+	(text_box "QUESTIONS:\n\nTODO:\n~ cube mx ss\n~ make rpp circuit look nice\n~ steal psom buck calcs\n~ buck test points\n~ fan pwm in logic analyzer\n~ switch to pmos - scrapped\n~ temp range/voltage range\n~ bypass connector for buck\n~ pmos for pump pwm pin\n~ new pmos\n~ 3.3V header"
 		(exclude_from_sim no)
 		(at 16.51 142.24 0)

Commit message: moved psom to make room for usb
Parts:
- removed J5: SFH11-PBPC-D05-ST-BK, UTSVT_Connectors:CONN_SFH11-xxxC-D05-ST-XX_SUL, symbol UTSVT_Connectors:SFH11-PBPC-D05-ST-BK
Connections:
- net FAN1_PWM: now also J4.4; no longer J4.7
- net FAN2_PWM: no longer J4.3
- net FAN2_TACH: no longer J4.8
- net FAN_SCL: now also J4.5
- net FAN_SDA: now also J4.3
- net FLOW: now also J4.6
- net PUMP_PWM: now also J4.8
- net TEMP1: now also J1.9 (ADC1_IN7); no longer J1.11 (ADC1_IN9)
- net TEMP2: now also J1.11 (ADC1_IN9); no longer J1.9 (ADC1_IN7), J4.4
- net TEMP3: no longer J4.6
- net ~{SMBALERT}: now also J4.7
- no-connect marks 13 -> 10
Other:
- note removed: "only outputs, check pinout"
