File: PTN-PumpControlBoard.kicad_sch (KiCad schematic)
At the start: 32 parts, among them J1 Auxilary, J2 53307-2471, J3 PWR_CAN, J4 SFH11-PBPC-D05-ST-BK

Commit message: almost all footprints
Parts:
- D1, D2, D3, D4, D5, D6: footprint Diode_SMD:D_0603_1608Metric -> Diode_SMD:D_SMB; P/N CPDUC5V0R-HF -> SMBJ30CD-M3/I

Commit message: subcircuit layout
Parts:
- removed H2, H3, H4: MountingHole, MountingHole:MountingHole_3.2mm_M3, symbol Mechanical:MountingHole
- added H2, H3, H4: MountingHole, MountingHole:MountingHole_3.2mm_M3_Pad_TopBottom, symbol Mechanical:MountingHole_Pad
- H1: footprint MountingHole:MountingHole_3.2mm_M3 -> MountingHole:MountingHole_3.2mm_M3_Pad_TopBottom; symbol Mechanical:MountingHole -> Mechanical:MountingHole_Pad; now left out of the parts list
Connections:
- net TEMP1: no longer J1.9 (Temp1+)
- net TEMP2: no longer J1.10 (Temp2+)
- new net TEMP_IN1: J1.9 (Temp1+)
- new net TEMP_IN2: J1.10 (Temp2+)
- no-connect marks 0 -> 4

Commit message: main circuitry done
Parts:
- added J1: PWR_CAN, Connector_Molex:Molex_Nano-Fit_105310-xx06_2x03_P2.50mm_Vertical, symbol Connector_Generic:Conn_02x03_Top_Bottom
- added J10: PumpFans, UTSVT_Connectors:Molex_Nano-Fit_105310-xx10_2x05_P2.50mm_Vertical, symbol Connector_Generic:Conn_02x05_Top_Bottom
- added J2: PumpTemp, Connector_Molex:Molex_Nano-Fit_105310-xx08_2x04_P2.50mm_Vertical, symbol Connector_Generic:Conn_02x04_Top_Bottom
- added J3: FlowFan, Connector_Molex:Molex_Nano-Fit_105310-xx12_2x06_P2.50mm_Vertical, symbol Connector_Generic:Conn_02x06_Top_Bottom
- added J9: FlowTemp, UTSVT_Connectors:Molex_Nano-Fit_105310-xx10_2x05_P2.50mm_Vertical, symbol Connector_Generic:Conn_02x05_Top_Bottom
- renumbered J2 to J4, J4 to J5, J3 to J7, J1 to J8
Connections:
- net +12V: now also J10.1 (Pin_1), J2.1 (Pin_1), J3.1 (Pin_1), J3.3 (Pin_3), J9.1 (Pin_1), J9.3 (Pin_3)
- net +24V: now also J10.3 (Pin_3), J3.4 (Pin_4)
- net 24V_IN: now also J1.1 (Pin_1)
- net AGND: now also J2.7 (Pin_7), J2.8 (Pin_8), J9.10 (Pin_10), J9.9 (Pin_9)
- net CAN_H: now also J1.2 (Pin_2), J1.5 (Pin_5)
- net CAN_L: now also J1.3 (Pin_3), J1.6 (Pin_6)
- net FAN1_PWM: now also J10.9 (Pin_9), J3.11 (Pin_11)
- net FAN1_TACH: now also J10.4 (Pin_4), J3.5 (Pin_5)
- net FAN2_PWM: now also J10.10 (Pin_10), J3.12 (Pin_12)
- net FAN2_TACH: now also J10.5 (Pin_5), J3.6 (Pin_6)
- net FLOW1_SIG: now also J3.2 (Pin_2), J9.2 (Pin_2)
- net FLOW2_SIG: now also J3.8 (Pin_8), J9.7 (Pin_7)
- net GND: now also J1.4 (Pin_4), J10.6 (Pin_6), J10.8 (Pin_8), J2.5 (Pin_5), J3.10 (Pin_10), J3.7 (Pin_7), J3.9 (Pin_9), J9.6 (Pin_6), J9.8 (Pin_8)
- net PUMP_PWM: now also J5.4 (CH6), J10.7 (Pin_7), J2.6 (Pin_6); no longer J5.3 (CH7)
- net PUMP_TACH: now also J5.3 (CH7), J10.2 (Pin_2), J2.2 (Pin_2)
- net TEMP_IN1: now also J2.3 (Pin_3), J9.4 (Pin_4)
- net TEMP_IN2: now also J2.4 (Pin_4), J9.5 (Pin_5)
- net ~{SMBALERT}: no longer J5.4 (CH6)

Commit message: it's almost prettyyy
Parts:
- J2: value PumpTemp -> Pump_Temp
- J3: value FlowFan -> Flow_Fan
Changed lines of the file:
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@@
 			)
 		)
-		(property "Value" "FlowFan"
+		(property "Value" "Flow_Fan"
 			(at 233.68 -46.99 0)
 			(effects
@@
 			)
 		)
-		(property "Value" "PumpTemp"
+		(property "Value" "Pump_Temp"
 			(at 181.61 -45.72 0)
 			(effects

Commit message: lakshays bs
Changed lines of the file:
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@@
 		)
 	)
+	(text_box "to do:\n- turn pin header into 0 ohms\n- remove temp from logic analyzer and add tps\n- planes for 12V\n- put inductor on back And close to chip\n- round corners"
+		(exclude_from_sim no)
+		(at 251.46 139.7 0)
+		(size 30.48 20.32)
+		(margins 0.9525 0.9525 0.9525 0.9525)
+		(stroke
+			(width 0)
+			(type solid)
+		)
+		(fill
+			(type none)
+		)
+		(effects
+			(font
+				(size 1.27 1.27)
+			)
+			(justify left top)
+		)
+	)
 	(text_box "LOGOS"
 		(exclude_from_sim no)
@@
 			"////////////////////////////////////////////////////////////////////////////"
 			"////////////////////////////////////////////////////////////////////////////"
-			"/////////////////////////////////////////////////////////////w=="
+			"/////////////////////////////////////////////////////////////wAAAAAAAAAAAAAA"
+			"AAAAAAAAAAAAAAAAAAAAAAAAAAAAAAAAAAAAAAAAAAAAAAAAAAAAAAAAAAAAAAAAAAAAAAAAAAAA"
+			"AAAAAAAAAAAAAAAAAAAAAAAAAAAAAAAAAAAAAAAAAAAAAAAAAAAAAAAAAAAAAAAAAAAAAAAAAAAA"
+			"AAAAAAAAAAAAAAAAAAAAAAAAAAAAAAAAAAAAAAAAAAAAAAAAAAAAAAAAAAAAAAAAAAAAAAAAAAAA"
+			"AAAAAAAAAAAAAAAAAAAAAAAAAAAAAAAAAAAAAAAAAAAAAAAAAAAAAAAAAAAAAAAAAAAAAAAAAAAA"
+			"AAAAAAAAAAAAAAAAAAAAAAAAAAAAAAAAAAAAAAAAAAAAAAAAAAAAAAAAAAAAAAAAAAAAAAAAAAAA"
+			"AAAAAAAAAAAAAAAAAAAAAAAAAAAAAAAAAAAAAAAAAAAAAAAAAAAAAAAAAAAAAAAAAAAAAAAAAAAA"
+			"AAAAAAAAAAAAAAAAAAAAAAAAAAAAAAAAAAAAAAAAAAAAAAAAAAAAAAAAAAAAAAAAAAAAAAAAAAAA"
+			"AAAAAAAAAAAAAAAAAAAAAAAAAAAAAAAAAAAAAAAAAAAAAAAAAAAAAAAAAAAAAAAAAAAAAAAAAAAA"
+			"AAAAAAAAAAAAAAAAAAAAAAAAAAAAAAAAAAAAAAAAAAAAAAAAAAAAAAAAAAAAAAAAAAAAAAAAAAAA"
+			"AAAAAAAAAAAAAAAAAAAAAAAAAAAAAAAAAAAAAAAAAAAAAAAAAAAAAAAAAAAAAAAAAAAAAAAAAAAA"
+			"AAAAAAAAAAAAAAAAAAAAAAAAAAAAAAAAAAAAAAAAAAAAAAAAAAAAAAAAAAAAAAAAAAAAAAAAAAAA"
+			"AAAAAAAAAAAAAAAAAAAAAAAAAAAAAAAAAAAAAAAAAAAAAAAAAAAAAAAAAAAAAAAAAAAAAAAAAAAA"
+			"AAAAAAAAAAAAAAAAAAAAAAAAAAAAAAAAAAAAAAAAAAAAAAAAAAAAAAAAAAAAAAAAAAAAAAAAAAAA"
+			"AAAAAAAAAAAAAAAAAAAAAAAAAAAAAAAAAAAAAAAAAAAAAAAAAAAAAAAAAAAAAAAAAAAAAAAAAAAA"
+			"AAAAAAAAAAAAAAAAAAAAAAAAAAAAAAAAAAAAAAAAAAAAAAAAAAAAAAAAAAAAAAAAAAAAAAAAAAAA"
+			"AAAAAAAAAAAAAAAAAAAAAAAAAAAAAAAAAAAAAAAAAAAAAAAAAAAAAAAAAAAAAAAAAAAAAAAAAAAA"
+			"AAAAAAAAAAAAAAAAAAAAAAAAAAAAAAAAAAAAAAAAAAAAAAAAAAAAAAAAAAAAAAAAAAAAAAAAAAAA"
+			"AAAAAAAAAAAAAAAAAAAAAAAAAAAAAAAAAAAAAAAAAAAAAAAAAAAAAAAAAAAAAA=="
 		)
 	)

Commit message: jic
Connections:
- net TEMP1: no longer J5.10 (CH0)
- no-connect marks 4 -> 5
Changed lines of the file:
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@@
 		)
 	)
-	(text_box "to do:\n- turn pin header into 0 ohms\n- remove temp from logic analyzer and add tps\n- planes for 12V\n- put inductor on back And close to chip\n- round corners"
+	(text_box "to do:\n- remove temp from logic analyzer and add tps\n- planes for 12V, 12V bucked\n- round corners\n- move pwr debug elsewhere"
 		(exclude_from_sim no)
 		(at 251.46 139.7 0)
@@
 		(at 22.86 132.08)
 	)
+	(no_connect
+		(at 170.18 74.93)
+	)
 	(wire
 		(pts
@@
 		(effects
 			(font
-				(size 1.27 1.27)
-			)
-			(justify right bottom)
-		)
-	)
-	(label "TEMP1"
-		(at 170.18 74.93 180)
-		(effects
-			(font

Commit message: almost there
Parts:
- removed J10: PumpFans, UTSVT_Connectors:Molex_Nano-Fit_105310-xx10_2x05_P2.50mm_Vertical, symbol Connector_Generic:Conn_02x05_Top_Bottom
- removed J9: FlowTemp, UTSVT_Connectors:Molex_Nano-Fit_105310-xx10_2x05_P2.50mm_Vertical, symbol Connector_Generic:Conn_02x05_Top_Bottom

Commit message: lookin cute
Connections:
- net FAN_CHIP: now also J4.14 (SPI2_MISO); no longer J4.18 (SPI2_SCK)
- net FLOW_LED: now also J4.18 (SPI2_SCK); no longer J4.14 (SPI2_MISO)
- net LED1: now also J4.19 (SPI1_NSS); no longer J4.17 (SPI1_MOSI)
- net TEMP_LED: now also J4.17 (SPI1_MOSI); no longer J4.19 (SPI1_NSS)
Changed lines of the file:
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@@
+		)
+	)
+	(label "TEMP_LED"
+		(at 130.81 85.09 0)
+		(effects
+			(font
+				(size 1.27 1.27)
+			)
+			(justify left bottom)
 		)
 	)
@@
 		)
 	)
-	(label "TEMP_LED"
-		(at 130.81 80.01 0)
-		(effects
-			(font
-				(size 1.27 1.27)
-			)
-			(justify left bottom)
-		)
-	)
 	(label "FAN_CHIP"
 		(at 59.69 152.4 0)
@@
 		)
 	)
-	(label "FLOW_LED"
-		(at 130.81 76.2 0)
-		(effects
-			(font
-				(size 1.27 1.27)
-			)
-			(justify left bottom)
-		)
-	)
 	(label "FAN_SCL"
 		(at 170.18 85.09 180)
@@
 		)
 	)
-	(label "LED1"
-		(at 130.81 85.09 0)
-		(effects
-			(font
-				(size 1.27 1.27)
-			)
-			(justify left bottom)
-		)
-	)
 	(label "FAN1_PWM"
 		(at 170.18 82.55 180)
@@
 		)
 	)
-	(label "FAN_CHIP"
-		(at 130.81 71.12 0)
-		(effects
-			(font
-				(size 1.27 1.27)
-			)
-			(justify left bottom)
-		)
-	)
 	(label "TEMP2"
 		(at 130.81 60.96 0)
@@
 		)
 	)
+	(label "FLOW_LED"
+		(at 130.81 71.12 0)
+		(effects
+			(font
+				(size 1.27 1.27)
+			)
+			(justify left bottom)
+		)
+	)
 	(label "FAN2_TACH"
 		(at 227.33 -31.75 180)
@@
 		)
 	)
+	(label "LED1"
+		(at 130.81 80.01 0)
+		(effects
+			(font
+				(size 1.27 1.27)
+			)
+			(justify left bottom)
+		)
+	)
 	(label "FLOW1"
 		(at 170.18 87.63 180)
@@
 		(effects
 			(font
+				(size 1.27 1.27)
+			)
+			(justify left bottom)
+		)
+	)
+	(label "FAN_CHIP"
+		(at 130.81 76.2 0)
+		(effects
+			(font
