File: TempSensors.kicad_sch (KiCad schematic)
At the start: 30 parts, among them U7 TLV9002QDRQ1, U8 TLV9002QDRQ1

Commit message: added kicad bild submodule
Parts:
- C10, C11, C8, C9: value 1uF -> .1uF
- R25, R27, R30: value 10k -> 0
Connections:
- net AGND: now also C10.2, C8.2
- net VDDA: now also U7.6 (V+), U8.6 (V+)
Other:
- moved on the sheet: C10, C8
Changed lines of the file:
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@@
 	)
 	(junction
+		(at 209.55 35.56)
+		(diameter 0)
+		(color 0 0 0 0)
+	)
+	(junction
 		(at 142.24 63.5)
 		(diameter 0)
@@
 	)
 	(junction
+		(at 146.05 100.33)
+		(diameter 0)
+		(color 0 0 0 0)
+	)
+	(junction
 		(at 163.83 44.45)
 		(diameter 0)
@@
 	(wire
 		(pts
-			(xy 209.55 62.23) (xy 209.55 63.5)
+			(xy 146.05 100.33) (xy 158.75 100.33)
 		)
 		(stroke
@@
 	(wire
 		(pts
-			(xy 73.66 116.84) (xy 74.93 116.84)
+			(xy 209.55 62.23) (xy 209.55 63.5)
 		)
 		(stroke
@@
 	(wire
 		(pts
-			(xy 73.66 107.95) (xy 74.93 107.95)
+			(xy 73.66 116.84) (xy 74.93 116.84)
 		)
 		(stroke
@@
 	(wire
 		(pts
-			(xy 120.65 41.91) (xy 123.19 41.91)
+			(xy 73.66 107.95) (xy 74.93 107.95)
 		)
 		(stroke
@@
 	(wire
 		(pts
-			(xy 167.64 44.45) (xy 167.64 52.07)
+			(xy 120.65 41.91) (xy 123.19 41.91)
 		)
 		(stroke
@@
 	(wire
 		(pts
-			(xy 74.93 44.45) (xy 78.74 44.45)
+			(xy 167.64 44.45) (xy 167.64 52.07)
 		)
 		(stroke
@@
 	(wire
 		(pts
-			(xy 58.42 62.23) (xy 58.42 63.5)
+			(xy 74.93 44.45) (xy 78.74 44.45)
 		)
 		(stroke
@@
 	(wire
 		(pts
-			(xy 78.74 44.45) (xy 78.74 52.07)
+			(xy 58.42 62.23) (xy 58.42 63.5)
 		)
 		(stroke
@@
 	(wire
 		(pts
-			(xy 209.55 33.02) (xy 209.55 34.29)
+			(xy 78.74 44.45) (xy 78.74 52.07)
 		)
 		(stroke
@@
 	(wire
 		(pts
+			(xy 209.55 35.56) (xy 219.71 35.56)
+		)
+		(stroke
+			(width 0)
+			(type default)
+		)
+	)
+	(wire
+		(pts
 			(xy 53.34 127) (xy 58.42 127)
 		)
@@
 	(wire
 		(pts
-			(xy 209.55 39.37) (xy 209.55 40.64)
+			(xy 209.55 35.56) (xy 209.55 40.64)
+		)
+		(stroke
+			(width 0)
+			(type default)
+		)
+	)
+	(wire
+		(pts
+			(xy 209.55 33.02) (xy 209.55 35.56)
 		)
 		(stroke
@@
 	(wire
 		(pts
+			(xy 146.05 100.33) (xy 146.05 105.41)
+		)
+		(stroke
+			(width 0)
+			(type default)
+		)
+	)
+	(wire
+		(pts
 			(xy 163.83 44.45) (xy 167.64 44.45)
 		)
@@
 			)
 		)
-		(property "Value" "1uF"
+		(property "Value" ".1uF"
 			(at 142.24 126.238 0)
 			(effects
@@
 			)
 		)
-		(property "Value" "10k"
+		(property "Value" "0"
 			(at 60.96 123.1899 0)
 			(effects
@@
 	(symbol
 		(lib_id "Device:C_Small")
-		(at 209.55 36.83 0)
+		(at 219.71 38.1 0)
 		(unit 1)
 		(exclude_from_sim no)
@@
 		(dnp no)
 		(property "Reference" "C8"
-			(at 205.74 36.068 0)
+			(at 215.9 37.338 0)
 			(effects
 				(font
@@
 			)
 		)
-		(property "Value" "1uF"
-			(at 205.74 38.608 0)
+		(property "Value" ".1uF"
+			(at 215.9 39.878 0)
 			(effects
 				(font
@@
 		)
 		(property "Footprint" "Capacitor_SMD:C_0805_2012Metric"
-			(at 209.55 36.83 0)
+			(at 219.71 38.1 0)
 			(effects
 				(font
@@
 		)
 		(property "Datasheet" "https://www.mouser.com/datasheet/2/447/KEM_C1006_X5R_SMD-3316465.pdf"
-			(at 209.55 36.83 0)
+			(at 219.71 38.1 0)
 			(effects
 				(font
@@
 		)
 		(property "Description" "Unpolarized capacitor, small symbol"
-			(at 209.55 36.83 0)
+			(at 219.71 38.1 0)
 			(effects
 				(font
@@
 		)
 		(property "P/N" "C0805C105K5PACTU"
-			(at 209.55 36.83 0)
+			(at 219.71 38.1 0)
 			(effects
 				(font
@@
 			)
 		)
-		(property "Value" "1uF"
+		(property "Value" ".1uF"
 			(at 205.74 61.468 0)
 			(effects
@@
 	(symbol
 		(lib_id "Device:C_Small")
-		(at 146.05 102.87 0)
+		(at 158.75 102.87 0)
 		(unit 1)
 		(exclude_from_sim no)
@@
 		(dnp no)
 		(property "Reference" "C10"
-			(at 142.24 102.108 0)
+			(at 154.94 102.108 0)
 			(effects
 				(font
@@
 			)
 		)
-		(property "Value" "1uF"
-			(at 142.24 104.648 0)
+		(property "Value" ".1uF"
+			(at 154.94 104.648 0)
 			(effects
 				(font
@@
 		)
 		(property "Footprint" "Capacitor_SMD:C_0805_2012Metric"
-			(at 146.05 102.87 0)
+			(at 158.75 102.87 0)
 			(effects
 				(font
@@
 		)
 		(property "Datasheet" "https://www.mouser.com/datasheet/2/447/KEM_C1006_X5R_SMD-3316465.pdf"
-			(at 146.05 102.87 0)
+			(at 158.75 102.87 0)
 			(effects
 				(font
@@
 		)
 		(property "Description" "Unpolarized capacitor, small symbol"
-			(at 146.05 102.87 0)
+			(at 158.75 102.87 0)
 			(effects
 				(font
@@
 		)
 		(property "P/N" "C0805C105K5PACTU"
-			(at 146.05 102.87 0)
+			(at 158.75 102.87 0)
 			(effects
 				(font
@@
 			)
 		)
-		(property "Value" "10k"
+		(property "Value" "0"
 			(at 149.86 59.6899 0)
 			(effects
@@
 	(symbol
 		(lib_id "power:GND")
+		(at 158.75 105.41 0)
+		(unit 1)
+		(exclude_from_sim no)
+		(in_bom yes)
+		(on_board yes)
+		(dnp no)
+		(property "Reference" "#PWR065"
+			(at 158.75 111.76 0)
+			(effects
+				(font
+					(size 1.27 1.27)
+				)
+				(hide yes)
+			)
+		)
+		(property "Value" "AGND"
+			(at 158.75 108.966 0)
+			(effects
+				(font
+					(size 1.27 1.27)
+				)
+			)
+		)
+		(property "Footprint" ""
+			(at 158.75 105.41 0)
+			(effects
+				(font
+					(size 1.27 1.27)
+				)
+				(hide yes)
+			)
+		)
+		(property "Datasheet" ""
+			(at 158.75 105.41 0)
+			(effects
+				(font
+					(size 1.27 1.27)
+				)
+				(hide yes)
+			)
+		)
+		(property "Description" "Power symbol creates a global label with name \"GND\" , ground"
+			(at 158.75 105.41 0)
+			(effects
+				(font
+					(size 1.27 1.27)
+				)
+				(hide yes)
+			)
+		)
+		(pin "1"
+		)
+		(instances
+			(project "PTN-PumpControlBoard"
+				(path "/591f46f8-eb1d-42dc-a4cb-8182eac4ef58/0e5255e2-25aa-4e9a-a6ff-997dc3e398fd"
+					(reference "#PWR065")
+					(unit 1)
+				)
+			)
+		)
+	)
+	(symbol
+		(lib_id "power:GND")
+		(at 219.71 40.64 0)
+		(unit 1)
+		(exclude_from_sim no)
+		(in_bom yes)
+		(on_board yes)
+		(dnp no)
+		(property "Reference" "#PWR064"
+			(at 219.71 46.99 0)
+			(effects
+				(font
+					(size 1.27 1.27)
+				)
+				(hide yes)
+			)
+		)
+		(property "Value" "AGND"
+			(at 219.71 44.196 0)
+			(effects
+				(font
+					(size 1.27 1.27)
+				)
+			)
+		)
+		(property "Footprint" ""
+			(at 219.71 40.64 0)
+			(effects
+				(font
+					(size 1.27 1.27)
+				)
+				(hide yes)
+			)
+		)
+		(property "Datasheet" ""
+			(at 219.71 40.64 0)
+			(effects
+				(font
+					(size 1.27 1.27)
+				)
+				(hide yes)
+			)
+		)
+		(property "Description" "Power symbol creates a global label with name \"GND\" , ground"
+			(at 219.71 40.64 0)
+			(effects
+				(font
+					(size 1.27 1.27)
+				)
+				(hide yes)
+			)
+		)
+		(pin "1"
+		)
+		(instances
+			(project "PTN-PumpControlBoard"
+				(path "/591f46f8-eb1d-42dc-a4cb-8182eac4ef58/0e5255e2-25aa-4e9a-a6ff-997dc3e398fd"
+					(reference "#PWR064")
+					(unit 1)
+				)
+			)
+		)
+	)
+	(symbol
+		(lib_id "power:GND")
 		(at 38.1 64.77 0)
 		(unit 1)
@@
 			)
 		)
-		(property "Value" "10k"
+		(property "Value" "0"
 			(at 60.96 59.6899 0)
 			(effects
