File: TempSensors.kicad_sch (KiCad schematic)
At the start: 30 parts, among them U7 TLV9002QDRQ1, U8 TLV9002QDRQ1

Commit message: low pass for temp & flyback diodes
Parts:
- added C12, C13, C14: 15uF, Capacitor_SMD:C_0805_2012Metric, symbol Device:C_Small
- added R4, R7, R8: 1k, Resistor_SMD:R_0603_1608Metric, symbol Device:R_US
- R25, R27, R30: now not fitted
Connections:
- net AGND: now also C12.2, C13.2, C14.2
- net TEMP_SEN1: now also C12.1, R4.2; no longer R17.1, T_TP1.1, U7.7
- net TEMP_SEN2: now also C13.1, R7.2; no longer R28.1, T_TP2.1, U7.5
- net TEMP_SEN3: now also C14.1, R8.2; no longer R31.1, T_TP3.1, U8.7
- new net: R28.1, R7.1, T_TP2.1, U7.5
- new net: R17.1, R4.1, T_TP1.1, U7.7
- new net: R31.1, R8.1, T_TP3.1, U8.7
Other:
- moved on the sheet: C10, C11, C6, C8, C9, R2, R26, R28, TEMP2, T_OUT5, T_TP2, U7B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

Commit message: fixed all review notes for schematic
Parts:
- removed C10: .1uF, Capacitor_SMD:C_0805_2012Metric, symbol Device:C_Small
- removed U8: TLV9002QDRQ1, OpAmp:SOIC127P600X175-8N, symbol Amplifier_Operational:OP249GS
- added C11: .1uF, Capacitor_SMD:C_0805_2012Metric, symbol Device:C_Small
- added IC1, IC2: TLV9002QDRQ1, OpAmp:SOIC127P600X175-8N, symbol OpAmp:TLV9002QDRQ1
- added U4: TLV9002QDRQ1, OpAmp:SOIC127P600X175-8N, symbol Amplifier_Operational:OP249GS
- renumbered C14 to C10, C11 to C12, C5 to C3, C12 to C4, C6 to C5, C13 to C6, C8 to C7, C9 to C8, C7 to C9, R16 to R10, R1 to R11, R17 to R12, R4 to R13, R25 to R14, R26 to R15, R2 to R16, R28 to R17, R7 to R18, R27 to R19, R29 to R20, R3 to R21, R31 to R22, R8 to R23, R30 to R24, TEMP3 to TEMP2, TEMP2 to TEMP3, T_OUT4 to T_OUT1, T_OUT6 to T_OUT2, T_OUT5 to T_OUT3, T_TP3 to T_TP2, T_TP2 to T_TP3, U7 to U3
Connections:
- net AGND: now also C11.2, IC1.4 (V-), IC2.4 (V-)
- net VDDA: now also U3.8 (V+), C11.1, IC1.8 (V+), IC2.8 (V+), U4.8 (V+); no longer U3.6 (V+)
- net at C12.1: now also U4.4 (V-)
- net IN1+: now reaches C3.1, R11.2
- net IN1+: now also U3.3 (+), IC1.3 (IN1+); no longer U3.1 (+)
- net OUT2: now reaches R17.1, R18.1, T_TP3.1
- net OUT2: now also U3.7, IC1.7 (OUT2); no longer U3.5
- net OUT1: now reaches R12.1, R13.1, T_TP1.1
- net OUT1: now also U3.1, IC1.1 (OUT1); no longer U3.7
- net IN1-: now reaches R12.2, R14.1
- net IN1-: now also U3.2 (-), IC1.2 (IN1-); no longer U3.8 (-)
- net IN2+: now reaches C5.1, R16.2
- net IN2+: now also U3.5 (+), IC1.5 (IN2+); no longer U3.3 (+)
- net IN3-: now reaches R22.2, R24.1
- net IN3-: now also IC2.2 (IN1-), U4.2 (-)
- net OUT3: now reaches R22.1, R23.1, T_TP2.1
- net OUT3: now also IC2.1 (OUT1), U4.1
- net at C8.1: now also U3.4 (V-); no longer U3.2 (V-)
- net IN2-: now reaches R17.2, R19.1
- net IN2-: now also U3.6 (-), IC1.6 (IN2-); no longer U3.4 (-)
- net IN3+: now reaches C9.1, R21.2
- net IN3+: now also IC2.3 (IN1+), U4.3 (+)
- no-connect marks 3 -> 6
Other:
- note added: "used dummy symbols in other boxes for schematic clarity"
- moved on the sheet: C12, C7, C8, U3C

Commit message: review notes
Connections:
- net AGND: no longer IC1.4 (V-), IC2.4 (V-)
- net V2-: now reaches C12.1, U4.4 (V-)
- net V2-: now also IC2.4 (V-)
- net V1-: now reaches C8.1, U3.4 (V-)
- net V1-: now also IC1.4 (V-)
Other:
- note added: "write lowest and highest temp possible + voltage"

Commit message: schematic changes before switching submodules
Changed lines of the file:
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@@
+		)
+	)
+	(text_box "TEMP SENSORS:\n\nMin: -40C, 191.8k, 3.136V\nMax: 120C, 0.583k, 0.182V"
+		(exclude_from_sim no)
+		(at 120.65 139.7 0)
+		(size 47.625 10.16)
+		(margins 0.9525 0.9525 0.9525 0.9525)
+		(stroke
+			(width 0)
+			(type solid)
+		)
+		(fill
+			(type none)
+		)
+		(effects
+			(font
+				(size 1.27 1.27)
+				(thickness 0.1588)
+			)
+			(justify left top)
 		)
 	)

Commit message: fixed submodule, schematic basically done
Other:
- note removed: "write lowest and highest temp possible + voltage"
- moved on the sheet: C10, C11, C12, C3, C4, C5, C6, C7, C8, C9, IC1, IC2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

Commit message: finalized schematic (pls be the last time)
Parts:
- renumbered R10 to R12, R11 to R13, R12 to R14, R13 to R15, R14 to R16, R15 to R17, R16 to R18, R17 to R19, R18 to R20, R19 to R21, R20 to R22, R21 to R23, R22 to R24, R23 to R25, R24 to R26
Other:
- note added: "op amp has no associated footprint, only for schematic readability"
- note added: "symbols that have the actual footprints"
- note removed: "used dummy symbols in other boxes for schematic clarity"
Changed lines of the file:
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@@
 		)
 	)
-	(text "used dummy symbols in other boxes for schematic clarity"
+	(text "op amp has no associated footprint, only for schematic readability"
 		(exclude_from_sim no)
-		(at 61.976 183.642 0)
+		(at 70.104 144.526 0)
+		(effects
+			(font
+				(size 1.27 1.27)
+			)
+		)
+	)
+	(text "op amp has no associated footprint, only for schematic readability"
+		(exclude_from_sim no)
+		(at 70.104 85.09 0)
+		(effects
+			(font
+				(size 1.27 1.27)
+			)
+		)
+	)
+	(text "symbols that have the actual footprints"
+		(exclude_from_sim no)
+		(at 71.374 183.642 0)
+		(effects
+			(font
+				(size 1.27 1.27)
+			)
+		)
+	)
+	(text "op amp has no associated footprint, only for schematic readability"
+		(exclude_from_sim no)
+		(at 171.704 85.09 0)
 		(effects
 			(font
@@
 		(dnp no)
 		(fields_autoplaced yes)
-		(property "Reference" "R11"
+		(property "Reference" "R13"
 			(at 46.99 48.26 90)
 			(effects
@@
 			(project ""
 				(path "/591f46f8-eb1d-42dc-a4cb-8182eac4ef58/0e5255e2-25aa-4e9a-a6ff-997dc3e398fd"
-					(reference "R11")
+					(reference "R13")
 					(unit 1)
 				)
@@
 		(dnp no)
 		(fields_autoplaced yes)
-		(property "Reference" "R18"
+		(property "Reference" "R20"
 			(at 187.96 50.8 90)
 			(effects
@@
 			(project "PTN-PumpControlBoard"
 				(path "/591f46f8-eb1d-42dc-a4cb-8182eac4ef58/0e5255e2-25aa-4e9a-a6ff-997dc3e398fd"
-					(reference "R18")
+					(reference "R20")
 					(unit 1)
 				)
@@
 		(dnp no)
 		(fields_autoplaced yes)
-		(property "Reference" "R16"
+		(property "Reference" "R18"
 			(at 148.59 48.26 90)
 			(effects
@@
 			(project "PTN-PumpControlBoard"
 				(path "/591f46f8-eb1d-42dc-a4cb-8182eac4ef58/0e5255e2-25aa-4e9a-a6ff-997dc3e398fd"
-					(reference "R16")
+					(reference "R18")
 					(unit 1)
 				)
@@
 		(on_board yes)
 		(dnp yes)
-		(property "Reference" "R24"
+		(property "Reference" "R26"
 			(at 60.96 129.5399 0)
 			(effects
@@
 			(project "PTN-PumpControlBoard"
 				(path "/591f46f8-eb1d-42dc-a4cb-8182eac4ef58/0e5255e2-25aa-4e9a-a6ff-997dc3e398fd"
-					(reference "R24")
+					(reference "R26")
 					(unit 1)
 				)
@@
 		(on_board yes)
 		(dnp no)
-		(property "Reference" "R10"
+		(property "Reference" "R12"
 			(at 40.64 44.4499 0)
 			(effects
@@
 			(project "PTN-PumpControlBoard"
 				(path "/591f46f8-eb1d-42dc-a4cb-8182eac4ef58/0e5255e2-25aa-4e9a-a6ff-997dc3e398fd"
-					(reference "R10")
+					(reference "R12")
 					(unit 1)
 				)
@@
 		(on_board yes)
 		(dnp no)
-		(property "Reference" "R20"
+		(property "Reference" "R22"
 			(at 40.64 104.1399 0)
 			(effects
@@
 			(project "PTN-PumpControlBoard"
 				(path "/591f46f8-eb1d-42dc-a4cb-8182eac4ef58/0e5255e2-25aa-4e9a-a6ff-997dc3e398fd"
-					(reference "R20")
+					(reference "R22")
 					(unit 1)
 				)
@@
 		(on_board yes)
 		(dnp no)
-		(property "Reference" "R12"
+		(property "Reference" "R14"
 			(at 67.8181 68.58 90)
 			(effects
@@
 			(project "PTN-PumpControlBoard"
 				(path "/591f46f8-eb1d-42dc-a4cb-8182eac4ef58/0e5255e2-25aa-4e9a-a6ff-997dc3e398fd"
-					(reference "R12")
+					(reference "R14")
 					(unit 1)
 				)
@@
 		(dnp no)
 		(fields_autoplaced yes)
-		(property "Reference" "R13"
+		(property "Reference" "R15"
 			(at 86.36 50.8 90)
 			(effects
@@
 			(project "PTN-PumpControlBoard"
 				(path "/591f46f8-eb1d-42dc-a4cb-8182eac4ef58/0e5255e2-25aa-4e9a-a6ff-997dc3e398fd"
-					(reference "R13")
+					(reference "R15")
 					(unit 1)
 				)
@@
 		(on_board yes)
 		(dnp no)
-		(property "Reference" "R17"
+		(property "Reference" "R19"
 			(at 169.4181 68.58 90)
 			(effects
@@
 			(project "PTN-PumpControlBoard"
 				(path "/591f46f8-eb1d-42dc-a4cb-8182eac4ef58/0e5255e2-25aa-4e9a-a6ff-997dc3e398fd"
-					(reference "R17")
+					(reference "R19")
 					(unit 1)
 				)
@@
 		(dnp no)
 		(fields_autoplaced yes)
-		(property "Reference" "R23"
+		(property "Reference" "R25"
 			(at 86.36 110.49 90)
 			(effects
@@
 			(project "PTN-PumpControlBoard"
 				(path "/591f46f8-eb1d-42dc-a4cb-8182eac4ef58/0e5255e2-25aa-4e9a-a6ff-997dc3e398fd"
-					(reference "R23")
+					(reference "R25")
 					(unit 1)
 				)
@@
 		(on_board yes)
 		(dnp no)
-		(property "Reference" "R22"
+		(property "Reference" "R24"
 			(at 67.8181 128.27 90)
 			(effects
@@
 			(project "PTN-PumpControlBoard"
 				(path "/591f46f8-eb1d-42dc-a4cb-8182eac4ef58/0e5255e2-25aa-4e9a-a6ff-997dc3e398fd"
-					(reference "R22")
+					(reference "R24")
 					(unit 1)
 				)
@@
 		(on_board yes)
 		(dnp yes)
-		(property "Reference" "R19"
+		(property "Reference" "R21"
 			(at 162.56 69.8499 0)
 			(effects
@@
 			(project "PTN-PumpControlBoard"
 				(path "/591f46f8-eb1d-42dc-a4cb-8182eac4ef58/0e5255e2-25aa-4e9a-a6ff-997dc3e398fd"
-					(reference "R19")
+					(reference "R21")
 					(unit 1)
 				)
@@
 		(dnp no)
 		(fields_autoplaced yes)
-		(property "Reference" "R21"
+		(property "Reference" "R23"
 			(at 46.99 107.95 90)
 			(effects
@@
 			(project "PTN-PumpControlBoard"
 				(path "/591f46f8-eb1d-42dc-a4cb-8182eac4ef58/0e5255e2-25aa-4e9a-a6ff-997dc3e398fd"
-					(reference "R21")
+					(reference "R23")
 					(unit 1)
 				)
@@
 		(on_board yes)
 		(dnp yes)
-		(property "Reference" "R14"
+		(property "Reference" "R16"
 			(at 60.96 69.8499 0)
 			(effects
@@
 			(project "PTN-PumpControlBoard"
 				(path "/591f46f8-eb1d-42dc-a4cb-8182eac4ef58/0e5255e2-25aa-4e9a-a6ff-997dc3e398fd"
-					(reference "R14")
+					(reference "R16")
 					(unit 1)
 				)
@@
 		(on_board yes)
 		(dnp no)
-		(property "Reference" "R15"
+		(property "Reference" "R17"
 			(at 142.24 44.4499 0)
 			(effects
@@
 			(project "PTN-PumpControlBoard"
 				(path "/591f46f8-eb1d-42dc-a4cb-8182eac4ef58/0e5255e2-25aa-4e9a-a6ff-997dc3e398fd"
-					(reference "R15")
+					(reference "R17")
 					(unit 1)
 				)

Commit message: fan and temp subcircuits
Parts:
- removed T_OUT2, T_OUT3, T_TP2, T_TP3: Pad_TP, UTSVT_Special:TestPoint_HEX_3mmID, symbol Connector:TestPoint
- renumbered TEMP3 to TEMP2, TEMP2 to TEMP3

Commit message: rounded corners and added rpp bypass
Parts:
- TEMP1, TEMP2, TEMP3: footprint Connector_Molex:Molex_Nano-Fit_105309-xx02_1x02_P2.50mm_Vertical -> UTSVT_Connectors:Molex_Nano-Fit_105309-xx02_1x02_P2.50mm_Vertical
Other:
- moved on the sheet: T_OUT1
Changed lines of the file:
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@@
 	(wire
 		(pts
-			(xy 34.29 54.61) (xy 34.29 62.23)
+			(xy 34.29 49.53) (xy 34.29 62.23)
 		)
 		(stroke
@@
 	(wire
 		(pts
-			(xy 31.75 54.61) (xy 34.29 54.61)
+			(xy 31.75 49.53) (xy 34.29 49.53)
 		)
 		(stroke
@@
 	)
 	(symbol
+		(lib_id "Connector_Generic:Conn_01x02")
+		(at 128.27 62.23 0)
+		(mirror y)
+		(unit 1)
+		(exclude_from_sim no)
+		(in_bom yes)
+		(on_board yes)
+		(dnp no)
+		(property "Reference" "TEMP2"
+			(at 128.27 71.12 0)
+			(effects
+				(font
+					(size 1.27 1.27)
+				)
+			)
+		)
+		(property "Value" "Conn_01x02"
+			(at 128.27 68.58 0)
+			(effects
+				(font
+					(size 1.27 1.27)
+				)
+			)
+		)
+		(property "Footprint" "UTSVT_Connectors:Molex_Nano-Fit_105309-xx02_1x02_P2.50mm_Vertical"
+			(at 128.27 62.23 0)
+			(effects
+				(font
+					(size 1.27 1.27)
+				)
+				(hide yes)
+			)
+		)
+		(property "Datasheet" "~"
+			(at 128.27 62.23 0)
+			(effects
+				(font
+					(size 1.27 1.27)
+				)
+				(hide yes)
+			)
+		)
+		(property "Description" "Generic connector, single row, 01x02, script generated (kicad-library-utils/schlib/autogen/connector/)"
+			(at 128.27 62.23 0)
+			(effects
+				(font
+					(size 1.27 1.27)
+				)
+				(hide yes)
+			)
+		)
+		(pin "2"
+		)
+		(pin "1"
+		)
+		(instances
+			(project "PTN-PumpControlBoard"
+				(path "/591f46f8-eb1d-42dc-a4cb-8182eac4ef58/0e5255e2-25aa-4e9a-a6ff-997dc3e398fd"
+					(reference "TEMP2")
+					(unit 1)
+				)
+			)
+		)
+	)
+	(symbol
 		(lib_id "Device:C_Small")
 		(at 181.61 127 0)
@@
 	)
 	(symbol
+		(lib_id "Connector_Generic:Conn_01x02")
+		(at 26.67 121.92 0)
+		(mirror y)
+		(unit 1)
+		(exclude_from_sim no)
+		(in_bom yes)
+		(on_board yes)
+		(dnp no)
+		(property "Reference" "TEMP3"
+			(at 26.67 130.81 0)
+			(effects
+				(font
+					(size 1.27 1.27)
+				)
+			)
+		)
+		(property "Value" "Conn_01x02"
+			(at 26.67 128.27 0)
+			(effects
+				(font
+					(size 1.27 1.27)
+				)
+			)
+		)
+		(property "Footprint" "UTSVT_Connectors:Molex_Nano-Fit_105309-xx02_1x02_P2.50mm_Vertical"
+			(at 26.67 121.92 0)
+			(effects
+				(font
+					(size 1.27 1.27)
+				)
+				(hide yes)
+			)
+		)
+		(property "Datasheet" "~"
+			(at 26.67 121.92 0)
+			(effects
+				(font
+					(size 1.27 1.27)
+				)
+				(hide yes)
+			)
+		)
+		(property "Description" "Generic connector, single row, 01x02, script generated (kicad-library-utils/schlib/autogen/connector/)"
+			(at 26.67 121.92 0)
+			(effects
+				(font
+					(size 1.27 1.27)
+				)
+				(hide yes)
+			)
+		)
+		(pin "2"
+		)
+		(pin "1"
+		)
+		(instances
+			(project "PTN-PumpControlBoard"
+				(path "/591f46f8-eb1d-42dc-a4cb-8182eac4ef58/0e5255e2-25aa-4e9a-a6ff-997dc3e398fd"
+					(reference "TEMP3")
+					(unit 1)
+				)
+			)
+		)
+	)
+	(symbol
 		(lib_id "Device:R_US")
 		(at 46.99 54.61 90)
@@
 	(symbol
 		(lib_id "Connector:TestPoint")
-		(at 31.75 54.61 90)
+		(at 31.75 49.53 90)
 		(unit 1)
 		(exclude_from_sim no)
@@
 		(fields_autoplaced yes)
 		(property "Reference" "T_OUT1"
-			(at 28.448 49.53 90)
+			(at 28.448 44.45 90)
 			(effects
 				(font
@@
 		)
 		(property "Value" "Pad_TP"
-			(at 28.448 52.07 90)
+			(at 28.448 46.99 90)
 			(effects
 				(font
@@
 		)
 		(property "Footprint" "UTSVT_Special:TestPoint_HEX_3mmID"
-			(at 31.75 49.53 0)
+			(at 31.75 44.45 0)
 			(effects
 				(font
@@
 		)
 		(property "Datasheet" "~"
-			(at 31.75 49.53 0)
+			(at 31.75 44.45 0)
 			(effects
 				(font
@@
 		)
 		(property "Description" "test point"
-			(at 31.75 54.61 0)
+			(at 31.75 49.53 0)
 			(effects
 				(font
@@
 	)
 	(symbol
-		(lib_id "Connector_Generic:Conn_01x02")
-		(at 26.67 121.92 0)
-		(mirror y)
-		(unit 1)
-		(exclude_from_sim no)
-		(in_bom yes)
-		(on_board yes)
-		(dnp no)
-		(property "Reference" "TEMP3"
-			(at 26.67 130.81 0)
-			(effects
-				(font
-					(size 1.27 1.27)
-				)
-			)
-		)
-		(property "Value" "Conn_01x02"
-			(at 26.67 128.27 0)
-			(effects
-				(font
-					(size 1.27 1.27)
-				)
-			)
-		)
-		(property "Footprint" "Connector_Molex:Molex_Nano-Fit_105309-xx02_1x02_P2.50mm_Vertical"
-			(at 26.67 121.92 0)
-			(effects
-				(font
-					(size 1.27 1.27)
-				)
-				(hide yes)
-			)
-		)
-		(property "Datasheet" "https://koolance.com/files/products/manuals/Koolance_sen-ap008g_specifications.pdf"
-			(at 26.67 121.92 0)
-			(effects
-				(font
-					(size 1.27 1.27)
-				)
-				(hide yes)
-			)
-		)
-		(property "Description" "Generic connector, single row, 01x02, script generated (kicad-library-utils/schlib/autogen/connector/)"
-			(at 26.67 121.92 0)
-			(effects
-				(font
-					(size 1.27 1.27)
-				)
-				(hide yes)
-			)
-		)
-		(pin "1"
-		)
-		(pin "2"
-		)
-		(instances
-			(project "PTN-PumpControlBoard"
-				(path "/591f46f8-eb1d-42dc-a4cb-8182eac4ef58/0e5255e2-25aa-4e9a-a6ff-997dc3e398fd"
-					(reference "TEMP3")
-					(unit 1)
-				)
-			)
-		)
-	)
-	(symbol
 		(lib_id "Device:C_Small")
 		(at 231.14 71.12 0)
@@
 	)
 	(symbol
-		(lib_id "Connector_Generic:Conn_01x02")
-		(at 26.67 62.23 0)
-		(mirror y)
-		(unit 1)
-		(exclude_from_sim no)
-		(in_bom yes)
-		(on_board yes)
-		(dnp no)
-		(property "Reference" "TEMP1"
-			(at 26.67 71.12 0)
-			(effects
-				(font
-					(size 1.27 1.27)
-				)
-			)
-		)
-		(property "Value" "Conn_01x02"
-			(at 26.67 68.58 0)
-			(effects
-				(font
-					(size 1.27 1.27)
-				)
-			)
-		)
-		(property "Footprint" "Connector_Molex:Molex_Nano-Fit_105309-xx02_1x02_P2.50mm_Vertical"
-			(at 26.67 62.23 0)
-			(effects
-				(font
-					(size 1.27 1.27)
-				)
-				(hide yes)
-			)
-		)
-		(property "Datasheet" "https://koolance.com/files/products/manuals/Koolance_sen-ap008g_specifications.pdf"
-			(at 26.67 62.23 0)
-			(effects
-				(font
-					(size 1.27 1.27)
-				)
-				(hide yes)
-			)
-		)
-		(property "Description" "Generic connector, single row, 01x02, script generated (kicad-library-utils/schlib/autogen/connector/)"
-			(at 26.67 62.23 0)
-			(effects
-				(font
-					(size 1.27 1.27)
-				)
-				(hide yes)
-			)
-		)
-		(pin "1"
-		)
-		(pin "2"
-		)
-		(instances
-			(project "PTN-PumpControlBoard"
-				(path "/591f46f8-eb1d-42dc-a4cb-8182eac4ef58/0e5255e2-25aa-4e9a-a6ff-997dc3e398fd"
-					(reference "TEMP1")
-					(unit 1)
-				)
-			)
-		)
-	)
-	(symbol
 		(lib_id "Device:C_Small")
 		(at 198.12 105.41 0)
@@
 	)
 	(symbol
-		(lib_id "Connector_Generic:Conn_01x02")
-		(at 128.27 62.23 0)
-		(mirror y)
-		(unit 1)
-		(exclude_from_sim no)
-		(in_bom yes)
-		(on_board yes)
-		(dnp no)
-		(property "Reference" "TEMP2"
-			(at 128.27 71.12 0)
-			(effects
-				(font
-					(size 1.27 1.27)
-				)
-			)
-		)
-		(property "Value" "Conn_01x02"
-			(at 128.27 68.58 0)
-			(effects
-				(font
-					(size 1.27 1.27)
-				)
-			)
-		)
-		(property "Footprint" "Connector_Molex:Molex_Nano-Fit_105309-xx02_1x02_P2.50mm_Vertical"
-			(at 128.27 62.23 0)
-			(effects
-				(font
-					(size 1.27 1.27)
-				)
-				(hide yes)
-			)
-		)
-		(property "Datasheet" "https://koolance.com/files/products/manuals/Koolance_sen-ap008g_specifications.pdf"
-			(at 128.27 62.23 0)
-			(effects
-				(font
-					(size 1.27 1.27)
-				)
-				(hide yes)
-			)
-		)
-		(property "Description" "Generic connector, single row, 01x02, script generated (kicad-library-utils/schlib/autogen/connector/)"
-			(at 128.27 62.23 0)
-			(effects
-				(font
-					(size 1.27 1.27)
-				)
-				(hide yes)
-			)
-		)
-		(pin "1"
-		)
-		(pin "2"
-		)
-		(instances
-			(project "PTN-PumpControlBoard"
-				(path "/591f46f8-eb1d-42dc-a4cb-8182eac4ef58/0e5255e2-25aa-4e9a-a6ff-997dc3e398fd"
-					(reference "TEMP2")
-					(unit 1)
-				)
-			)
-		)
-	)
-	(symbol
 		(lib_name "OP249GS_1")
 		(lib_id "Amplifier_Operational:OP249GS")
@@
 				)
 			)
+		)
+	)
+	(symbol
+		(lib_id "Connector_Generic:Conn_01x02")
+		(at 26.67 62.23 0)
+		(mirror y)
+		(unit 1)
+		(exclude_from_sim no)
+		(in_bom yes)
+		(on_board yes)
+		(dnp no)
+		(property "Reference" "TEMP1"
+			(at 26.67 71.12 0)
+			(effects
+				(font
+					(size 1.27 1.27)
+				)
+			)
+		)
+		(property "Value" "Conn_01x02"
+			(at 26.67 68.58 0)
+			(effects
+				(font
+					(size 1.27 1.27)
+				)
+			)
+		)
+		(property "Footprint" "UTSVT_Connectors:Molex_Nano-Fit_105309-xx02_1x02_P2.50mm_Vertical"
+			(at 26.67 62.23 0)
+			(effects
+				(font
+					(size 1.27 1.27)
+				)
+				(hide yes)
+			)
+		)
+		(property "Datasheet" "~"
+			(at 26.67 62.23 0)
+			(effects
+				(font
+					(size 1.27 1.27)
+				)
+				(hide yes)
+			)
+		)
+		(property "Description" "Generic connector, single row, 01x02, script generated (kicad-library-utils/schlib/autogen/connector/)"
+			(at 26.67 62.23 0)
+			(effects
+				(font
+					(size 1.27 1.27)
+				)
+				(hide yes)
+			)
+		)
+		(pin "2"
+		)
+		(pin "1"
+		)
+		(instances
+			(project "PTN-PumpControlBoard"
+				(path "/591f46f8-eb1d-42dc-a4cb-8182eac4ef58/0e5255e2-25aa-4e9a-a6ff-997dc3e398fd"
+					(reference "TEMP1")
+					(unit 1)
+				)
+			)
