File: TempSensors.kicad_sch (KiCad schematic)
At the start: 34 parts, among them IC1 TLV9002QDRQ1, IC2 TLV9002QDRQ1, U3 TLV9002QDRQ1, U4 TLV9002QDRQ1

Commit message: initial schem changes
Parts:
- removed C10: 15uF, Capacitor_SMD:C_0805_2012Metric, symbol Device:C_Small
- removed C11, C12: .1uF, Capacitor_SMD:C_0805_2012Metric, symbol Device:C_Small
- removed C9: 1uF, Capacitor_SMD:C_0805_2012Metric, symbol Device:C_Small
- removed IC1, IC2: TLV9002QDRQ1, OpAmp:SOIC127P600X175-8N, symbol OpAmp:TLV9002QDRQ1
- removed R22: 10k, Resistor_SMD:R_0603_1608Metric, symbol Device:R_US
- removed R23: 15k, Resistor_SMD:R_0603_1608Metric, symbol Device:R_US
- removed R24, R26: 0, Resistor_SMD:R_0603_1608Metric, symbol Device:R_US
- removed R25: 1k, Resistor_SMD:R_0603_1608Metric, symbol Device:R_US
- removed TEMP1, TEMP2, TEMP3: Conn_01x02, UTSVT_Connectors:Molex_Nano-Fit_105309-xx02_1x02_P2.50mm_Vertical, symbol Connector_Generic:Conn_01x02
- removed T_OUT1, T_TP1: Pad_TP, UTSVT_Special:TestPoint_HEX_3mmID, symbol Connector:TestPoint
- removed U4: TLV9002QDRQ1, OpAmp:SOIC127P600X175-8N, symbol Amplifier_Operational:OP249GS
- U3: footprint OpAmp:SOIC127P600X175-8N -> Package_SO:SOIC-8_3.9x4.9mm_P1.27mm
Connections:
- net Temp2+: now reaches R17.2, R18.1
- net Temp1+: now reaches R12.2, R13.1
- no-connect marks 6 -> 0
Other:
- note removed: "op amp has no associated footprint, only for schematic readability"
- note removed: "symbols that have the actual footprints"
