File: Fans.kicad_sch (KiCad schematic)
At the start: 12 parts, among them Q1 NMOS, Q2 NMOS

Commit message: Initial layout with 1 pump, 2 temp, 1 flow all on front side
Parts:
- Q1, Q2: footprint Package_TO_SOT_SMD:LFPAK33 -> Package_TO_SOT_SMD:SOT-23
Changed lines of the file:
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@@
+	)
+	(symbol
+		(lib_id "power:GND")
+		(at 114.3 63.5 0)
+		(unit 1)
+		(exclude_from_sim no)
+		(in_bom yes)
+		(on_board yes)
+		(dnp no)
+		(fields_autoplaced yes)
+		(property "Reference" "#PWR016"
+			(at 114.3 69.85 0)
+			(effects
+				(font
+					(size 1.27 1.27)
+				)
+				(hide yes)
+			)
+		)
+		(property "Value" "GND"
+			(at 114.3 68.58 0)
+			(effects
+				(font
+					(size 1.27 1.27)
+				)
+			)
+		)
+		(property "Footprint" ""
+			(at 114.3 63.5 0)
+			(effects
+				(font
+					(size 1.27 1.27)
+				)
+				(hide yes)
+			)
+		)
+		(property "Datasheet" ""
+			(at 114.3 63.5 0)
+			(effects
+				(font
+					(size 1.27 1.27)
+				)
+				(hide yes)
+			)
+		)
+		(property "Description" "Power symbol creates a global label with name \"GND\" , ground"
+			(at 114.3 63.5 0)
+			(effects
+				(font
+					(size 1.27 1.27)
+				)
+				(hide yes)
+			)
+		)
+		(pin "1"
+		)
+		(instances
+			(project "PTN-PumpControlBoard"
+				(path "/591f46f8-eb1d-42dc-a4cb-8182eac4ef58/d90f7da4-ca39-48c6-8d97-b8d1e37c7dd0"
+					(reference "#PWR016")
+					(unit 1)
+				)
+			)
+		)
+	)
+	(symbol
+		(lib_id "Device:R_US")
+		(at 113.03 114.3 0)
+		(unit 1)
+		(exclude_from_sim no)
+		(in_bom yes)
+		(on_board yes)
+		(dnp no)
+		(property "Reference" "R8"
+			(at 115.57 113.0299 0)
+			(effects
+				(font
+					(size 1.27 1.27)
+				)
+				(justify left)
+			)
+		)
+		(property "Value" "1k"
+			(at 115.57 115.5699 0)
+			(effects
+				(font
+					(size 1.27 1.27)
+				)
+				(justify left)
+			)
+		)
+		(property "Footprint" "Resistor_SMD:R_0805_2012Metric"
+			(at 114.046 114.554 90)
+			(effects
+				(font
+					(size 1.27 1.27)
+				)
+				(hide yes)
+			)
+		)
+		(property "Datasheet" "~"
+			(at 113.03 114.3 0)
+			(effects
+				(font
+					(size 1.27 1.27)
+				)
+				(hide yes)
+			)
+		)
+		(property "Description" "Resistor, US symbol"
+			(at 113.03 114.3 0)
+			(effects
+				(font
+					(size 1.27 1.27)
+				)
+				(hide yes)
+			)
+		)
+		(pin "1"
+		)
+		(pin "2"
+		)
+		(instances
+			(project "PTN-PumpControlBoard"
+				(path "/591f46f8-eb1d-42dc-a4cb-8182eac4ef58/d90f7da4-ca39-48c6-8d97-b8d1e37c7dd0"
+					(reference "R8")
+					(unit 1)
+				)
+			)
+		)
+	)
+	(symbol
+		(lib_id "Device:D")
+		(at 52.07 38.1 270)
+		(unit 1)
+		(exclude_from_sim no)
+		(in_bom yes)
+		(on_board yes)
+		(dnp no)
+		(fields_autoplaced yes)
+		(property "Reference" "D1"
+			(at 54.61 36.8299 90)
+			(effects
+				(font
+					(size 1.27 1.27)
+				)
+				(justify left)
+			)
+		)
+		(property "Value" "1N4448W"
+			(at 54.61 39.3699 90)
+			(effects
+				(font
+					(size 1.27 1.27)
+				)
+				(justify left)
+			)
+		)
+		(property "Footprint" "Diode_SMD:D_SOD-323"
+			(at 52.07 38.1 0)
+			(effects
+				(font
+					(size 1.27 1.27)
+				)
+				(hide yes)
+			)
+		)
+		(property "Datasheet" "https://www.vishay.com/docs/85722/1n4448w.pdf"
+			(at 52.07 38.1 0)
+			(effects
+				(font
+					(size 1.27 1.27)
+				)
+				(hide yes)
+			)
+		)
+		(property "Description" "Diode"
+			(at 52.07 38.1 0)
+			(effects
+				(font
+					(size 1.27 1.27)
+				)
+				(hide yes)
+			)
+		)
+		(property "Sim.Device" "D"
+			(at 52.07 38.1 0)
+			(effects
+				(font
+					(size 1.27 1.27)
+				)
+				(hide yes)
+			)
+		)
+		(property "Sim.Pins" "1=K 2=A"
+			(at 52.07 38.1 0)
+			(effects
+				(font
+					(size 1.27 1.27)
+				)
+				(hide yes)
+			)
+		)
+		(pin "1"
+		)
+		(pin "2"
+		)
+		(instances
+			(project "PTN-PumpControlBoard"
+				(path "/591f46f8-eb1d-42dc-a4cb-8182eac4ef58/d90f7da4-ca39-48c6-8d97-b8d1e37c7dd0"
+					(reference "D1")
+					(unit 1)
+				)
+			)
+		)
 	)
 	(symbol
@@
 			)
 		)
-		(property "Footprint" "Package_TO_SOT_SMD:LFPAK33"
+		(property "Footprint" "Package_TO_SOT_SMD:SOT-23"
 			(at 66.04 50.8 0)
 			(effects
@@
 	)
 	(symbol
-		(lib_id "power:GND")
-		(at 114.3 63.5 0)
-		(unit 1)
-		(exclude_from_sim no)
-		(in_bom yes)
-		(on_board yes)
-		(dnp no)
-		(fields_autoplaced yes)
-		(property "Reference" "#PWR016"
-			(at 114.3 69.85 0)
-			(effects
-				(font
-					(size 1.27 1.27)
-				)
-				(hide yes)
-			)
-		)
-		(property "Value" "GND"
-			(at 114.3 68.58 0)
-			(effects
-				(font
-					(size 1.27 1.27)
-				)
-			)
-		)
-		(property "Footprint" ""
-			(at 114.3 63.5 0)
-			(effects
-				(font
-					(size 1.27 1.27)
-				)
-				(hide yes)
-			)
-		)
-		(property "Datasheet" ""
-			(at 114.3 63.5 0)
-			(effects
-				(font
-					(size 1.27 1.27)
-				)
-				(hide yes)
-			)
-		)
-		(property "Description" "Power symbol creates a global label with name \"GND\" , ground"
-			(at 114.3 63.5 0)
-			(effects
-				(font
-					(size 1.27 1.27)
-				)
-				(hide yes)
-			)
-		)
-		(pin "1"
-		)
-		(instances
-			(project "PTN-PumpControlBoard"
-				(path "/591f46f8-eb1d-42dc-a4cb-8182eac4ef58/d90f7da4-ca39-48c6-8d97-b8d1e37c7dd0"
-					(reference "#PWR016")
-					(unit 1)
-				)
-			)
-		)
-	)
-	(symbol
-		(lib_id "Device:R_US")
-		(at 113.03 114.3 0)
-		(unit 1)
-		(exclude_from_sim no)
-		(in_bom yes)
-		(on_board yes)
-		(dnp no)
-		(property "Reference" "R8"
-			(at 115.57 113.0299 0)
-			(effects
-				(font
-					(size 1.27 1.27)
-				)
-				(justify left)
-			)
-		)
-		(property "Value" "1k"
-			(at 115.57 115.5699 0)
-			(effects
-				(font
-					(size 1.27 1.27)
-				)
-				(justify left)
-			)
-		)
-		(property "Footprint" "Resistor_SMD:R_0805_2012Metric"
-			(at 114.046 114.554 90)
-			(effects
-				(font
-					(size 1.27 1.27)
-				)
-				(hide yes)
-			)
-		)
-		(property "Datasheet" "~"
-			(at 113.03 114.3 0)
-			(effects
-				(font
-					(size 1.27 1.27)
-				)
-				(hide yes)
-			)
-		)
-		(property "Description" "Resistor, US symbol"
-			(at 113.03 114.3 0)
-			(effects
-				(font
-					(size 1.27 1.27)
-				)
-				(hide yes)
-			)
-		)
-		(pin "1"
-		)
-		(pin "2"
-		)
-		(instances
-			(project "PTN-PumpControlBoard"
-				(path "/591f46f8-eb1d-42dc-a4cb-8182eac4ef58/d90f7da4-ca39-48c6-8d97-b8d1e37c7dd0"
-					(reference "R8")
-					(unit 1)
-				)
-			)
-		)
-	)
-	(symbol
-		(lib_id "Device:D")
-		(at 52.07 38.1 270)
-		(unit 1)
-		(exclude_from_sim no)
-		(in_bom yes)
-		(on_board yes)
-		(dnp no)
-		(fields_autoplaced yes)
-		(property "Reference" "D1"
-			(at 54.61 36.8299 90)
-			(effects
-				(font
-					(size 1.27 1.27)
-				)
-				(justify left)
-			)
-		)
-		(property "Value" "1N4448W"
-			(at 54.61 39.3699 90)
-			(effects
-				(font
-					(size 1.27 1.27)
-				)
-				(justify left)
-			)
-		)
-		(property "Footprint" "Diode_SMD:D_SOD-323"
-			(at 52.07 38.1 0)
-			(effects
-				(font
-					(size 1.27 1.27)
-				)
-				(hide yes)
-			)
-		)
-		(property "Datasheet" "https://www.vishay.com/docs/85722/1n4448w.pdf"
-			(at 52.07 38.1 0)
-			(effects
-				(font
-					(size 1.27 1.27)
-				)
-				(hide yes)
-			)
-		)
-		(property "Description" "Diode"
-			(at 52.07 38.1 0)
-			(effects
-				(font
-					(size 1.27 1.27)
-				)
-				(hide yes)
-			)
-		)
-		(property "Sim.Device" "D"
-			(at 52.07 38.1 0)
-			(effects
-				(font
-					(size 1.27 1.27)
-				)
-				(hide yes)
-			)
-		)
-		(property "Sim.Pins" "1=K 2=A"
-			(at 52.07 38.1 0)
-			(effects
-				(font
-					(size 1.27 1.27)
-				)
-				(hide yes)
-			)
-		)
-		(pin "1"
-		)
-		(pin "2"
-		)
-		(instances
-			(project "PTN-PumpControlBoard"
-				(path "/591f46f8-eb1d-42dc-a4cb-8182eac4ef58/d90f7da4-ca39-48c6-8d97-b8d1e37c7dd0"
-					(reference "D1")
-					(unit 1)
-				)
-			)
-		)
-	)
-	(symbol
 		(lib_id "Connector_Generic:Conn_01x03")
 		(at 78.74 38.1 0)
@@
 			)
 		)
-		(property "Footprint" "Package_TO_SOT_SMD:LFPAK33"
+		(property "Footprint" "Package_TO_SOT_SMD:SOT-23"
 			(at 64.77 120.65 0)
 			(effects

Commit message: schematic with 12V components, unigain buffers & extra temp sensor
Parts:
- removed Q1, Q2: NMOS, Package_TO_SOT_SMD:SOT-23, symbol Simulation_SPICE:NMOS
- added Q3, Q4: IRLML0030, Package_TO_SOT_SMD:SOT-23, symbol Transistor_FET:IRLML0030
- FAN1, FAN2: footprint UTSVT_Connectors:Molex_MicroFit3.0_1x3xP3.00mm_PolarizingPeg_Vertical -> Connector_Molex:Molex_Nano-Fit_105309-xx03_1x03_P2.50mm_Vertical
Connections:
- net GND: now also Q3.2 (S), Q4.2 (S)
- net PWM1: now also Q3.1 (G)
- net PWM2: now also Q4.1 (G)
- net at D1.2 (A), FAN1.3 (Pin_3): now also Q3.3 (D)
- net at D2.2 (A), FAN2.3 (Pin_3): now also Q4.3 (D)
- net TACH1_IN renamed TACH1_12V
- net TACH1_OUT renamed TACH1
- net TACH2_IN renamed TACH2_12V
- net TACH2_OUT renamed TACH2
Other:
- moved on the sheet: D1, D2, FAN1, FAN2, R10, R5, R6, R7, R8, R9

Commit message: repicked parts to be 24V tolerant and changed corresponding circuitry
Parts:
- removed D1, D2: 1N4448W, Diode_SMD:D_SOD-323, symbol Device:D
- removed FAN1, FAN2: Conn_01x03, Connector_Molex:Molex_Nano-Fit_105309-xx03_1x03_P2.50mm_Vertical, symbol Connector_Generic:Conn_01x03
- removed Q3, Q4: IRLML0030, Package_TO_SOT_SMD:SOT-23, symbol Transistor_FET:IRLML0030
- removed R10, R7: 10k, Resistor_SMD:R_0805_2012Metric, symbol Device:R_US
- removed R8: 1k, Resistor_SMD:R_0805_2012Metric, symbol Device:R_US
- removed R9: 380, Resistor_SMD:R_0805_2012Metric, symbol Device:R_US
- added D2, D3: VSSAF522-M3/H, UTSVT_Passive:DO-221AC, symbol Diode:C3D25170H
- added FAN1, FAN2: Conn_01x04, Connector_Molex:Molex_Nano-Fit_105309-xx04_1x04_P2.50mm_Vertical, symbol Connector_Generic:Conn_01x04
- R6: value 380 -> 1k
Connections:
- net GND: now also D2.2 (A), D3.2 (A), FAN1.4 (Pin_4), FAN2.4 (Pin_4); no longer R6.2
- net PWM1: now also FAN1.3 (Pin_3)
- net PWM2: now also FAN2.3 (Pin_3)
- net TACH1: now also FAN1.2 (Pin_2); no longer R6.1
- net TACH2: now also R6.2, FAN2.2 (Pin_2)
- net TACH1_12V renamed +3.3V
- net +3.3V: now also R6.1
- new net +24V: D2.1 (K), D3.1 (K), FAN1.1 (Pin_1), FAN2.1 (Pin_1)

Commit message: reworked layout with 24V components but no testpoints & headers
Parts:
- removed D2, D3: VSSAF522-M3/H, UTSVT_Passive:DO-221AC, symbol Diode:C3D25170H
Changed lines of the file:
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@@
 		)
 	)
-	(text_box "datasheet stipulates 3 pin fan with TACH or PWM so I've added circutry for both, I just won't use one pin"
+	(text_box "- datasheet stipulates 3 pin fan with TACH or PWM so I've added circutry for both, I just won't use one pin\n- do I need a flyback diode if I'm not controlling pwm manually with a fet?"
 		(exclude_from_sim no)
 		(at 234.95 19.05 0)
-		(size 30.48 10.16)
+		(size 30.48 16.51)
 		(margins 0.9525 0.9525 0.9525 0.9525)
 		(stroke
@@
 	)
 	(junction
-		(at 49.53 38.1)
-		(diameter 0)
-		(color 0 0 0 0)
-	)
-	(junction
-		(at 157.48 53.34)
-		(diameter 0)
-		(color 0 0 0 0)
-	)
-	(junction
-		(at 157.48 38.1)
-		(diameter 0)
-		(color 0 0 0 0)
-	)
-	(junction
-		(at 49.53 53.34)
-		(diameter 0)
-		(color 0 0 0 0)
-	)
-	(junction
 		(at 97.79 53.34)
 		(diameter 0)
@@
 	(wire
 		(pts
-			(xy 148.59 49.53) (xy 148.59 53.34)
-		)
-		(stroke
-			(width 0)
-			(type default)
-		)
-	)
-	(wire
-		(pts
-			(xy 49.53 38.1) (xy 40.64 38.1)
-		)
-		(stroke
-			(width 0)
-			(type default)
-		)
-	)
-	(wire
-		(pts
 			(xy 49.53 53.34) (xy 49.53 59.69)
 		)
@@
 	(wire
 		(pts
-			(xy 40.64 38.1) (xy 40.64 41.91)
-		)
-		(stroke
-			(width 0)
-			(type default)
-		)
-	)
-	(wire
-		(pts
 			(xy 97.79 40.64) (xy 97.79 43.18)
 		)
@@
 	(wire
 		(pts
-			(xy 40.64 53.34) (xy 49.53 53.34)
-		)
-		(stroke
-			(width 0)
-			(type default)
-		)
-	)
-	(wire
-		(pts
 			(xy 157.48 53.34) (xy 166.37 53.34)
 		)
@@
 	(wire
 		(pts
-			(xy 148.59 38.1) (xy 148.59 41.91)
-		)
-		(stroke
-			(width 0)
-			(type default)
-		)
-	)
-	(wire
-		(pts
 			(xy 93.98 53.34) (xy 97.79 53.34)
 		)
@@
 	(wire
 		(pts
-			(xy 40.64 49.53) (xy 40.64 53.34)
-		)
-		(stroke
-			(width 0)
-			(type default)
-		)
-	)
-	(wire
-		(pts
 			(xy 205.74 50.8) (xy 205.74 53.34)
 		)
@@
 	(wire
 		(pts
-			(xy 148.59 53.34) (xy 157.48 53.34)
-		)
-		(stroke
-			(width 0)
-			(type default)
-		)
-	)
-	(wire
-		(pts
 			(xy 166.37 41.91) (xy 167.64 41.91)
 		)
@@
 		(pts
 			(xy 205.74 40.64) (xy 205.74 43.18)
-		)
-		(stroke
-			(width 0)
-			(type default)
-		)
-	)
-	(wire
-		(pts
-			(xy 157.48 38.1) (xy 148.59 38.1)
 		)
 		(stroke
@@
 					(unit 1)
 				)
-			)
-		)
-	)
-	(symbol
-		(lib_id "Diode:C3D25170H")
-		(at 148.59 45.72 270)
-		(unit 1)
-		(exclude_from_sim no)
-		(in_bom yes)
-		(on_board yes)
-		(dnp no)
-		(property "Reference" "D3"
-			(at 151.13 43.18 90)
-			(effects
-				(font
-					(size 1.27 1.27)
-				)
-				(justify left)
-			)
-		)
-		(property "Value" "VSSAF522-M3/H"
-			(at 131.064 43.688 90)
-			(effects
-				(font
-					(size 1.27 1.27)
-				)
-				(justify left)
-			)
-		)
-		(property "Footprint" "UTSVT_Passive:DO-221AC"
-			(at 144.145 45.72 0)
-			(effects
-				(font
-					(size 1.27 1.27)
-				)
-				(hide yes)
-			)
-		)
-		(property "Datasheet" "https://www.mouser.com/ProductDetail/Vishay-General-Semiconductor/VSSAF522-M3-H?qs=UkDUCjYnTB00gpgD%2Fb%2Fw%252BA%3D%3D"
-			(at 148.59 45.72 0)
-			(effects
-				(font
-					(size 1.27 1.27)
-				)
-				(hide yes)
-			)
-		)
-		(property "Description" ""
-			(at 148.59 45.72 0)
-			(effects
-				(font
-					(size 1.27 1.27)
-				)
-				(hide yes)
-			)
-		)
-		(pin "1"
-		)
-		(pin "2"
-		)
-		(instances
-			(project "PTN-PumpControlBoard"
-				(path "/591f46f8-eb1d-42dc-a4cb-8182eac4ef58/d90f7da4-ca39-48c6-8d97-b8d1e37c7dd0"
-					(reference "D3")
-					(unit 1)
-				)
-			)
-		)
-	)
-	(symbol
-		(lib_id "Diode:C3D25170H")
-		(at 40.64 45.72 270)
-		(unit 1)
-		(exclude_from_sim no)
-		(in_bom yes)
-		(on_board yes)
-		(dnp no)
-		(property "Reference" "D2"
-			(at 43.18 43.18 90)
-			(effects
-				(font
-					(size 1.27 1.27)
-				)
-				(justify left)
-			)
-		)
-		(property "Value" "VSSAF522-M3/H"
-			(at 23.114 43.688 90)
-			(effects
-				(font
-					(size 1.27 1.27)
-				)
-				(justify left)
-			)
-		)
-		(property "Footprint" "UTSVT_Passive:DO-221AC"
-			(at 36.195 45.72 0)
-			(effects
-				(font
-					(size 1.27 1.27)
-				)
-				(hide yes)
-			)
-		)
-		(property "Datasheet" "https://www.mouser.com/ProductDetail/Vishay-General-Semiconductor/VSSAF522-M3-H?qs=UkDUCjYnTB00gpgD%2Fb%2Fw%252BA%3D%3D"
-			(at 40.64 45.72 0)
-			(effects
-				(font
-					(size 1.27 1.27)
-				)
-				(hide yes)
-			)
-		)
-		(property "Description" ""
-			(at 40.64 45.72 0)
-			(effects
-				(font
-					(size 1.27 1.27)
-				)
-				(hide yes)
-			)
-		)
-		(pin "1"
-		)
-		(pin "2"
-		)
-		(instances
-			(project "PTN-PumpControlBoard"
-				(path "/591f46f8-eb1d-42dc-a4cb-8182eac4ef58/d90f7da4-ca39-48c6-8d97-b8d1e37c7dd0"
-					(reference "D2")
-					(unit 1)
-				)

Commit message: added test points and headers, AGND and 12V not fully connected
Parts:
- added F_PWM1, F_TACH1, F_TACH2, GND1: Scope_TP, TestPoint:TestPoint_Keystone_5010-5014_Multipurpose, symbol Connector:TestPoint
- added F_PWM2: Scope_T1, TestPoint:TestPoint_Keystone_5010-5014_Multipurpose, symbol Connector:TestPoint
Connections:
- net GND: now also GND1.1
- net PWM1: now also F_PWM1.1
- net PWM2: now also F_PWM2.1
- net TACH1: now also F_TACH1.1
- net TACH2: now also F_TACH2.1
Other:
- moved on the sheet: R5, R6

Commit message: Fixed fan schematic based on review feedback
Parts:
- removed F_PWM1, F_TACH1, F_TACH2, GND1: Scope_TP, TestPoint:TestPoint_Keystone_5010-5014_Multipurpose, symbol Connector:TestPoint
- removed F_PWM2: Scope_T1, TestPoint:TestPoint_Keystone_5010-5014_Multipurpose, symbol Connector:TestPoint
- added C1, C2: 1uF, Capacitor_SMD:C_0805_2012Metric, symbol Device:C_Small
- added D1: VSSAF522-M3/H, UTSVT_Passive:DO-221AC, symbol Diode:C3D25170H
- added R18, R19, R20, R21, R22: 10k, Resistor_SMD:R_0805_2012Metric, symbol Device:R_US
- added R23, R24: 33k, Resistor_SMD:R_0805_2012Metric, symbol Device:R_US
- added U2: EMC2305-1-AP-TR, FanControl:QFN16_4x4MC_MCH, symbol 2024-11-02_21-04-42:EMC2305-1-AP-TR
- FAN1, FAN2: Notes Small signal control for pump -> (none)
- R5, R6: value 1k -> 5k
Connections:
- net +24V: now also D1.1 (K)
- net +3.3V: now also C1.1, C2.1, R18.2, R19.2, R20.2, R21.2, R22.2, R23.2, R24.2, U2.3 (VDD)
- net GND: now also C1.2, C2.2, D1.2 (A), U2.HTAB (EPAD)
- net PWM1 renamed FAN1_PWM
- net FAN1_PWM: now also R20.1, U2.5 (PWM1)
- net PWM2 renamed FAN2_PWM
- net FAN2_PWM: now also R22.1, U2.7 (PWM2)
- net TACH1 renamed FAN1_TACH
- net FAN1_TACH: now also U2.6 (TACH1)
- net TACH2 renamed FAN2_TACH
- net FAN2_TACH: now also U2.8 (TACH2)
- new net ADDR_SEL: R23.1, U2.4 (ADDR_SEL)
- new net CLK: R24.1, U2.11 (CLK)
- new net FAN_SCL: R19.1, U2.2 (SMCLK)
- new net FAN_SDA: R18.1, U2.1 (SMDATA)
- new net ~{SMBALERT}: R21.1, U2.12 (*ALERT)
- no-connect marks 0 -> 6
Other:
- note added: "PWM pins configed as open drain"
- moved on the sheet: FAN1, FAN2, R5, R6

Commit message: updated schematic with low pass for temp sensors and new resistor footprint
Parts:
- R18, R19, R20, R21, R22, R23, R24, R5, R6: footprint Resistor_SMD:R_0805_2012Metric -> Resistor_SMD:R_0603_1608Metric

Commit message: low pass for temp & flyback diodes
Parts:
- added D2: VSSAF522-M3/H, UTSVT_Passive:DO-221AC, symbol Diode:C3D25170H
Connections:
- net +24V: now also D2.1 (K)
- net GND: now also D2.2 (A)
