File: Fans.kicad_sch (KiCad schematic)
At the start: 16 parts, among them U2 EMC2305-1-AP-TR

Commit message: fixed all review notes for schematic
Parts:
- removed FAN1, FAN2: Conn_01x04, Connector_Molex:Molex_Nano-Fit_105309-xx04_1x04_P2.50mm_Vertical, symbol Connector_Generic:Conn_01x04
- removed R6: 5k, Resistor_SMD:R_0603_1608Metric, symbol Device:R_US
- added FAN1, FAN2: Conn_01x03, Connector_Molex:Molex_Nano-Fit_105309-xx03_1x03_P2.50mm_Vertical, symbol Connector_Generic:Conn_01x03
- added Q1, Q2: NMOS, UTSVT_Power:BUK7M1780EX, symbol Simulation_SPICE:NMOS
- added R2: 5k, Resistor_SMD:R_0603_1608Metric, symbol Device:R_US
- D7: renamed from D1; footprint UTSVT_Passive:DO-221AC -> UTSVT_Passive:MMDL101T1G
- D8: renamed from D2; footprint UTSVT_Passive:DO-221AC -> UTSVT_Passive:MMDL101T1G
- renumbered R5 to R1, R18 to R3, R23 to R4, R19 to R5, R21 to R6, R24 to R7, R20 to R8, R22 to R9
Connections:
- net +24V: now also D7.2 (A), D8.2 (A), FAN1.1 (Pin_1), FAN2.1 (Pin_1); no longer D7.1 (K), D8.1 (K)
- net +3.3V: now also R2.1
- net FAN1_PWM: now also Q1.2 (G)
- net FAN1_TACH: now also FAN1.2 (Pin_2)
- net FAN2_PWM: now also Q2.2 (G)
- net FAN2_TACH: now also FAN2.2 (Pin_2), R2.2
- net GND: now also D7.1 (K), D8.1 (K), Q1.3 (S), Q2.3 (S); no longer D7.2 (A), D8.2 (A)
- new net: FAN2.3 (Pin_3), Q2.1 (D)
- new net: FAN1.3 (Pin_3), Q1.1 (D)
Other:
- moved on the sheet: C1, C2, D7, D8, R3, R4, R5, R6, R7, R8, R9, U2

Commit message: set up layout
Parts:
- removed Q1, Q2: NMOS, UTSVT_Power:BUK7M1780EX, symbol Simulation_SPICE:NMOS
- added Q1, Q2: BUK7M27-80EX, Package_TO_SOT_SMD:LFPAK33, symbol Transistor_FET:BUK7M27-80EX
Connections:
- net FAN1_PWM: now also Q1.4 (G)
- net FAN2_PWM: now also Q2.4 (G)
- net GND: now also Q1.1 (S), Q1.2 (S), Q1.3 (S), Q2.1 (S), Q2.2 (S), Q2.3 (S)
- net at FAN2.3 (Pin_3): now also Q2.5 (D)
- net at FAN1.3 (Pin_3): now also Q1.5 (D)
Changed lines of the file:
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@@
 	)
 	(symbol
-		(lib_id "Simulation_SPICE:NMOS")
+		(lib_id "Transistor_FET:BUK7M27-80EX")
+		(at 124.46 49.53 0)
+		(unit 1)
+		(exclude_from_sim no)
+		(in_bom yes)
+		(on_board yes)
+		(dnp no)
+		(fields_autoplaced yes)
+		(property "Reference" "Q2"
+			(at 130.81 48.2599 0)
+			(effects
+				(font
+					(size 1.27 1.27)
+				)
+				(justify left)
+			)
+		)
+		(property "Value" "BUK7M27-80EX"
+			(at 130.81 50.7999 0)
+			(effects
+				(font
+					(size 1.27 1.27)
+				)
+				(justify left)
+			)
+		)
+		(property "Footprint" "Package_TO_SOT_SMD:LFPAK33"
+			(at 129.54 51.435 0)
+			(effects
+				(font
+					(size 1.27 1.27)
+					(italic yes)
+				)
+				(justify left)
+				(hide yes)
+			)
+		)
+		(property "Datasheet" "https://assets.nexperia.com/documents/data-sheet/BUK7M27-80E.pdf"
+			(at 129.54 53.34 0)
+			(effects
+				(font
+					(size 1.27 1.27)
+				)
+				(justify left)
+				(hide yes)
+			)
+		)
+		(property "Description" "30A Id, 80V Vds, N-Channel TrenchMOS MOSFET, 27mOhm Ron, 19.5nC Qqd, -55 to 175 °C, LFPAK33"
+			(at 124.46 49.53 0)
+			(effects
+				(font
+					(size 1.27 1.27)
+				)
+				(hide yes)
+			)
+		)
+		(pin "2"
+		)
+		(pin "3"
+		)
+		(pin "1"
+		)
+		(pin "5"
+		)
+		(pin "4"
+		)
+		(instances
+			(project "PTN-PumpControlBoard"
+				(path "/591f46f8-eb1d-42dc-a4cb-8182eac4ef58/d90f7da4-ca39-48c6-8d97-b8d1e37c7dd0"
+					(reference "Q2")
+					(unit 1)
+				)
+			)
+		)
+	)
+	(symbol
+		(lib_id "Diode:C3D25170H")
+		(at 176.53 38.1 90)
+		(unit 1)
+		(exclude_from_sim no)
+		(in_bom yes)
+		(on_board yes)
+		(dnp no)
+		(property "Reference" "D7"
+			(at 173.99 40.64 90)
+			(effects
+				(font
+					(size 1.27 1.27)
+				)
+				(justify left)
+			)
+		)
+		(property "Value" "VSSAF522-M3/H"
+			(at 194.056 40.132 90)
+			(effects
+				(font
+					(size 1.27 1.27)
+				)
+				(justify left)
+			)
+		)
+		(property "Footprint" "UTSVT_Passive:MMDL101T1G"
+			(at 180.975 38.1 0)
+			(effects
+				(font
+					(size 1.27 1.27)
+				)
+				(hide yes)
+			)
+		)
+		(property "Datasheet" "https://www.mouser.com/ProductDetail/Vishay-General-Semiconductor/VSSAF522-M3-H?qs=UkDUCjYnTB00gpgD%2Fb%2Fw%252BA%3D%3D"
+			(at 176.53 38.1 0)
+			(effects
+				(font
+					(size 1.27 1.27)
+				)
+				(hide yes)
+			)
+		)
+		(property "Description" ""
+			(at 176.53 38.1 0)
+			(effects
+				(font
+					(size 1.27 1.27)
+				)
+				(hide yes)
+			)
+		)
+		(pin "1"
+		)
+		(pin "2"
+		)
+		(instances
+			(project "PTN-PumpControlBoard"
+				(path "/591f46f8-eb1d-42dc-a4cb-8182eac4ef58/d90f7da4-ca39-48c6-8d97-b8d1e37c7dd0"
+					(reference "D7")
+					(unit 1)
+				)
+			)
+		)
+	)
+	(symbol
+		(lib_id "Transistor_FET:BUK7M27-80EX")
 		(at 50.8 49.53 0)
 		(unit 1)
@@
 			)
 		)
-		(property "Value" "NMOS"
+		(property "Value" "BUK7M27-80EX"
 			(at 57.15 50.7999 0)
 			(effects
@@
 			)
 		)
-		(property "Footprint" "UTSVT_Power:BUK7M1780EX"
-			(at 55.88 46.99 0)
-			(effects
-				(font
-					(size 1.27 1.27)
-				)
+		(property "Footprint" "Package_TO_SOT_SMD:LFPAK33"
+			(at 55.88 51.435 0)
+			(effects
+				(font
+					(size 1.27 1.27)
+					(italic yes)
+				)
+				(justify left)
 				(hide yes)
 			)
 		)
 		(property "Datasheet" "https://assets.nexperia.com/documents/data-sheet/BUK7M27-80E.pdf"
-			(at 50.8 62.23 0)
-			(effects
-				(font
-					(size 1.27 1.27)
-				)
-				(hide yes)
-			)
-		)
-		(property "Description" "N-MOSFET transistor, drain/source/gate"
+			(at 55.88 53.34 0)
+			(effects
+				(font
+					(size 1.27 1.27)
+				)
+				(justify left)
+				(hide yes)
+			)
+		)
+		(property "Description" "30A Id, 80V Vds, N-Channel TrenchMOS MOSFET, 27mOhm Ron, 19.5nC Qqd, -55 to 175 °C, LFPAK33"
 			(at 50.8 49.53 0)
 			(effects
@@
 			)
 		)
-		(property "Sim.Device" "NMOS"
-			(at 50.8 66.675 0)
-			(effects
-				(font
-					(size 1.27 1.27)
-				)
-				(hide yes)
-			)
-		)
-		(property "Sim.Type" "VDMOS"
-			(at 50.8 68.58 0)
-			(effects
-				(font
-					(size 1.27 1.27)
-				)
-				(hide yes)
-			)
-		)
-		(property "Sim.Pins" "1=D 2=G 3=S"
-			(at 50.8 64.77 0)
-			(effects
-				(font
-					(size 1.27 1.27)
-				)
-				(hide yes)
-			)
+		(pin "2"
 		)
 		(pin "3"
 		)
-		(pin "2"
-		)
-		(pin "1"
+		(pin "1"
+		)
+		(pin "5"
+		)
+		(pin "4"
 		)
 		(instances
@@
 				(path "/591f46f8-eb1d-42dc-a4cb-8182eac4ef58/d90f7da4-ca39-48c6-8d97-b8d1e37c7dd0"
 					(reference "Q1")
-					(unit 1)
-				)
-			)
-		)
-	)
-	(symbol
-		(lib_id "Diode:C3D25170H")
-		(at 176.53 38.1 90)
-		(unit 1)
-		(exclude_from_sim no)
-		(in_bom yes)
-		(on_board yes)
-		(dnp no)
-		(property "Reference" "D7"
-			(at 173.99 40.64 90)
-			(effects
-				(font
-					(size 1.27 1.27)
-				)
-				(justify left)
-			)
-		)
-		(property "Value" "VSSAF522-M3/H"
-			(at 194.056 40.132 90)
-			(effects
-				(font
-					(size 1.27 1.27)
-				)
-				(justify left)
-			)
-		)
-		(property "Footprint" "UTSVT_Passive:MMDL101T1G"
-			(at 180.975 38.1 0)
-			(effects
-				(font
-					(size 1.27 1.27)
-				)
-				(hide yes)
-			)
-		)
-		(property "Datasheet" "https://www.mouser.com/ProductDetail/Vishay-General-Semiconductor/VSSAF522-M3-H?qs=UkDUCjYnTB00gpgD%2Fb%2Fw%252BA%3D%3D"
-			(at 176.53 38.1 0)
-			(effects
-				(font
-					(size 1.27 1.27)
-				)
-				(hide yes)
-			)
-		)
-		(property "Description" ""
-			(at 176.53 38.1 0)
-			(effects
-				(font
-					(size 1.27 1.27)
-				)
-				(hide yes)
-			)
-		)
-		(pin "1"
-		)
-		(pin "2"
-		)
-		(instances
-			(project "PTN-PumpControlBoard"
-				(path "/591f46f8-eb1d-42dc-a4cb-8182eac4ef58/d90f7da4-ca39-48c6-8d97-b8d1e37c7dd0"
-					(reference "D7")
 					(unit 1)
 				)
@@
 					(unit 1)
 				)
-			)
-		)
-	)
-	(symbol
-		(lib_id "Simulation_SPICE:NMOS")
-		(at 124.46 49.53 0)
-		(unit 1)
-		(exclude_from_sim no)
-		(in_bom yes)
-		(on_board yes)
-		(dnp no)
-		(fields_autoplaced yes)
-		(property "Reference" "Q2"
-			(at 130.81 48.2599 0)
-			(effects
-				(font
-					(size 1.27 1.27)
-				)
-				(justify left)
-			)
-		)
-		(property "Value" "NMOS"
-			(at 130.81 50.7999 0)
-			(effects
-				(font
-					(size 1.27 1.27)
-				)
-				(justify left)
-			)
-		)
-		(property "Footprint" "UTSVT_Power:BUK7M1780EX"
-			(at 129.54 46.99 0)
-			(effects
-				(font
-					(size 1.27 1.27)
-				)
-				(hide yes)
-			)
-		)
-		(property "Datasheet" "https://assets.nexperia.com/documents/data-sheet/BUK7M27-80E.pdf"
-			(at 124.46 62.23 0)
-			(effects
-				(font
-					(size 1.27 1.27)
-				)
-				(hide yes)
-			)
-		)
-		(property "Description" "N-MOSFET transistor, drain/source/gate"
-			(at 124.46 49.53 0)
-			(effects
-				(font
-					(size 1.27 1.27)
-				)
-				(hide yes)
-			)
-		)
-		(property "Sim.Device" "NMOS"
-			(at 124.46 66.675 0)
-			(effects
-				(font
-					(size 1.27 1.27)
-				)
-				(hide yes)
-			)
-		)
-		(property "Sim.Type" "VDMOS"
-			(at 124.46 68.58 0)
-			(effects
-				(font
-					(size 1.27 1.27)
-				)
-				(hide yes)
-			)
-		)
-		(property "Sim.Pins" "1=D 2=G 3=S"
-			(at 124.46 64.77 0)
-			(effects
-				(font
-					(size 1.27 1.27)
-				)
-				(hide yes)
-			)
-		)
-		(pin "3"
-		)
-		(pin "2"
-		)
-		(pin "1"
-		)
-		(instances
-			(project "PTN-PumpControlBoard"
-				(path "/591f46f8-eb1d-42dc-a4cb-8182eac4ef58/d90f7da4-ca39-48c6-8d97-b8d1e37c7dd0"
-					(reference "Q2")
-					(unit 1)
-				)

Commit message: review notes
Connections:
- net FAN1_PWM: now also U2.7 (PWM2); no longer U2.5 (PWM1)
- net FAN1_TACH: now also U2.8 (TACH2); no longer U2.6 (TACH1)
- net FAN2_PWM: now also U2.5 (PWM1); no longer U2.7 (PWM2)
- net FAN2_TACH: now also U2.6 (TACH1); no longer U2.8 (TACH2)
- net GND: no longer D7.1 (K), D8.1 (K)
- net NET2: now reaches FAN2.3 (Pin_3), Q2.5 (D)
- net NET2: now also D8.1 (K)
- net NET1: now reaches FAN1.3 (Pin_3), Q1.5 (D)
- net NET1: now also D7.1 (K)
Other:
- note added: "test point/logic analyzer for pwm (1x)"

Commit message: schematic changes before switching submodules
Parts:
- added R36, R37: 100k, Resistor_SMD:R_0603_1608Metric, symbol Device:R_US
- Q1, Q2: value BUK7M27-80EX -> PSMN8R5-40MSDX
Connections:
- net FAN1_PWM: now also R36.1
- net FAN2_PWM: now also R37.1
- net GND: now also R36.2, R37.2
Other:
- note removed: "test point/logic analyzer for pwm (1x)"

Commit message: fixed submodule, schematic basically done
Other:
- moved on the sheet: R3, R4, R5, R6, R7, R8, R9

Commit message: finalized schematic (pls be the last time)
Parts:
- renumbered R4 to R10, R7 to R11, R36 to R2, R2 to R3, R37 to R4, R3 to R5, R5 to R6, R6 to R7
Changed lines of the file:
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@@
 		(dnp no)
 		(fields_autoplaced yes)
-		(property "Reference" "R6"
+		(property "Reference" "R7"
 			(at 181.61 82.5499 0)
 			(effects
@@
 			(project "PTN-PumpControlBoard"
 				(path "/591f46f8-eb1d-42dc-a4cb-8182eac4ef58/d90f7da4-ca39-48c6-8d97-b8d1e37c7dd0"
-					(reference "R6")
+					(reference "R7")
 					(unit 1)
 				)
@@
 		(dnp no)
 		(fields_autoplaced yes)
-		(property "Reference" "R4"
+		(property "Reference" "R10"
 			(at 140.97 104.1399 0)
 			(effects
@@
 			(project "PTN-PumpControlBoard"
 				(path "/591f46f8-eb1d-42dc-a4cb-8182eac4ef58/d90f7da4-ca39-48c6-8d97-b8d1e37c7dd0"
-					(reference "R4")
+					(reference "R10")
 					(unit 1)
 				)
@@
 		(dnp no)
 		(fields_autoplaced yes)
-		(property "Reference" "R7"
+		(property "Reference" "R11"
 			(at 181.61 104.1399 0)
 			(effects
@@
 			(project "PTN-PumpControlBoard"
 				(path "/591f46f8-eb1d-42dc-a4cb-8182eac4ef58/d90f7da4-ca39-48c6-8d97-b8d1e37c7dd0"
-					(reference "R7")
+					(reference "R11")
 					(unit 1)
 				)
@@
 		(dnp no)
 		(fields_autoplaced yes)
-		(property "Reference" "R5"
+		(property "Reference" "R6"
 			(at 160.02 82.5499 0)
 			(effects
@@
 			(project "PTN-PumpControlBoard"
 				(path "/591f46f8-eb1d-42dc-a4cb-8182eac4ef58/d90f7da4-ca39-48c6-8d97-b8d1e37c7dd0"
-					(reference "R5")
+					(reference "R6")
 					(unit 1)
 				)
@@
 		(on_board yes)
 		(dnp no)
-		(property "Reference" "R37"
+		(property "Reference" "R4"
 			(at 119.38 53.3399 0)
 			(effects
@@
 			(project "PTN-PumpControlBoard"
 				(path "/591f46f8-eb1d-42dc-a4cb-8182eac4ef58/d90f7da4-ca39-48c6-8d97-b8d1e37c7dd0"
-					(reference "R37")
+					(reference "R4")
 					(unit 1)
 				)
@@
 		(on_board yes)
 		(dnp no)
-		(property "Reference" "R2"
+		(property "Reference" "R3"
 			(at 120.65 34.2899 0)
 			(effects
@@
 			(project "PTN-PumpControlBoard"
 				(path "/591f46f8-eb1d-42dc-a4cb-8182eac4ef58/d90f7da4-ca39-48c6-8d97-b8d1e37c7dd0"
-					(reference "R2")
+					(reference "R3")
 					(unit 1)
 				)
@@
 		(dnp no)
 		(fields_autoplaced yes)
-		(property "Reference" "R3"
+		(property "Reference" "R5"
 			(at 139.7 82.5499 0)
 			(effects
@@
 			(project "PTN-PumpControlBoard"
 				(path "/591f46f8-eb1d-42dc-a4cb-8182eac4ef58/d90f7da4-ca39-48c6-8d97-b8d1e37c7dd0"
-					(reference "R3")
+					(reference "R5")
 					(unit 1)
 				)
@@
 		(on_board yes)
 		(dnp no)
-		(property "Reference" "R36"
+		(property "Reference" "R2"
 			(at 45.72 53.3399 0)
 			(effects
@@
 			(project "PTN-PumpControlBoard"
 				(path "/591f46f8-eb1d-42dc-a4cb-8182eac4ef58/d90f7da4-ca39-48c6-8d97-b8d1e37c7dd0"
-					(reference "R36")
-					(unit 1)
-				)
+					(reference "R2")
+					(unit 1)
+				)

Commit message: fixed diodes and some traces
Connections:
- net +24V: now also D7.1 (K), D8.1 (K); no longer D7.2 (A), D8.2 (A)
- net NET1: now also D7.2 (A); no longer D7.1 (K)
- net NET2: now also D8.2 (A); no longer D8.1 (K)
Other:
- moved on the sheet: D7, D8
Changed lines of the file:
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@@
 			"AGEAAABBAAAATwAAAGsAAAAwAAAAQwAAAEcAAABGAAAAVAAAAHEAAABJAAAARAAAAHEAAABzAAAA"
 			"egAAAEUAAAA0AAAAagAAADQAAAAzAAAAUwAAAEsAAABGAAAAVAAAADUAAABvAAAANgAAAGoAAAA1"
-			"AAAAZwAAAGsAAABCAAAAUQAAAHEAAABEAAAAMg=="
+			"AAAAZwAAAGsAAABCAAAAUQAAAHEAAABEAAAAMgAAAEoAAABQAAAAMwAAAHAAAAAxAAAARwAAAG4A"
+			"AABGAAAAOQAAADcAAAAzAAAAawAAAFYAAABSAAAANwAAAFAAAABtAAAAOAAAADQAAABTAAAALwAA"
+			"AHQAAABOAAAALwAAAHIAAAArAAAAUAAAAGIAAAByAAAAdAAAAGEAAABJAAAAaQAAADEAAABoAAAA"
+			"WgAAAEIAAABWAAAAegAAAHEAAAByAAAAYgAAAEEAAABKAAAASAAAAC8AAABiAAAAcwAAAE4AAAA1"
+			"AAAAawAAADQAAABRAAAAbAAAAGIAAABsAAAATAAAAEkAAABkAAAAQwAAAEIAAAA2AAAASAAAAEQA"
+			"AABFAAAAWgAAAEwAAAAwAAAAWAAAAC8AAAAvAAAANgAAAFYAAAAyAAAARQAAAHMAAABIAAAAWAAA"
+			"AHYAAABzAAAAcwAAAGQAAAB6AAAAMQAAAHEAAAA3AAAARAAAAEsAAAB1AAAANwAAAG4AAABBAAAA"
+			"UgAAAFoAAAArAAAASwAAAGkAAABGAAAAMQAAAHEAAABrAAAAYwAAAGgAAAA1AAAAagAAAEUAAABu"
+			"AAAAMQAAAHEAAAB6AAAARgAAAEMAAABVAAAATgAAAHAAAABNAAAANQAAAG0AAABHAAAAUgAAAG8A"
+			"AAA0AAAANQAAAG4AAABPAAAARwAAAG0AAAAyAAAASgAAAFMAAABnAAAAVwAAADEAAABYAAAASQAA"
+			"AGkAAABZAAAAcAAAADIAAAB0AAAAVwAAAE0AAABWAAAAZgAAAFUAAAAyAAAAVwAAAG8AAABlAAAA"
+			"RwAAAGIAAAAvAAAAWQAAAGQAAABDAAAAYwAAAGMAAAAyAAAAQwAAAHgAAABJAAAAeQAAAEsAAABY"
+			"AAAATwAAAGIAAABPAAAAUAAAADgAAABhAAAAbgAAAEsAAABqAAAAWAAAAHkAAABwAAAAWQAAAGUA"
+			"AABoAAAATgAAAGUAAABsAAAARQAAAFUAAABPAAAAdAAAAFUAAABtAAAAagAAADMAAABOAAAASAAA"
+			"AFoAAABGAAAAaQAAAHcAAABsAAAAUAAAADQAAABKAAAAWQAAAGoAAABNAAAAdAAAAHUAAABtAAAA"
+			"aQAAAHoAAABGAAAATgAAAG8AAAAyAAAAMwAAADAAAAB5AAAAdQAAAEgAAAAyAAAAeAAAAEsAAABW"
+			"AAAAZQAAAGcAAABNAAAARwAAAEQAAABCAAAAQQAAADQAAAA5AAAAMwAAADEAAABHAAAAUQAAAEQA"
+			"AABMAAAARwAAAGwAAABWAAAAbQAAAFcAAABOAAAANAAAAGcAAABtAAAAZQAAAEgAAABQAAAAVAAA"
+			"AFUAAABXAAAAOAAAAEwAAABiAAAAaQAAAEQAAA=="
 		)
 	)
@@
 			"QUFEVUFBQUJUQUFBQWNRQUFBR3NBQUFCWkFBQUFiQUFBQUVrQUFBQjFBQUFBU0FBQUFIRUFBQUJv"
 			"QUFBQVpBQUFBRkVBQUFCdkFBQUFRUUFBQUZFQUFBQkpBQUFBUVFBQUFGRUFBQUJKQUFBQVp3QUFB"
-			"Rw=="
+			"R6SdmiHz8JsLMHjbwdyHQ/68Y5rKxcIcyceN/zsSWAjmtj3seixO+4OWzgw8aYdUc6RzwpP/URCs"
+			"FVQB2PwFsYmhf3SDmknX3E57ikhvi0X2AAAAAAABAAAAAwAAAClFbnRydXN0IFJvb3QgQ2VydGlm"
+			"aWNhdGlvbiBBdXRob3JpdHkgLSBHMgAAAAAAAClFbnRydXN0IFJvb3QgQ2VydGlmaWNhdGlvbiBB"
+			"dXRob3JpdHkgLSBHMgAAAAAAAMEwgb4xCzAJBgNVBAYTAlVTMRYwFAYDVQQKEw1FTlRSVVNULCBJ"
+			"TkMuMSgwJgYDVQQLEx9TRUUgV1dXLkVOVFJVU1QuTkVUL0xFR0FMLVRFUk1TMTkwNwYDVQQLEzAo"
+			"QykgMjAwOSBFTlRSVVNULCBJTkMuIC0gRk9SIEFVVEhPUklaRUQgVVNFIE9OTFkxMjAwBgNVBAMT"
+			"KUVOVFJVU1QgUk9PVCBDRVJUSUZJQ0FUSU9OIEFVVEhPUklUWSAtIEcyAAAAAAAAwTCBvjELMAkG"
+			"A1UEBhMCVVMxFjAUBgNVBAoTDUVOVFJVU1QsIElOQy4xKDAmBgNVBAsTH1NFRSBXV1cuRU5UUlVT"
+			"VC5ORVQvTEVHQUwtVEVSTVMxOTA3BgNVBAsTMChDKSAyMDA5IEVOVFJVU1QsIElOQy4gLSBGT1Ig"
+			"QVVUSE9SSVpFRCBVU0UgT05MWTEyMDAGA1UEAxMpRU5UUlVTVCBST09UIENFUlRJRklDQVRJT04g"
+			"QVVUSE9SSVRZIC0gRzIAAAAAAAAESlOMKAAAABRqciZ60B7vfec7aVHUbI2fkBJmqwAAABRqciZ6"
+			"0B7vfec7aVHUbI2fkBJmqwAACegAAAABAAAAPQAAAAAAAAfRAAAAAAAACBEAAAgVAAAIGQAACDkA"
+			"AAhZAAAI4QAACaUAAAm5AAAJ0TCCB80wgga1oAMCAQICEB3CmLwCUPIISFLY9BaFJk8wDQYJKoZI"
+			"hvcNAQELBQAwgboxCzAJBgNVBAYTAlVTMRYwFAYDVQQKEw1FbnRydXN0LCBJbmMuMSgwJgYDVQQL"
+			"Ex9TZWUgd3d3LmVudHJ1c3QubmV0L2xlZ2FsLXRlcm1zMTkwNwYDVQQLEzAoYykgMjAxMiBFbnRy"
+			"dXN0LCBJbmMuIC0gZm9yIGF1dGhvcml6ZWQgdXNlIG9ubHkxLjAsBgNVBAMTJUVudHJ1c3QgQ2Vy"
+			"dGlmaWNhdGlvbiBBdXRob3JpdHkgLSBMMUswHhcNMjMwNDEyMjExNDI5WhcNMjQwMjI5MjExNDI5"
+			"WjCBgTELMAkGA1UEBhMCVVMxDjAMBgNVBAgTBVRleGFzMQ8wDQYDVQQHEwZBdXN0aW4xKzApBgNV"
+			"BA=="
 		)
 	)
@@
 	(symbol
 		(lib_id "Diode:C3D25170H")
-		(at 176.53 38.1 90)
+		(at 176.53 38.1 270)
 		(unit 1)
 		(exclude_from_sim no)
@@
 		(dnp no)
 		(property "Reference" "D7"
-			(at 173.99 40.64 90)
+			(at 179.07 35.56 90)
 			(effects
 				(font
@@
 		)
 		(property "Value" "VSSAF522-M3/H"
-			(at 194.056 40.132 90)
+			(at 159.004 36.068 90)
 			(effects
 				(font
@@
 		)
 		(property "Footprint" "UTSVT_Passive:MMDL101T1G"
-			(at 180.975 38.1 0)
+			(at 172.085 38.1 0)
 			(effects
 				(font
@@
 	(symbol
 		(lib_id "Diode:C3D25170H")
-		(at 203.2 38.1 90)
+		(at 203.2 38.1 270)
 		(unit 1)
 		(exclude_from_sim no)
@@
 		(dnp no)
 		(property "Reference" "D8"
-			(at 200.66 40.64 90)
+			(at 205.74 35.56 90)
 			(effects
 				(font
@@
 		)
 		(property "Value" "VSSAF522-M3/H"
-			(at 220.726 40.132 90)
+			(at 185.674 36.068 90)
 			(effects
 				(font
@@
 		)
 		(property "Footprint" "UTSVT_Passive:MMDL101T1G"
-			(at 207.645 38.1 0)
+			(at 198.755 38.1 0)
 			(effects
 				(font
