File: Pump.kicad_sch (KiCad schematic)
At the start: 1 part

Commit message: schematic with 12V components, unigain buffers & extra temp sensor
Parts:
- added R11: R_Shunt_US, symbol Device:R_Shunt_US
- added R12: 1k, Resistor_SMD:R_0805_2012Metric, symbol Device:R_US
- added R13: 380, Resistor_SMD:R_0805_2012Metric, symbol Device:R_US
- PUMP1: footprint UTSVT_Connectors:Molex_MicroFit3.0_1x4xP3.00mm_PolarizingPeg_Vertical -> Connector_Molex:Molex_Nano-Fit_105309-xx04_1x04_P2.50mm_Vertical
Connections:
- net GND: now also R11.4, R13.2; no longer PUMP1.4 (Pin_4)
- net PG: now also R12.2, R13.1; no longer PUMP1.1 (Pin_1)
- new net: PUMP1.4 (Pin_4), R11.1
- new net PG_12V: PUMP1.1 (Pin_1), R12.1
- new net SHUNT_A: R11.2
- new net SHUNT_B: R11.3
Other:
- moved on the sheet: PUMP1

Commit message: repicked parts to be 24V tolerant and changed corresponding circuitry
Parts:
- removed R11: R_Shunt_US, symbol Device:R_Shunt_US
- removed R12: 1k, Resistor_SMD:R_0805_2012Metric, symbol Device:R_US
- removed R13: 380, Resistor_SMD:R_0805_2012Metric, symbol Device:R_US
- added R15: 1k, Resistor_SMD:R_0805_2012Metric, symbol Device:R_US
Connections:
- net GND: now also PUMP1.4 (Pin_4)
- net +12V renamed FG
- net FG: now also R15.2
- net PG_12V renamed +24V
- new net +3.3V: R15.1
Other:
- note added: "correct val?"

Commit message: added test points and headers, AGND and 12V not fully connected
Parts:
- added GND2, P_FG1, P_PWM1: Scope_TP, TestPoint:TestPoint_Keystone_5010-5014_Multipurpose, symbol Connector:TestPoint
Connections:
- net FG: now also P_FG1.1
- net GND: now also GND2.1
- net PWM3: now also P_PWM1.1
Other:
- moved on the sheet: PUMP1, R15

Commit message: filled zones finally workinggggg
Changed lines of the file:
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@@
 		(on_board yes)
 		(dnp no)
+		(fields_autoplaced yes)
 		(property "Reference" "#PWR042"
 			(at 44.45 39.37 0)
@@
 		)
 		(property "Value" "+3.3V"
-			(at 44.45 31.75 0)
+			(at 44.45 30.48 0)
 			(effects
 				(font
@@
 		)
 		(instances
-			(project "PTN-PumpControlBoard"
+			(project ""
 				(path "/591f46f8-eb1d-42dc-a4cb-8182eac4ef58/49b28e86-cfde-410d-931b-2f924e16f8d9"
 					(reference "#PWR042")

Commit message: Fixed fan schematic based on review feedback
Parts:
- removed GND2, P_FG1, P_PWM1: Scope_TP, TestPoint:TestPoint_Keystone_5010-5014_Multipurpose, symbol Connector:TestPoint
Other:
- moved on the sheet: R15

Commit message: updated schematic with low pass for temp sensors and new resistor footprint
Parts:
- R15: footprint Resistor_SMD:R_0805_2012Metric -> Resistor_SMD:R_0603_1608Metric
Changed lines of the file:
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@@
 			)
 		)
-		(property "Footprint" "Resistor_SMD:R_0805_2012Metric"
+		(property "Footprint" "Resistor_SMD:R_0603_1608Metric"
 			(at 54.356 40.894 90)
 			(effects

Commit message: fixed all review notes for schematic
Parts:
- R31: renamed from R15; value 1k -> 10k
Other:
- note removed: "correct val?"
Changed lines of the file:
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@@
 	(generator_version "9.0")
 	(paper "A4")
-	(text "correct val?"
-		(exclude_from_sim no)
-		(at 45.72 40.64 0)
-		(effects
-			(font
-				(size 1.27 1.27)
-			)
-		)
-	)
 	(text_box "Pump: 24V, 9.5W\nFG_FEEDBACK: open drain output RPM=30*f\nPWM: 3.3V logic"
 		(exclude_from_sim no)
@@
 		(dnp no)
 		(fields_autoplaced yes)
-		(property "Reference" "#PWR043"
+		(property "Reference" "#PWR064"
 			(at 71.12 40.64 0)
 			(effects
@@
 			(project "PTN-PumpControlBoard"
 				(path "/591f46f8-eb1d-42dc-a4cb-8182eac4ef58/49b28e86-cfde-410d-931b-2f924e16f8d9"
-					(reference "#PWR043")
+					(reference "#PWR064")
 					(unit 1)
 				)
@@
 		(dnp no)
 		(fields_autoplaced yes)
-		(property "Reference" "#PWR044"
+		(property "Reference" "#PWR065"
 			(at 71.12 54.61 0)
 			(effects
@@
 			(project "PTN-PumpControlBoard"
 				(path "/591f46f8-eb1d-42dc-a4cb-8182eac4ef58/49b28e86-cfde-410d-931b-2f924e16f8d9"
-					(reference "#PWR044")
+					(reference "#PWR065")
 					(unit 1)
 				)
@@
 		(dnp no)
 		(fields_autoplaced yes)
-		(property "Reference" "#PWR042"
+		(property "Reference" "#PWR063"
 			(at 53.34 39.37 0)
 			(effects
@@
 			(project ""
 				(path "/591f46f8-eb1d-42dc-a4cb-8182eac4ef58/49b28e86-cfde-410d-931b-2f924e16f8d9"
-					(reference "#PWR042")
+					(reference "#PWR063")
 					(unit 1)
 				)
@@
 		(on_board yes)
 		(dnp no)
-		(property "Reference" "R15"
+		(property "Reference" "R31"
 			(at 55.88 39.3699 0)
 			(effects
@@
 			)
 		)
-		(property "Value" "1k"
+		(property "Value" "10k"
 			(at 55.88 41.9099 0)
 			(effects
@@
 			(project "PTN-PumpControlBoard"
 				(path "/591f46f8-eb1d-42dc-a4cb-8182eac4ef58/49b28e86-cfde-410d-931b-2f924e16f8d9"
-					(reference "R15")
+					(reference "R31")
 					(unit 1)
 				)
