File: Pump.kicad_sch (KiCad schematic)
At the start: 2 parts

Commit message: review notes
Parts:
- added D10: VSSAF522-M3/H, UTSVT_Passive:MMDL101T1G, symbol Diode:C3D25170H
Connections:
- net +24V: now also D10.2 (A)
- net GND: now also D10.1 (K)
Other:
- note added: "pmos for pwm pin"
Changed lines of the file:
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@@
 	(generator_version "9.0")
 	(paper "A4")
+	(text "pmos for pwm pin"
+		(exclude_from_sim no)
+		(at 65.278 25.146 0)
+		(effects
+			(font
+				(size 1.27 1.27)
+			)
+		)
+	)
 	(text_box "Pump: 24V, 9.5W\nFG_FEEDBACK: open drain output RPM=30*f\nPWM: 3.3V logic"
 		(exclude_from_sim no)
@@
 	(wire
 		(pts
+			(xy 24.13 48.26) (xy 24.13 45.72)
+		)
+		(stroke
+			(width 0)
+			(type default)
+		)
+	)
+	(wire
+		(pts
 			(xy 53.34 44.45) (xy 72.39 44.45)
 		)
@@
 		(pts
 			(xy 71.12 36.83) (xy 71.12 39.37)
+		)
+		(stroke
+			(width 0)
+			(type default)
+		)
+	)
+	(wire
+		(pts
+			(xy 24.13 34.29) (xy 24.13 38.1)
 		)
 		(stroke
@@
 	(symbol
 		(lib_id "power:+24V")
+		(at 24.13 34.29 0)
+		(unit 1)
+		(exclude_from_sim no)
+		(in_bom yes)
+		(on_board yes)
+		(dnp no)
+		(fields_autoplaced yes)
+		(property "Reference" "#PWR074"
+			(at 24.13 38.1 0)
+			(effects
+				(font
+					(size 1.27 1.27)
+				)
+				(hide yes)
+			)
+		)
+		(property "Value" "+24V"
+			(at 24.13 29.21 0)
+			(effects
+				(font
+					(size 1.27 1.27)
+				)
+			)
+		)
+		(property "Footprint" ""
+			(at 24.13 34.29 0)
+			(effects
+				(font
+					(size 1.27 1.27)
+				)
+				(hide yes)
+			)
+		)
+		(property "Datasheet" ""
+			(at 24.13 34.29 0)
+			(effects
+				(font
+					(size 1.27 1.27)
+				)
+				(hide yes)
+			)
+		)
+		(property "Description" "Power symbol creates a global label with name \"+24V\""
+			(at 24.13 34.29 0)
+			(effects
+				(font
+					(size 1.27 1.27)
+				)
+				(hide yes)
+			)
+		)
+		(pin "1"
+		)
+		(instances
+			(project "PTN-PumpControlBoard"
+				(path "/591f46f8-eb1d-42dc-a4cb-8182eac4ef58/49b28e86-cfde-410d-931b-2f924e16f8d9"
+					(reference "#PWR074")
+					(unit 1)
+				)
+			)
+		)
+	)
+	(symbol
+		(lib_id "power:+24V")
 		(at 71.12 36.83 0)
 		(unit 1)
@@
 	)
 	(symbol
+		(lib_id "power:GND")
+		(at 24.13 48.26 0)
+		(unit 1)
+		(exclude_from_sim no)
+		(in_bom yes)
+		(on_board yes)
+		(dnp no)
+		(fields_autoplaced yes)
+		(property "Reference" "#PWR075"
+			(at 24.13 54.61 0)
+			(effects
+				(font
+					(size 1.27 1.27)
+				)
+				(hide yes)
+			)
+		)
+		(property "Value" "GND"
+			(at 24.13 53.34 0)
+			(effects
+				(font
+					(size 1.27 1.27)
+				)
+			)
+		)
+		(property "Footprint" ""
+			(at 24.13 48.26 0)
+			(effects
+				(font
+					(size 1.27 1.27)
+				)
+				(hide yes)
+			)
+		)
+		(property "Datasheet" ""
+			(at 24.13 48.26 0)
+			(effects
+				(font
+					(size 1.27 1.27)
+				)
+				(hide yes)
+			)
+		)
+		(property "Description" "Power symbol creates a global label with name \"GND\" , ground"
+			(at 24.13 48.26 0)
+			(effects
+				(font
+					(size 1.27 1.27)
+				)
+				(hide yes)
+			)
+		)
+		(pin "1"
+		)
+		(instances
+			(project "PTN-PumpControlBoard"
+				(path "/591f46f8-eb1d-42dc-a4cb-8182eac4ef58/49b28e86-cfde-410d-931b-2f924e16f8d9"
+					(reference "#PWR075")
+					(unit 1)
+				)
+			)
+		)
+	)
+	(symbol
 		(lib_id "power:+3.3V")
 		(at 53.34 35.56 0)
@@
 					(unit 1)
 				)
+			)
+		)
+	)
+	(symbol
+		(lib_id "Diode:C3D25170H")
+		(at 24.13 41.91 90)
+		(unit 1)
+		(exclude_from_sim no)
+		(in_bom yes)
+		(on_board yes)
+		(dnp no)
+		(property "Reference" "D10"
+			(at 21.59 44.45 90)
+			(effects
+				(font
+					(size 1.27 1.27)
+				)
+				(justify left)
+			)
+		)
+		(property "Value" "VSSAF522-M3/H"
+			(at 41.656 43.942 90)
+			(effects
+				(font
+					(size 1.27 1.27)
+				)
+				(justify left)
+			)
+		)
+		(property "Footprint" "UTSVT_Passive:MMDL101T1G"
+			(at 28.575 41.91 0)
+			(effects
+				(font
+					(size 1.27 1.27)
+				)
+				(hide yes)
+			)
+		)
+		(property "Datasheet" "https://www.mouser.com/ProductDetail/Vishay-General-Semiconductor/VSSAF522-M3-H?qs=UkDUCjYnTB00gpgD%2Fb%2Fw%252BA%3D%3D"
+			(at 24.13 41.91 0)
+			(effects
+				(font
+					(size 1.27 1.27)
+				)
+				(hide yes)
+			)
+		)
+		(property "Description" ""
+			(at 24.13 41.91 0)
+			(effects
+				(font
+					(size 1.27 1.27)
+				)
+				(hide yes)
+			)
+		)
+		(pin "1"
+		)
+		(pin "2"
+		)
+		(instances
+			(project "PTN-PumpControlBoard"
+				(path "/591f46f8-eb1d-42dc-a4cb-8182eac4ef58/49b28e86-cfde-410d-931b-2f924e16f8d9"
+					(reference "D10")
+					(unit 1)
+				)

Commit message: schematic changes before switching submodules
Parts:
- added Q5: PSMN8R5-40MSDX, Package_TO_SOT_SMD:LFPAK33, symbol Transistor_FET:BUK7M27-80EX
- added R32: 100, Resistor_SMD:R_0603_1608Metric, symbol Device:R_US
- added R33: 100k, Resistor_SMD:R_0603_1608Metric, symbol Device:R_US
- added R34: 10k, Resistor_SMD:R_0603_1608Metric, symbol Device:R_US
Connections:
- net +3.3V: now also R34.1
- net GND: now also Q5.1 (S), Q5.2 (S), Q5.3 (S), R33.2
- net PWM3: now also R32.1
- new net: Q5.4 (G), R32.2, R33.1
- new net PWM: Q5.5 (D), R34.2
Other:
- note added: "flipping logic in sw"
- note removed: "pmos for pwm pin"
- moved on the sheet: D10, PUMP1, R31

Commit message: finalized schematic (pls be the last time)
Parts:
- renumbered R31 to R33, R32 to R34, R33 to R35, R34 to R36
Changed lines of the file:
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@@
 		(on_board yes)
 		(dnp no)
-		(property "Reference" "R32"
+		(property "Reference" "R34"
 			(at 133.35 38.862 90)
 			(effects
@@
 			(project "PTN-PumpControlBoard"
 				(path "/591f46f8-eb1d-42dc-a4cb-8182eac4ef58/49b28e86-cfde-410d-931b-2f924e16f8d9"
-					(reference "R32")
+					(reference "R34")
 					(unit 1)
 				)
@@
 		(on_board yes)
 		(dnp no)
-		(property "Reference" "R31"
+		(property "Reference" "R33"
 			(at 69.85 39.3699 0)
 			(effects
@@
 			(project "PTN-PumpControlBoard"
 				(path "/591f46f8-eb1d-42dc-a4cb-8182eac4ef58/49b28e86-cfde-410d-931b-2f924e16f8d9"
-					(reference "R31")
+					(reference "R33")
 					(unit 1)
 				)
@@
 		(on_board yes)
 		(dnp no)
-		(property "Reference" "R34"
+		(property "Reference" "R36"
 			(at 151.13 27.9399 0)
 			(effects
@@
 			(project "PTN-PumpControlBoard"
 				(path "/591f46f8-eb1d-42dc-a4cb-8182eac4ef58/49b28e86-cfde-410d-931b-2f924e16f8d9"
-					(reference "R34")
+					(reference "R36")
 					(unit 1)
 				)
@@
 		(on_board yes)
 		(dnp no)
-		(property "Reference" "R33"
+		(property "Reference" "R35"
 			(at 139.7 48.2599 0)
 			(effects
@@
 			(project "PTN-PumpControlBoard"
 				(path "/591f46f8-eb1d-42dc-a4cb-8182eac4ef58/49b28e86-cfde-410d-931b-2f924e16f8d9"
-					(reference "R33")
-					(unit 1)
-				)
+					(reference "R35")
+					(unit 1)
+				)

Commit message: all subcircuits other than rpp
Connections:
- net FG: now also PUMP1.2 (Pin_2); no longer PUMP1.3 (Pin_3)
- net PWM3: now also PUMP1.3 (Pin_3); no longer PUMP1.2 (Pin_2)
Other:
- moved on the sheet: R33
Changed lines of the file:
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@@
 	)
 	(junction
-		(at 67.31 44.45)
+		(at 67.31 41.91)
 		(diameter 0)
 		(color 0 0 0 0)
@@
 	(wire
 		(pts
-			(xy 67.31 44.45) (xy 86.36 44.45)
-		)
-		(stroke
-			(width 0)
-			(type default)
-		)
-	)
-	(wire
-		(pts
 			(xy 124.46 43.18) (xy 128.27 43.18)
 		)
@@
 	(wire
 		(pts
-			(xy 67.31 35.56) (xy 67.31 36.83)
-		)
-		(stroke
-			(width 0)
-			(type default)
-		)
-	)
-	(wire
-		(pts
 			(xy 85.09 46.99) (xy 86.36 46.99)
 		)
@@
 	(wire
 		(pts
-			(xy 82.55 41.91) (xy 86.36 41.91)
-		)
-		(stroke
-			(width 0)
-			(type default)
-		)
-	)
-	(wire
-		(pts
 			(xy 85.09 39.37) (xy 86.36 39.37)
 		)
@@
 	(wire
 		(pts
+			(xy 82.55 44.45) (xy 86.36 44.45)
+		)
+		(stroke
+			(width 0)
+			(type default)
+		)
+	)
+	(wire
+		(pts
 			(xy 85.09 36.83) (xy 85.09 39.37)
 		)
@@
 	(wire
 		(pts
+			(xy 67.31 41.91) (xy 86.36 41.91)
+		)
+		(stroke
+			(width 0)
+			(type default)
+		)
+	)
+	(wire
+		(pts
 			(xy 148.59 33.02) (xy 148.59 35.56)
 		)
@@
 	(wire
 		(pts
-			(xy 64.77 44.45) (xy 67.31 44.45)
+			(xy 64.77 41.91) (xy 67.31 41.91)
 		)
 		(stroke
@@
 		(pts
 			(xy 148.59 35.56) (xy 154.94 35.56)
+		)
+		(stroke
+			(width 0)
+			(type default)
+		)
+	)
+	(wire
+		(pts
+			(xy 67.31 33.02) (xy 67.31 34.29)
 		)
 		(stroke
@@
 	(hierarchical_label "PWM3"
 		(shape input)
-		(at 82.55 41.91 180)
+		(at 82.55 44.45 180)
 		(effects
 			(font
@@
 	(hierarchical_label "FG"
 		(shape output)
-		(at 64.77 44.45 180)
+		(at 64.77 41.91 180)
 		(effects
 			(font
@@
 	(symbol
 		(lib_id "power:+3.3V")
-		(at 67.31 35.56 0)
+		(at 67.31 33.02 0)
 		(unit 1)
 		(exclude_from_sim no)
@@
 		(fields_autoplaced yes)
 		(property "Reference" "#PWR063"
-			(at 67.31 39.37 0)
+			(at 67.31 36.83 0)
 			(effects
 				(font
@@
 		)
 		(property "Value" "+3.3V"
-			(at 67.31 30.48 0)
+			(at 67.31 27.94 0)
 			(effects
 				(font
@@
 		)
 		(property "Footprint" ""
-			(at 67.31 35.56 0)
+			(at 67.31 33.02 0)
 			(effects
 				(font
@@
 		)
 		(property "Datasheet" ""
-			(at 67.31 35.56 0)
+			(at 67.31 33.02 0)
 			(effects
 				(font
@@
 		)
 		(property "Description" "Power symbol creates a global label with name \"+3.3V\""
-			(at 67.31 35.56 0)
-			(effects
-				(font
-					(size 1.27 1.27)
-				)
-				(hide yes)
-			)
-		)
-		(pin "1"
-		)
-		(instances
-			(project ""
+			(at 67.31 33.02 0)
+			(effects
+				(font
+					(size 1.27 1.27)
+				)
+				(hide yes)
+			)
+		)
+		(pin "1"
+		)
+		(instances
+			(project "PTN-PumpControlBoard"
 				(path "/591f46f8-eb1d-42dc-a4cb-8182eac4ef58/49b28e86-cfde-410d-931b-2f924e16f8d9"
 					(reference "#PWR063")
@@
 	(symbol
 		(lib_id "Device:R_US")
-		(at 67.31 40.64 0)
+		(at 67.31 38.1 0)
 		(unit 1)
 		(exclude_from_sim no)
@@
 		(dnp no)
 		(property "Reference" "R33"
+			(at 69.85 36.8299 0)
+			(effects
+				(font
+					(size 1.27 1.27)
+				)
+				(justify left)
+			)
+		)
+		(property "Value" "10k"
 			(at 69.85 39.3699 0)
 			(effects
@@
 			)
 		)
-		(property "Value" "10k"
-			(at 69.85 41.9099 0)
-			(effects
-				(font
-					(size 1.27 1.27)
-				)
-				(justify left)
-			)
-		)
 		(property "Footprint" "Resistor_SMD:R_0603_1608Metric"
-			(at 68.326 40.894 90)
+			(at 68.326 38.354 90)
 			(effects
 				(font
@@
 		)
 		(property "Datasheet" "~"
-			(at 67.31 40.64 0)
+			(at 67.31 38.1 0)
 			(effects
 				(font
@@
 		)
 		(property "Description" "Resistor, US symbol"
-			(at 67.31 40.64 0)
-			(effects
-				(font
+			(at 67.31 38.1 0)
+			(effects
+				(font

Commit message: rounded corners and added rpp bypass
Parts:
- PUMP1: footprint Connector_Molex:Molex_Nano-Fit_105309-xx04_1x04_P2.50mm_Vertical -> UTSVT_Connectors:Molex_Nano-Fit_105309-xx04_1x04_P2.50mm_Vertical; Notes Small signal control for pump -> (none)
Changed lines of the file:
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@@
+	)
+	(symbol
+		(lib_id "Connector_Generic:Conn_01x04")
+		(at 91.44 41.91 0)
+		(unit 1)
+		(exclude_from_sim no)
+		(in_bom yes)
+		(on_board yes)
+		(dnp no)
+		(fields_autoplaced yes)
+		(property "Reference" "PUMP1"
+			(at 93.98 41.9099 0)
+			(effects
+				(font
+					(size 1.27 1.27)
+				)
+				(justify left)
+			)
+		)
+		(property "Value" "Conn_01x04"
+			(at 93.98 44.4499 0)
+			(effects
+				(font
+					(size 1.27 1.27)
+				)
+				(justify left)
+			)
+		)
+		(property "Footprint" "UTSVT_Connectors:Molex_Nano-Fit_105309-xx04_1x04_P2.50mm_Vertical"
+			(at 91.44 41.91 0)
+			(effects
+				(font
+					(size 1.27 1.27)
+				)
+				(hide yes)
+			)
+		)
+		(property "Datasheet" "~"
+			(at 91.44 41.91 0)
+			(effects
+				(font
+					(size 1.27 1.27)
+				)
+				(hide yes)
+			)
+		)
+		(property "Description" "Generic connector, single row, 01x04, script generated (kicad-library-utils/schlib/autogen/connector/)"
+			(at 91.44 41.91 0)
+			(effects
+				(font
+					(size 1.27 1.27)
+				)
+				(hide yes)
+			)
+		)
+		(pin "3"
+		)
+		(pin "1"
+		)
+		(pin "2"
+		)
+		(pin "4"
+		)
+		(instances
+			(project "PTN-PumpControlBoard"
+				(path "/591f46f8-eb1d-42dc-a4cb-8182eac4ef58/49b28e86-cfde-410d-931b-2f924e16f8d9"
+					(reference "PUMP1")
+					(unit 1)
+				)
+			)
+		)
 	)
 	(symbol
@@
 					(unit 1)
 				)
-			)
-		)
-	)
-	(symbol
-		(lib_id "Connector_Generic:Conn_01x04")
-		(at 91.44 41.91 0)
-		(unit 1)
-		(exclude_from_sim no)
-		(in_bom yes)
-		(on_board yes)
-		(dnp no)
-		(fields_autoplaced yes)
-		(property "Reference" "PUMP1"
-			(at 93.98 41.9099 0)
-			(effects
-				(font
-					(size 1.27 1.27)
-				)
-				(justify left)
-			)
-		)
-		(property "Value" "Conn_01x04"
-			(at 93.98 44.4499 0)
-			(effects
-				(font
-					(size 1.27 1.27)
-				)
-				(justify left)
-			)
-		)
-		(property "Footprint" "Connector_Molex:Molex_Nano-Fit_105309-xx04_1x04_P2.50mm_Vertical"
-			(at 91.44 41.91 0)
-			(effects
-				(font
-					(size 1.27 1.27)
-				)
-				(hide yes)
-			)
-		)
-		(property "Datasheet" "https://www.rigidhvac.com/store/products/12v-24v-pump-reservoir-combo-65mm"
-			(at 91.44 41.91 0)
-			(effects
-				(font
-					(size 1.27 1.27)
-				)
-				(hide yes)
-			)
-		)
-		(property "Description" "Generic connector, single row, 01x04, script generated (kicad-library-utils/schlib/autogen/connector/)"
-			(at 91.44 41.91 0)
-			(effects
-				(font
-					(size 1.27 1.27)
-				)
-				(hide yes)
-			)
-		)
-		(property "Notes" "Small signal control for pump"
-			(at 91.44 41.91 0)
-			(effects
-				(font
-					(size 1.27 1.27)
-				)
-				(hide yes)
-			)
-		)
-		(pin "4"
-		)
-		(pin "2"
-		)
-		(pin "3"
-		)
-		(pin "1"
-		)
-		(instances
-			(project "PTN-PumpControlBoard"
-				(path "/591f46f8-eb1d-42dc-a4cb-8182eac4ef58/49b28e86-cfde-410d-931b-2f924e16f8d9"
-					(reference "PUMP1")
-					(unit 1)
-				)

Commit message: fixed header
Parts:
- removed Q5: PSMN8R5-40MSDX, Package_TO_SOT_SMD:LFPAK33, symbol Transistor_FET:BUK7M27-80EX
- removed R36: 10k, Resistor_SMD:R_0603_1608Metric, symbol Device:R_US
- added Q5: BUK6M61-60PX, BUK6M61-60PX:BUK9M34100EX, symbol BUK6M61-60PX:BUK6M61-60PX
- added Q6: PMOS, symbol Simulation_SPICE:PMOS
Connections:
- net +3.3V: now also Q5.1 (S_1), Q5.2 (S_2), Q5.3 (S_3), Q6.3 (S)
- net PWM: now also PUMP1.3 (Pin_3), Q5.10 (D_6), Q5.11 (D_7), Q5.5 (D_1), Q5.6 (D_2), Q5.7 (D_3), Q5.8 (D_4), Q5.9 (D_5), Q6.1 (D)
- net PWM3: no longer PUMP1.3 (Pin_3)
- net P_GATE: now reaches R34.2, R35.1
- net P_GATE: now also Q5.4 (G), Q6.2 (G)
Other:
- note added: "real nmos symbol with correct footprint"
- note added: "symbol for schematic clarity not populated on board"
- note removed: "flipping logic in sw"

Commit message: fixed cap vals + made schem pretty
Other:
- note added: "real pmos symbol with correct footprint"
- note removed: "real nmos symbol with correct footprint"
Changed lines of the file:
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@@
 		)
 	)
-	(text "real nmos symbol with correct footprint"
+	(text "real pmos symbol with correct footprint"
 		(exclude_from_sim no)
 		(at 206.248 55.118 0)
