File: Pump.kicad_sch (KiCad schematic)
At the start: 7 parts, among them Q5 BUK6M61-60PX, Q6 PMOS

Commit message: initial schem changes
Parts:
- removed Q5: BUK6M61-60PX, BUK6M61-60PX:BUK9M34100EX, symbol BUK6M61-60PX:BUK6M61-60PX
- removed Q6: PMOS, symbol Simulation_SPICE:PMOS
- removed R33: 10k, Resistor_SMD:R_0603_1608Metric, symbol Device:R_US
- removed R34: 100, Resistor_SMD:R_0603_1608Metric, symbol Device:R_US
- removed R35: 100k, Resistor_SMD:R_0603_1608Metric, symbol Device:R_US
- added FLOW1: Conn_01x03, Connector_Molex:Molex_Nano-Fit_105309-xx03_1x03_P2.50mm_Vertical, symbol Connector_Generic:Conn_01x03
- added Q7: PMOS, symbol Simulation_SPICE:PMOS
- added Q8: BUK6M61-60PX, BUK9M34100EX, symbol BUK6M61-60PX:BUK6M61-60PX
- added R27: 100, Resistor_SMD:R_0603_1608Metric, symbol Device:R_US
- added R28: 100k, Resistor_SMD:R_0603_1608Metric, symbol Device:R_US
- D10: footprint UTSVT_Passive:MMDL101T1G -> Package_TO_SOT_THT:TO-247-2_Vertical
Connections:
- net PWM is gone; now on net PWM3: PUMP1.3 (Pin_3)
- net +3.3V: now also Q7.3 (S), Q8.1 (S_1), Q8.2 (S_2), Q8.3 (S_3)
- net GND: now also FLOW1.2 (Pin_2), R28.2
- net FG: no longer names the net of PUMP1.2 (Pin_2)
- new net +5V: FLOW1.1 (Pin_1)
- new net FLOW_OUT: FLOW1.3 (Pin_3), R27.1
- new net FLOW_SEN: Q7.1 (D), Q8.10 (D_6), Q8.11 (D_7), Q8.5 (D_1), Q8.6 (D_2), Q8.7 (D_3), Q8.8 (D_4), Q8.9 (D_5)
- new net F_GATE: Q7.2 (G), Q8.4 (G), R27.2, R28.1
- no-connect marks 0 -> 1
Other:
- note added: "tach no work"
- moved on the sheet: D10, PUMP1
