File: FlowrateSensor.kicad_sch (KiCad schematic)
At the start: 4 parts, among them Q3 NMOS

Commit message: Initial layout with 1 pump, 2 temp, 1 flow all on front side
Parts:
- Q3: footprint Package_TO_SOT_SMD:LFPAK33 -> Package_TO_SOT_SMD:SOT-23
Changed lines of the file:
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@@
 			)
 		)
-		(property "Footprint" "Package_TO_SOT_SMD:LFPAK33"
+		(property "Footprint" "Package_TO_SOT_SMD:SOT-23"
 			(at 118.11 41.91 0)
 			(effects

Commit message: schematic with 12V components, unigain buffers & extra temp sensor
Parts:
- removed FLOW1: Conn_01x03, UTSVT_Connectors:Molex_MicroFit3.0_1x3xP3.00mm_PolarizingPeg_Vertical, symbol Connector_Generic:Conn_01x03
- removed Q3: NMOS, Package_TO_SOT_SMD:SOT-23, symbol Simulation_SPICE:NMOS
- removed R19, R20: 10k, Resistor_SMD:R_0805_2012Metric, symbol Device:R_US
- added FLOW2: Conn_01x03, Connector_Molex:Molex_Nano-Fit_105309-xx03_1x03_P2.50mm_Vertical, symbol Connector_Generic:Conn_01x03
- added R27: 1.4k, Resistor_SMD:R_0805_2012Metric, symbol Device:R_US
- added R28: 100, Resistor_SMD:R_0805_2012Metric, symbol Device:R_US
- added U5: TLV6001DCK, Package_TO_SOT_SMD:SOT-353_SC-70-5, symbol Amplifier_Operational:TLV6001DCK
Connections:
- net +12V: now also FLOW2.2 (Pin_2)
- net +3.3V: now also U5.5 (V+)
- net FLOW_OUT: now also FLOW2.1 (Pin_1), U5.1 (+)
- net FLOW_SEN: now also R27.1, U5.4
- net GND: now also FLOW2.3 (Pin_3), R28.2, U5.2 (V-)
- new net: R27.2, R28.1, U5.3 (-)

Commit message: repicked parts to be 24V tolerant and changed corresponding circuitry
Parts:
- renumbered FLOW2 to FLOW1, R28 to R13, R27 to R14, U5 to U6
Connections:
- net +12V is gone; now on net FLOW_OUT: FLOW1.2 (Pin_2)
- net FLOW_OUT: no longer FLOW1.1 (Pin_1)
- new net +24V: FLOW1.1 (Pin_1)
Changed lines of the file:
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@@
 	(generator_version "9.0")
 	(paper "A4")
-	(text_box "- Flow out between -200mV and 200mV\n- Detecting voltages above 150mV for rising edge\n- Gain of 15 (1 + 1.4k/100)\n- 0.2V -> 3V & 150mV -> 2.25V"
+	(text_box "- rated for 4.5-24 V (nothing higher exists)\n- only tested at 12V, if the following values are different, I'll change Rf\n- Flow out between -200mV and 200mV\n- Detecting voltages above 150mV for rising edge\n- Gain of 15 (1 + 1.4k/100)\n- 0.2V -> 3V & 150mV -> 2.25V"
 		(exclude_from_sim no)
 		(at 165.1 50.8 0)
-		(size 43.815 12.7)
+		(size 46.355 18.415)
 		(margins 0.9525 0.9525 0.9525 0.9525)
 		(stroke
@@
 	(wire
 		(pts
-			(xy 40.64 57.15) (xy 40.64 48.26)
+			(xy 54.61 57.15) (xy 58.42 57.15)
 		)
 		(stroke
@@
 	(wire
 		(pts
+			(xy 58.42 54.61) (xy 53.34 54.61)
+		)
+		(stroke
+			(width 0)
+			(type default)
+		)
+	)
+	(wire
+		(pts
 			(xy 130.81 50.8) (xy 133.35 50.8)
 		)
@@
 	(wire
 		(pts
-			(xy 54.61 54.61) (xy 58.42 54.61)
-		)
-		(stroke
-			(width 0)
-			(type default)
-		)
-	)
-	(wire
-		(pts
-			(xy 58.42 57.15) (xy 40.64 57.15)
-		)
-		(stroke
-			(width 0)
-			(type default)
-		)
-	)
-	(wire
-		(pts
 			(xy 119.38 59.69) (xy 119.38 58.42)
 		)
@@
 	(wire
 		(pts
+			(xy 53.34 54.61) (xy 53.34 48.26)
+		)
+		(stroke
+			(width 0)
+			(type default)
+		)
+	)
+	(wire
+		(pts
 			(xy 129.54 66.04) (xy 130.81 66.04)
 		)
@@
 	)
 	(label "FLOW_OUT"
-		(at 54.61 54.61 180)
+		(at 54.61 57.15 180)
 		(effects
 			(font
@@
 			)
 			(justify right bottom)
-		)
-	)
-	(label "+12V"
-		(at 40.64 48.26 0)
-		(effects
-			(font
-				(size 1.27 1.27)
-			)
-			(justify left bottom)
 		)
 	)
@@
 		(dnp no)
 		(fields_autoplaced yes)
-		(property "Reference" "#PWR044"
+		(property "Reference" "#PWR042"
 			(at 119.38 66.04 0)
 			(effects
@@
 			(project "PTN-PumpControlBoard"
 				(path "/591f46f8-eb1d-42dc-a4cb-8182eac4ef58/72cbb232-97a0-4b9b-a6b0-3f04462a78a5"
-					(reference "#PWR044")
+					(reference "#PWR042")
 					(unit 1)
 				)
@@
 		(dnp no)
 		(fields_autoplaced yes)
-		(property "Reference" "#PWR045"
+		(property "Reference" "#PWR041"
 			(at 101.6 64.77 0)
 			(effects
@@
 			(project "PTN-PumpControlBoard"
 				(path "/591f46f8-eb1d-42dc-a4cb-8182eac4ef58/72cbb232-97a0-4b9b-a6b0-3f04462a78a5"
-					(reference "#PWR045")
+					(reference "#PWR041")
 					(unit 1)
 				)
@@
 		(on_board yes)
 		(dnp no)
-		(property "Reference" "R27"
+		(property "Reference" "R14"
 			(at 123.6981 68.58 90)
 			(effects
@@
 			(project "PTN-PumpControlBoard"
 				(path "/591f46f8-eb1d-42dc-a4cb-8182eac4ef58/72cbb232-97a0-4b9b-a6b0-3f04462a78a5"
-					(reference "R27")
+					(reference "R14")
 					(unit 1)
 				)
@@
 		(dnp no)
 		(fields_autoplaced yes)
-		(property "Reference" "FLOW2"
+		(property "Reference" "FLOW1"
 			(at 66.04 55.8799 0)
 			(effects
@@
 			(project "PTN-PumpControlBoard"
 				(path "/591f46f8-eb1d-42dc-a4cb-8182eac4ef58/72cbb232-97a0-4b9b-a6b0-3f04462a78a5"
-					(reference "FLOW2")
+					(reference "FLOW1")
 					(unit 1)
 				)
@@
 		(dnp no)
 		(fields_autoplaced yes)
-		(property "Reference" "U5"
+		(property "Reference" "U6"
 			(at 134.62 44.3798 0)
 			(effects
@@
 			(project "PTN-PumpControlBoard"
 				(path "/591f46f8-eb1d-42dc-a4cb-8182eac4ef58/72cbb232-97a0-4b9b-a6b0-3f04462a78a5"
-					(reference "U5")
+					(reference "U6")
 					(unit 1)
 				)
@@
 		(on_board yes)
 		(dnp no)
-		(property "Reference" "R28"
+		(property "Reference" "R13"
 			(at 107.1881 55.88 90)
 			(effects
@@
 			(project "PTN-PumpControlBoard"
 				(path "/591f46f8-eb1d-42dc-a4cb-8182eac4ef58/72cbb232-97a0-4b9b-a6b0-3f04462a78a5"
-					(reference "R28")
+					(reference "R13")
+					(unit 1)
+				)
+			)
+		)
+	)
+	(symbol
+		(lib_id "power:+12V")
+		(at 53.34 48.26 0)
+		(unit 1)
+		(exclude_from_sim no)
+		(in_bom yes)
+		(on_board yes)
+		(dnp no)
+		(fields_autoplaced yes)
+		(property "Reference" "#PWR040"
+			(at 53.34 52.07 0)
+			(effects
+				(font
+					(size 1.27 1.27)
+				)
+				(hide yes)
+			)
+		)
+		(property "Value" "+24V"
+			(at 53.34 43.18 0)
+			(effects
+				(font
+					(size 1.27 1.27)
+				)
+			)
+		)
+		(property "Footprint" ""
+			(at 53.34 48.26 0)
+			(effects
+				(font
+					(size 1.27 1.27)
+				)
+				(hide yes)
+			)
+		)
+		(property "Datasheet" ""
+			(at 53.34 48.26 0)
+			(effects
+				(font
+					(size 1.27 1.27)
+				)
+				(hide yes)
+			)
+		)
+		(property "Description" "Power symbol creates a global label with name \"+12V\""
+			(at 53.34 48.26 0)
+			(effects
+				(font
+					(size 1.27 1.27)
+				)
+				(hide yes)
+			)
+		)
+		(pin "1"
+		)
+		(instances
+			(project "PTN-PumpControlBoard"
+				(path "/591f46f8-eb1d-42dc-a4cb-8182eac4ef58/72cbb232-97a0-4b9b-a6b0-3f04462a78a5"
+					(reference "#PWR040")
 					(unit 1)
 				)
@@
 		(dnp no)
 		(fields_autoplaced yes)
-		(property "Reference" "#PWR037"
+		(property "Reference" "#PWR043"
 			(at 53.34 71.12 0)
 			(effects
@@
 			(project "PTN-PumpControlBoard"
 				(path "/591f46f8-eb1d-42dc-a4cb-8182eac4ef58/72cbb232-97a0-4b9b-a6b0-3f04462a78a5"
-					(reference "#PWR037")
+					(reference "#PWR043")
 					(unit 1)
 				)
@@
 		(dnp no)
 		(fields_autoplaced yes)
-		(property "Reference" "#PWR043"
+		(property "Reference" "#PWR039"
 			(at 119.38 45.72 0)
 			(effects
@@
 			(project "PTN-PumpControlBoard"
 				(path "/591f46f8-eb1d-42dc-a4cb-8182eac4ef58/72cbb232-97a0-4b9b-a6b0-3f04462a78a5"
-					(reference "#PWR043")
+					(reference "#PWR039")
 					(unit 1)
 				)

Commit message: added test points and headers, AGND and 12V not fully connected
Parts:
- added FL_OUT1, FL_TP1: Scope_TP, TestPoint:TestPoint_Keystone_5010-5014_Multipurpose, symbol Connector:TestPoint
Connections:
- net FLOW_OUT: now also FL_OUT1.1
- net FLOW_SEN: now also FL_TP1.1
Changed lines of the file:
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@@
+	)
+	(junction
+		(at 134.62 50.8)
+		(diameter 0)
+		(color 0 0 0 0)
 	)
 	(junction
@@
 	)
 	(junction
+		(at 113.03 48.26)
+		(diameter 0)
+		(color 0 0 0 0)
+	)
+	(junction
 		(at 114.3 53.34)
 		(diameter 0)
@@
 	(wire
 		(pts
+			(xy 134.62 50.8) (xy 137.16 50.8)
+		)
+		(stroke
+			(width 0)
+			(type default)
+		)
+	)
+	(wire
+		(pts
 			(xy 54.61 57.15) (xy 58.42 57.15)
 		)
@@
 	(wire
 		(pts
-			(xy 130.81 50.8) (xy 133.35 50.8)
+			(xy 130.81 50.8) (xy 134.62 50.8)
 		)
 		(stroke
@@
 	(wire
 		(pts
-			(xy 111.76 48.26) (xy 114.3 48.26)
+			(xy 109.22 48.26) (xy 113.03 48.26)
 		)
 		(stroke
@@
 	(wire
 		(pts
+			(xy 113.03 43.18) (xy 113.03 48.26)
+		)
+		(stroke
+			(width 0)
+			(type default)
+		)
+	)
+	(wire
+		(pts
 			(xy 129.54 66.04) (xy 130.81 66.04)
 		)
@@
 		(pts
 			(xy 129.54 50.8) (xy 130.81 50.8)
+		)
+		(stroke
+			(width 0)
+			(type default)
+		)
+	)
+	(wire
+		(pts
+			(xy 134.62 50.8) (xy 134.62 58.42)
+		)
+		(stroke
+			(width 0)
+			(type default)
+		)
+	)
+	(wire
+		(pts
+			(xy 113.03 48.26) (xy 114.3 48.26)
 		)
 		(stroke
@@
 	)
 	(label "FLOW_OUT"
-		(at 111.76 48.26 180)
+		(at 109.22 48.26 180)
 		(effects
 			(font
@@
 	(hierarchical_label "FLOW_SEN"
 		(shape output)
-		(at 133.35 50.8 0)
+		(at 137.16 50.8 0)
 		(effects
 			(font
@@
 	)
 	(symbol
+		(lib_id "Connector:TestPoint")
+		(at 113.03 43.18 90)
+		(unit 1)
+		(exclude_from_sim no)
+		(in_bom yes)
+		(on_board yes)
+		(dnp no)
+		(fields_autoplaced yes)
+		(property "Reference" "FL_OUT1"
+			(at 109.728 38.1 90)
+			(effects
+				(font
+					(size 1.27 1.27)
+				)
+			)
+		)
+		(property "Value" "Scope_TP"
+			(at 109.728 40.64 90)
+			(effects
+				(font
+					(size 1.27 1.27)
+				)
+			)
+		)
+		(property "Footprint" "TestPoint:TestPoint_Keystone_5010-5014_Multipurpose"
+			(at 113.03 38.1 0)
+			(effects
+				(font
+					(size 1.27 1.27)
+				)
+				(hide yes)
+			)
+		)
+		(property "Datasheet" "~"
+			(at 113.03 38.1 0)
+			(effects
+				(font
+					(size 1.27 1.27)
+				)
+				(hide yes)
+			)
+		)
+		(property "Description" "test point"
+			(at 113.03 43.18 0)
+			(effects
+				(font
+					(size 1.27 1.27)
+				)
+				(hide yes)
+			)
+		)
+		(pin "1"
+		)
+		(instances
+			(project "PTN-PumpControlBoard"
+				(path "/591f46f8-eb1d-42dc-a4cb-8182eac4ef58/72cbb232-97a0-4b9b-a6b0-3f04462a78a5"
+					(reference "FL_OUT1")
+					(unit 1)
+				)
+			)
+		)
+	)
+	(symbol
 		(lib_id "power:GND")
 		(at 119.38 59.69 0)
@@
 		(dnp no)
 		(fields_autoplaced yes)
-		(property "Reference" "#PWR042"
+		(property "Reference" "#PWR041"
 			(at 119.38 66.04 0)
 			(effects
@@
 			(project "PTN-PumpControlBoard"
 				(path "/591f46f8-eb1d-42dc-a4cb-8182eac4ef58/72cbb232-97a0-4b9b-a6b0-3f04462a78a5"
-					(reference "#PWR042")
+					(reference "#PWR041")
 					(unit 1)
 				)
@@
 		(dnp no)
 		(fields_autoplaced yes)
-		(property "Reference" "#PWR041"
+		(property "Reference" "#PWR039"
 			(at 101.6 64.77 0)
 			(effects
@@
 			(project "PTN-PumpControlBoard"
 				(path "/591f46f8-eb1d-42dc-a4cb-8182eac4ef58/72cbb232-97a0-4b9b-a6b0-3f04462a78a5"
-					(reference "#PWR041")
+					(reference "#PWR039")
 					(unit 1)
 				)
@@
 	)
 	(symbol
+		(lib_id "Connector:TestPoint")
+		(at 134.62 58.42 270)
+		(unit 1)
+		(exclude_from_sim no)
+		(in_bom yes)
+		(on_board yes)
+		(dnp no)
+		(fields_autoplaced yes)
+		(property "Reference" "FL_TP1"
+			(at 139.7 57.1499 90)
+			(effects
+				(font
+					(size 1.27 1.27)
+				)
+				(justify left)
+			)
+		)
+		(property "Value" "Scope_TP"
+			(at 139.7 59.6899 90)
+			(effects
+				(font
+					(size 1.27 1.27)
+				)
+				(justify left)
+			)
+		)
+		(property "Footprint" "TestPoint:TestPoint_Keystone_5010-5014_Multipurpose"
+			(at 134.62 63.5 0)
+			(effects
+				(font
+					(size 1.27 1.27)
+				)
+				(hide yes)
+			)
+		)
+		(property "Datasheet" "~"
+			(at 134.62 63.5 0)
+			(effects
+				(font
+					(size 1.27 1.27)
+				)
+				(hide yes)
+			)
+		)
+		(property "Description" "test point"
+			(at 134.62 58.42 0)
+			(effects
+				(font
+					(size 1.27 1.27)
+				)
+				(hide yes)
+			)
+		)
+		(pin "1"
+		)
+		(instances
+			(project "PTN-PumpControlBoard"
+				(path "/591f46f8-eb1d-42dc-a4cb-8182eac4ef58/72cbb232-97a0-4b9b-a6b0-3f04462a78a5"
+					(reference "FL_TP1")
+					(unit 1)
+				)
+			)
+		)
+	)
+	(symbol
 		(lib_id "power:+12V")
 		(at 53.34 48.26 0)
@@
 		(dnp no)
 		(fields_autoplaced yes)
-		(property "Reference" "#PWR040"
+		(property "Reference" "#PWR037"
 			(at 53.34 52.07 0)
 			(effects
@@
 			(project "PTN-PumpControlBoard"
 				(path "/591f46f8-eb1d-42dc-a4cb-8182eac4ef58/72cbb232-97a0-4b9b-a6b0-3f04462a78a5"
-					(reference "#PWR040")
+					(reference "#PWR037")
 					(unit 1)
 				)
@@
 		(dnp no)
 		(fields_autoplaced yes)
-		(property "Reference" "#PWR043"
+		(property "Reference" "#PWR038"
 			(at 53.34 71.12 0)
 			(effects
@@
 			(project "PTN-PumpControlBoard"
 				(path "/591f46f8-eb1d-42dc-a4cb-8182eac4ef58/72cbb232-97a0-4b9b-a6b0-3f04462a78a5"
-					(reference "#PWR043")
+					(reference "#PWR038")
 					(unit 1)
 				)
@@
 		(dnp no)
 		(fields_autoplaced yes)
-		(property "Reference" "#PWR039"
+		(property "Reference" "#PWR040"
 			(at 119.38 45.72 0)
 			(effects
@@
 			(project "PTN-PumpControlBoard"
 				(path "/591f46f8-eb1d-42dc-a4cb-8182eac4ef58/72cbb232-97a0-4b9b-a6b0-3f04462a78a5"
-					(reference "#PWR039")
-					(unit 1)
-				)
+					(reference "#PWR040")
+					(unit 1)
+				)

Commit message: Fixed fan schematic based on review feedback
Parts:
- removed FL_OUT1, FL_TP1: Scope_TP, TestPoint:TestPoint_Keystone_5010-5014_Multipurpose, symbol Connector:TestPoint
Connections:
- net FLOW_OUT: now also FLOW1.3 (Pin_3); no longer FLOW1.2 (Pin_2)
- net GND: now also FLOW1.2 (Pin_2); no longer FLOW1.3 (Pin_3)
Changed lines of the file:
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@@
-	)
-	(junction
-		(at 134.62 50.8)
-		(diameter 0)
-		(color 0 0 0 0)
 	)
 	(junction
@@
 	)
 	(junction
-		(at 113.03 48.26)
-		(diameter 0)
-		(color 0 0 0 0)
-	)
-	(junction
 		(at 114.3 53.34)
 		(diameter 0)
@@
 	(wire
 		(pts
-			(xy 134.62 50.8) (xy 137.16 50.8)
-		)
-		(stroke
-			(width 0)
-			(type default)
-		)
-	)
-	(wire
-		(pts
-			(xy 54.61 57.15) (xy 58.42 57.15)
+			(xy 130.81 50.8) (xy 137.16 50.8)
 		)
 		(stroke
@@
 	(wire
 		(pts
-			(xy 58.42 54.61) (xy 53.34 54.61)
-		)
-		(stroke
-			(width 0)
-			(type default)
-		)
-	)
-	(wire
-		(pts
-			(xy 130.81 50.8) (xy 134.62 50.8)
+			(xy 46.99 54.61) (xy 58.42 54.61)
 		)
 		(stroke
@@
 	(wire
 		(pts
-			(xy 109.22 48.26) (xy 113.03 48.26)
-		)
-		(stroke
-			(width 0)
-			(type default)
-		)
-	)
-	(wire
-		(pts
 			(xy 113.03 53.34) (xy 114.3 53.34)
 		)
@@
 	(wire
 		(pts
-			(xy 53.34 54.61) (xy 53.34 48.26)
-		)
-		(stroke
-			(width 0)
-			(type default)
-		)
-	)
-	(wire
-		(pts
-			(xy 113.03 43.18) (xy 113.03 48.26)
+			(xy 46.99 54.61) (xy 46.99 48.26)
+		)
+		(stroke
+			(width 0)
+			(type default)
+		)
+	)
+	(wire
+		(pts
+			(xy 46.99 57.15) (xy 58.42 57.15)
 		)
 		(stroke
@@
 	(wire
 		(pts
-			(xy 53.34 59.69) (xy 53.34 64.77)
+			(xy 46.99 57.15) (xy 46.99 62.23)
 		)
 		(stroke
@@
 	(wire
 		(pts
-			(xy 58.42 59.69) (xy 53.34 59.69)
-		)
-		(stroke
-			(width 0)
-			(type default)
-		)
-	)
-	(wire
-		(pts
 			(xy 129.54 50.8) (xy 130.81 50.8)
 		)
@@
 	(wire
 		(pts
-			(xy 134.62 50.8) (xy 134.62 58.42)
-		)
-		(stroke
-			(width 0)
-			(type default)
-		)
-	)
-	(wire
-		(pts
-			(xy 113.03 48.26) (xy 114.3 48.26)
+			(xy 109.22 48.26) (xy 114.3 48.26)
 		)
 		(stroke
@@
 	)
 	(label "FLOW_OUT"
-		(at 54.61 57.15 180)
+		(at 58.42 59.69 180)
 		(effects
 			(font
@@
 			)
 			(justify left)
-		)
-	)
-	(symbol
-		(lib_id "Connector:TestPoint")
-		(at 113.03 43.18 90)
-		(unit 1)
-		(exclude_from_sim no)
-		(in_bom yes)
-		(on_board yes)
-		(dnp no)
-		(fields_autoplaced yes)
-		(property "Reference" "FL_OUT1"
-			(at 109.728 38.1 90)
-			(effects
-				(font
-					(size 1.27 1.27)
-				)
-			)
-		)
-		(property "Value" "Scope_TP"
-			(at 109.728 40.64 90)
-			(effects
-				(font
-					(size 1.27 1.27)
-				)
-			)
-		)
-		(property "Footprint" "TestPoint:TestPoint_Keystone_5010-5014_Multipurpose"
-			(at 113.03 38.1 0)
-			(effects
-				(font
-					(size 1.27 1.27)
-				)
-				(hide yes)
-			)
-		)
-		(property "Datasheet" "~"
-			(at 113.03 38.1 0)
-			(effects
-				(font
-					(size 1.27 1.27)
-				)
-				(hide yes)
-			)
-		)
-		(property "Description" "test point"
-			(at 113.03 43.18 0)
-			(effects
-				(font
-					(size 1.27 1.27)
-				)
-				(hide yes)
-			)
-		)
-		(pin "1"
-		)
-		(instances
-			(project "PTN-PumpControlBoard"
-				(path "/591f46f8-eb1d-42dc-a4cb-8182eac4ef58/72cbb232-97a0-4b9b-a6b0-3f04462a78a5"
-					(reference "FL_OUT1")
-					(unit 1)
-				)
-			)
 		)
 	)
@@
 	)
 	(symbol
-		(lib_id "Connector:TestPoint")
-		(at 134.62 58.42 270)
-		(unit 1)
-		(exclude_from_sim no)
-		(in_bom yes)
-		(on_board yes)
-		(dnp no)
-		(fields_autoplaced yes)
-		(property "Reference" "FL_TP1"
-			(at 139.7 57.1499 90)
-			(effects
-				(font
-					(size 1.27 1.27)
-				)
-				(justify left)
-			)
-		)
-		(property "Value" "Scope_TP"
-			(at 139.7 59.6899 90)
-			(effects
-				(font
-					(size 1.27 1.27)
-				)
-				(justify left)
-			)
-		)
-		(property "Footprint" "TestPoint:TestPoint_Keystone_5010-5014_Multipurpose"
-			(at 134.62 63.5 0)
-			(effects
-				(font
-					(size 1.27 1.27)
-				)
-				(hide yes)
-			)
-		)
-		(property "Datasheet" "~"
-			(at 134.62 63.5 0)
-			(effects
-				(font
-					(size 1.27 1.27)
-				)
-				(hide yes)
-			)
-		)
-		(property "Description" "test point"
-			(at 134.62 58.42 0)
-			(effects
-				(font
-					(size 1.27 1.27)
-				)
-				(hide yes)
-			)
-		)
-		(pin "1"
-		)
-		(instances
-			(project "PTN-PumpControlBoard"
-				(path "/591f46f8-eb1d-42dc-a4cb-8182eac4ef58/72cbb232-97a0-4b9b-a6b0-3f04462a78a5"
-					(reference "FL_TP1")
-					(unit 1)
-				)
-			)
-		)
-	)
-	(symbol
 		(lib_id "power:+12V")
-		(at 53.34 48.26 0)
+		(at 46.99 48.26 0)
 		(unit 1)
 		(exclude_from_sim no)
@@
 		(fields_autoplaced yes)
 		(property "Reference" "#PWR037"
-			(at 53.34 52.07 0)
+			(at 46.99 52.07 0)
 			(effects
 				(font
@@
 		)
 		(property "Value" "+24V"
-			(at 53.34 43.18 0)
+			(at 46.99 43.18 0)
 			(effects
 				(font
@@
 		)
 		(property "Footprint" ""
-			(at 53.34 48.26 0)
+			(at 46.99 48.26 0)
 			(effects
 				(font
@@
 		)
 		(property "Datasheet" ""
-			(at 53.34 48.26 0)
+			(at 46.99 48.26 0)
 			(effects
 				(font
@@
 		)
 		(property "Description" "Power symbol creates a global label with name \"+12V\""
-			(at 53.34 48.26 0)
+			(at 46.99 48.26 0)
 			(effects
 				(font
@@
 	(symbol
 		(lib_id "power:GND")
-		(at 53.34 64.77 0)
+		(at 46.99 62.23 0)
 		(unit 1)
 		(exclude_from_sim no)
@@
 		(fields_autoplaced yes)
 		(property "Reference" "#PWR038"
-			(at 53.34 71.12 0)
+			(at 46.99 68.58 0)
 			(effects
 				(font
@@
 		)
 		(property "Value" "GND"
-			(at 53.34 69.85 0)
+			(at 46.99 67.31 0)
 			(effects
 				(font
@@
 		)
 		(property "Footprint" ""
-			(at 53.34 64.77 0)
+			(at 46.99 62.23 0)
 			(effects
 				(font
@@
 		)
 		(property "Datasheet" ""
-			(at 53.34 64.77 0)
+			(at 46.99 62.23 0)
 			(effects
 				(font
@@
 		)
 		(property "Description" "Power symbol creates a global label with name \"GND\" , ground"
-			(at 53.34 64.77 0)
-			(effects
-				(font
+			(at 46.99 62.23 0)
+			(effects
+				(font

Commit message: updated schematic with low pass for temp sensors and new resistor footprint
Parts:
- R13, R14: footprint Resistor_SMD:R_0805_2012Metric -> Resistor_SMD:R_0603_1608Metric
Changed lines of the file:
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@@
 			)
 		)
-		(property "Footprint" "Resistor_SMD:R_0805_2012Metric"
+		(property "Footprint" "Resistor_SMD:R_0603_1608Metric"
 			(at 125.476 67.056 90)
 			(effects
@@
 			)
 		)
-		(property "Footprint" "Resistor_SMD:R_0805_2012Metric"
+		(property "Footprint" "Resistor_SMD:R_0603_1608Metric"
 			(at 108.966 54.356 90)
 			(effects

Commit message: fixed all review notes for schematic
Parts:
- removed R13: 100, Resistor_SMD:R_0603_1608Metric, symbol Device:R_US
- removed R14: 1.4k, Resistor_SMD:R_0603_1608Metric, symbol Device:R_US
- removed U6: TLV6001DCK, Package_TO_SOT_SMD:SOT-353_SC-70-5, symbol Amplifier_Operational:TLV6001DCK
- added C13: 1uF, Capacitor_SMD:C_0805_2012Metric, symbol Device:C_Small
- added C14: 15uF, Capacitor_SMD:C_0805_2012Metric, symbol Device:C_Small
- added C15, C16: .1uF, Capacitor_SMD:C_0805_2012Metric, symbol Device:C_Small
- added IC3: TLV9002QDRQ1, OpAmp:SOIC127P600X175-8N, symbol OpAmp:TLV9002QDRQ1
- added PS1: TSR_1-24120SM, TSR_1-24120SM:TSR124120SM, symbol TSR_1-24120SM:TSR_1-24120SM
- added Q3: NMOS, UTSVT_Power:BUK7M1780EX, symbol Simulation_SPICE:NMOS
- added R25, R28, R30: 0, Resistor_SMD:R_0603_1608Metric, symbol Device:R_US
- added R26: 10k, Resistor_SMD:R_0603_1608Metric, symbol Device:R_US
- added R27: 15k, Resistor_SMD:R_0603_1608Metric, symbol Device:R_US
- added R29: 1k, Resistor_SMD:R_0603_1608Metric, symbol Device:R_US
- added T_TP4: Pad_TP, UTSVT_Special:TestPoint_HEX_3mmID, symbol Connector:TestPoint
- added U5: TLV9002QDRQ1, OpAmp:SOIC127P600X175-8N, symbol Amplifier_Operational:OP249GS
- FLOW1: Notes jst xhp 3 connector for flowrate sensor -> VG-FLOW-0_5-BSP Brass 1/2" Hall-Effect Flow Sensor with BSP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
Connections:
- net +24V: now also PS1.1 (+VIN); no longer FLOW1.1 (Pin_1)
- net +3.3V: now also C16.1, IC3.8 (V+), R26.2, U5.8 (V+)
- net FLOW_OUT: now also R25.1
- net FLOW_SEN: now also C14.1, R29.2
- net GND: now also C13.2, C14.2, C15.2, C16.2, IC3.4 (V-), PS1.7 (GND_1), PS1.9 (GND_2), Q3.3 (S), R30.2
- new net: Q3.1 (D), R26.1, R27.1
- new net: C15.1, U5.4 (V-)
- new net: Q3.2 (G), R25.2
- new net +12V: FLOW1.1 (Pin_1), PS1.5 (+VOUT)
- new net IN4+: C13.1, IC3.3 (IN1+), R27.2, U5.3 (+)
- new net IN4-: IC3.2 (IN1-), R28.2, R30.1, U5.2 (-)
- new net OUT4: IC3.1 (OUT1), R28.1, R29.1, T_TP4.1, U5.1
- no-connect marks 0 -> 8
Other:
- note added: "actual op amp footprint"
- note added: "buck to 12V"
- note added: "is it better to use standard buck that's on psom?"
- note added: "reverse logic in SW"
