File: FlowrateSensor.kicad_sch (KiCad schematic)
At the start: 16 parts, among them IC3 TLV9002QDRQ1, Q3 BUK7M27-80EX, U5 TLV9002QDRQ1

Commit message: review notes
Parts:
- removed C13: 1uF, Capacitor_SMD:C_0805_2012Metric, symbol Device:C_Small
- removed C14: 15uF, Capacitor_SMD:C_0805_2012Metric, symbol Device:C_Small
- removed C15, C16: .1uF, Capacitor_SMD:C_0805_2012Metric, symbol Device:C_Small
- removed IC3: TLV9002QDRQ1, OpAmp:SOIC127P600X175-8N, symbol OpAmp:TLV9002QDRQ1
- removed R27: 15k, Resistor_SMD:R_0603_1608Metric, symbol Device:R_US
- removed R28, R30: 0, Resistor_SMD:R_0603_1608Metric, symbol Device:R_US
- removed R29: 1k, Resistor_SMD:R_0603_1608Metric, symbol Device:R_US
- removed T_TP4: Pad_TP, UTSVT_Special:TestPoint_HEX_3mmID, symbol Connector:TestPoint
- removed U5: TLV9002QDRQ1, OpAmp:SOIC127P600X175-8N, symbol Amplifier_Operational:OP249GS
Connections:
- net FLOW_SEN: now also Q3.5 (D), R26.1
- no-connect marks 8 -> 2
Other:
- note added: "- psom buck - add bypass connector - test points"
- note added: "bypass caps"
- note added: "check if psom pin is timer in/input capture"
- note added: "find one with external inductor"
- note added: "is it better to use standard buck that's on psom? - yes"
- note added: "switch to pmos"
- note removed: "actual op amp footprint"
- note removed: "is it better to use standard buck that's on psom?"

Commit message: schematic changes before switching submodules
Parts:
- removed PS1: TSR_1-24120SM, TSR_1-24120SM:TSR124120SM, symbol TSR_1-24120SM:TSR_1-24120SM
- added C18, C23, C34, C35: 10uF, Capacitor_SMD:C_0805_2012Metric_Pad1.18x1.45mm_HandSolder, symbol Device:C
- added C19: 1uF, Capacitor_SMD:C_0603_1608Metric_Pad1.08x0.95mm_HandSolder, symbol Device:C
- added C20: 10nF, Capacitor_SMD:C_0603_1608Metric_Pad1.08x0.95mm_HandSolder, symbol Device:C
- added C21: 3.3nF, Capacitor_SMD:C_0603_1608Metric_Pad1.08x0.95mm_HandSolder, symbol Device:C
- added C22: 0.1uF, Capacitor_SMD:C_0603_1608Metric_Pad1.08x0.95mm_HandSolder, symbol Device:C
- added D11: MBR230S1F, Diode_SMD:D_SOD-123F, symbol Device:D_Schottky
- added L1: 100uH, Inductor_SMD:L_Coilcraft_MSS1246-XXX, symbol Device:L
- added Q6: BUK6Y55-80PX, BUK6Y55-80PX:PHPT61002NYCLHX, symbol BUK6Y55-80PX:BUK6Y55-80PX
- added R27: 16k, Resistor_SMD:R_0603_1608Metric_Pad0.98x0.95mm_HandSolder, symbol Device:R
- added R29: ROSC, Resistor_SMD:R_0603_1608Metric_Pad0.98x0.95mm_HandSolder, symbol Device:R
- added R35: 100k, Resistor_SMD:R_0603_1608Metric, symbol Device:R_US
- added U6: TPS5405DR, UTSVT_Power:TPS5405DR, symbol utsvt_power:TPS5405DR
- Q3: value BUK7M27-80EX -> PSMN8R5-40MSDX
Connections:
- net +24V: now also C18.1, C19.1, U6.2 (VIN)
- net GND: now also C18.2, C19.2, C20.2, C23.2, C34.2, C35.2, D11.2 (A), R27.2, R29.2, R35.2, U6.7 (GND)
- net at Q3.4 (G), R25.2: now also R35.1
- new net: C22.1, U6.1 (BOOT)
- new net: C22.2, D11.1 (K), L1.1, U6.8 (LX)
- new net: C20.1, U6.4 (SS)
- new net: C21.1, U6.6 (COMP)
- new net: C21.2, R27.1
- new net +5V_BUCK: C23.1, C34.1, C35.1, L1.2, U6.5 (VSENSE)
- new net ROSC: R29.1, U6.3 (ROSC)
- no-connect marks 2 -> 0
Other:
- note added: "Cout > 28.8uF -> 30uF For 30uF, ESR < 120mΩ"
- note added: "DNP for 120 kHz switching frequency"
- note added: "L: 92uH -> 100uH ΔIl: 0.33A DC load: 1.2A Peak current: 1.53A"
- note added: "Ripple current: 487mA (243.5 mA per cap) Ripple voltage: 125mV"
- note added: "Slow start time: (10nF * 0.8v)/2uA = 4ms"
- note added: "Vin: 6.5v to 28v Vout: 4.85v to 5.15v"
- note added: "chat gave me these"
- note added: "i fucking hate math"
- note added: "pmos circuitry felt unnecessary, I'm just gonna invert in sw"
- note removed: "buck to 12V"
- note removed: "bypass caps"
- note removed: "find one with external inductor"
- note removed: "is it better to use standard buck that's on psom? - yes"
- note removed: "reverse logic in SW"
- note removed: "switch to pmos"
- moved on the sheet: FLOW1, R25, R26

Commit message: fixed submodule, schematic basically done
Parts:
- removed Q6: BUK6Y55-80PX, BUK6Y55-80PX:PHPT61002NYCLHX, symbol BUK6Y55-80PX:BUK6Y55-80PX
- added +5V: Pad_TP, UTSVT_Special:TestPoint_HEX_3mmID, symbol Connector:TestPoint
- added 5V_IN: Conn_01x02, UTSVT_Connectors:Molex_Nano-Fit_105309-xx02_1x02_P2.50mm_Vertical, symbol Connector_Generic:Conn_01x02
- added R30: 0, Resistor_SMD:R_0603_1608Metric, symbol Device:R_US
Connections:
- net +5V_BUCK is gone; now on net +5V: C23.1, C34.1, C35.1, L1.2, U6.5 (VSENSE)
- net +24V: now also R30.1; no longer C19.1, U6.2 (VIN)
- net GND: now also 5V_IN.2 (Pin_2)
- net +12V renamed +5V
- net +5V: now also +5V.1, 5V_IN.1 (Pin_1)
- new net: C19.1, R30.2, U6.2 (VIN)
Other:
- note added: "DNP RESISTOR IF BUCK DOESN'T WORK (USE EXTERNAL SUPPLY)"
- note added: "ravi fucking hates math"
- note removed: "- psom buck - add bypass connector - test points"
- note removed: "i fucking hate math"
- moved on the sheet: C18, C19, C20, C21, C22, C23, C34, C35, D11, L1, R27, R29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

Commit message: finalized schematic (pls be the last time)
Parts:
- renumbered +5V to +5V1, 5V_IN to 5V_IN1, C18 to C13, C19 to C14, C20 to C15, C21 to C16, C22 to C17, C23 to C18, C34 to C19, C35 to C20, R25 to R27, R35 to R28, R26 to R29, R27 to R31, R29 to R32
Changed lines of the file:
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@@
 		(dnp no)
 		(fields_autoplaced yes)
-		(property "Reference" "5V_IN"
+		(property "Reference" "5V_IN1"
 			(at 210.82 73.6599 0)
 			(effects
@@
 			(project ""
 				(path "/591f46f8-eb1d-42dc-a4cb-8182eac4ef58/72cbb232-97a0-4b9b-a6b0-3f04462a78a5"
-					(reference "5V_IN")
+					(reference "5V_IN1")
 					(unit 1)
 				)
@@
 		(on_board yes)
 		(dnp no)
-		(property "Reference" "C22"
+		(property "Reference" "C17"
 			(at 136.3472 101.7016 0)
 			(effects
@@
 			(project "PTN-PumpControlBoard"
 				(path "/591f46f8-eb1d-42dc-a4cb-8182eac4ef58/72cbb232-97a0-4b9b-a6b0-3f04462a78a5"
-					(reference "C22")
+					(reference "C17")
 					(unit 1)
 				)
@@
 		(on_board yes)
 		(dnp no)
-		(property "Reference" "C20"
+		(property "Reference" "C15"
 			(at 70.3072 111.8616 0)
 			(effects
@@
 			(project "PTN-PumpControlBoard"
 				(path "/591f46f8-eb1d-42dc-a4cb-8182eac4ef58/72cbb232-97a0-4b9b-a6b0-3f04462a78a5"
-					(reference "C20")
+					(reference "C15")
 					(unit 1)
 				)
@@
 		(dnp no)
 		(fields_autoplaced yes)
-		(property "Reference" "R26"
+		(property "Reference" "R29"
 			(at 129.54 29.2099 0)
 			(effects
@@
 			(project "PTN-PumpControlBoard"
 				(path "/591f46f8-eb1d-42dc-a4cb-8182eac4ef58/72cbb232-97a0-4b9b-a6b0-3f04462a78a5"
-					(reference "R26")
+					(reference "R29")
 					(unit 1)
 				)
@@
 		(on_board yes)
 		(dnp no)
-		(property "Reference" "C23"
+		(property "Reference" "C18"
 			(at 154.1272 113.1316 0)
 			(effects
@@
 			(project "PTN-PumpControlBoard"
 				(path "/591f46f8-eb1d-42dc-a4cb-8182eac4ef58/72cbb232-97a0-4b9b-a6b0-3f04462a78a5"
-					(reference "C23")
+					(reference "C18")
 					(unit 1)
 				)
@@
 		(dnp no)
 		(fields_autoplaced yes)
-		(property "Reference" "+5V"
+		(property "Reference" "+5V1"
 			(at 209.55 95.2499 90)
 			(effects
@@
 			(project "PTN-PumpControlBoard"
 				(path "/591f46f8-eb1d-42dc-a4cb-8182eac4ef58/72cbb232-97a0-4b9b-a6b0-3f04462a78a5"
-					(reference "+5V")
+					(reference "+5V1")
 					(unit 1)
 				)
@@
 		(on_board yes)
 		(dnp yes)
-		(property "Reference" "R29"
+		(property "Reference" "R32"
 			(at 93.218 133.4516 0)
 			(effects
@@
 			(project "PTN-PumpControlBoard"
 				(path "/591f46f8-eb1d-42dc-a4cb-8182eac4ef58/72cbb232-97a0-4b9b-a6b0-3f04462a78a5"
-					(reference "R29")
+					(reference "R32")
 					(unit 1)
 				)
@@
 		(on_board yes)
 		(dnp no)
-		(property "Reference" "C21"
+		(property "Reference" "C16"
 			(at 79.1972 118.2116 0)
 			(effects
@@
 			(project "PTN-PumpControlBoard"
 				(path "/591f46f8-eb1d-42dc-a4cb-8182eac4ef58/72cbb232-97a0-4b9b-a6b0-3f04462a78a5"
-					(reference "C21")
+					(reference "C16")
 					(unit 1)
 				)
@@
 		(on_board yes)
 		(dnp no)
-		(property "Reference" "R25"
+		(property "Reference" "R27"
 			(at 115.0619 40.64 90)
 			(effects
@@
 			(project "PTN-PumpControlBoard"
 				(path "/591f46f8-eb1d-42dc-a4cb-8182eac4ef58/72cbb232-97a0-4b9b-a6b0-3f04462a78a5"
-					(reference "R25")
+					(reference "R27")
 					(unit 1)
 				)
@@
 		(on_board yes)
 		(dnp no)
-		(property "Reference" "C18"
+		(property "Reference" "C13"
 			(at 57.6072 101.7016 0)
 			(effects
@@
 			(project "PTN-PumpControlBoard"
 				(path "/591f46f8-eb1d-42dc-a4cb-8182eac4ef58/72cbb232-97a0-4b9b-a6b0-3f04462a78a5"
-					(reference "C18")
+					(reference "C13")
 					(unit 1)
 				)
@@
 		(on_board yes)
 		(dnp no)
-		(property "Reference" "C35"
+		(property "Reference" "C20"
 			(at 176.9872 113.1316 0)
 			(effects
@@
 			(project "PTN-PumpControlBoard"
 				(path "/591f46f8-eb1d-42dc-a4cb-8182eac4ef58/72cbb232-97a0-4b9b-a6b0-3f04462a78a5"
-					(reference "C35")
+					(reference "C20")
 					(unit 1)
 				)
@@
 		(on_board yes)
 		(dnp no)
-		(property "Reference" "R27"
+		(property "Reference" "R31"
 			(at 77.978 128.3716 0)
 			(effects
@@
 			(project "PTN-PumpControlBoard"
 				(path "/591f46f8-eb1d-42dc-a4cb-8182eac4ef58/72cbb232-97a0-4b9b-a6b0-3f04462a78a5"
-					(reference "R27")
+					(reference "R31")
 					(unit 1)
 				)
@@
 		(on_board yes)
 		(dnp no)
-		(property "Reference" "C34"
+		(property "Reference" "C19"
 			(at 165.5572 113.1316 0)
 			(effects
@@
 			(project "PTN-PumpControlBoard"
 				(path "/591f46f8-eb1d-42dc-a4cb-8182eac4ef58/72cbb232-97a0-4b9b-a6b0-3f04462a78a5"
-					(reference "C34")
+					(reference "C19")
 					(unit 1)
 				)
@@
 		(on_board yes)
 		(dnp no)
-		(property "Reference" "R35"
+		(property "Reference" "R28"
 			(at 120.65 46.9899 0)
 			(effects
@@
 			(project "PTN-PumpControlBoard"
 				(path "/591f46f8-eb1d-42dc-a4cb-8182eac4ef58/72cbb232-97a0-4b9b-a6b0-3f04462a78a5"
-					(reference "R35")
+					(reference "R28")
 					(unit 1)
 				)
@@
 		(on_board yes)
 		(dnp no)
-		(property "Reference" "C19"
+		(property "Reference" "C14"
 			(at 67.7672 101.7016 0)
 			(effects
@@
 			(project "PTN-PumpControlBoard"
 				(path "/591f46f8-eb1d-42dc-a4cb-8182eac4ef58/72cbb232-97a0-4b9b-a6b0-3f04462a78a5"
-					(reference "C19")
-					(unit 1)
-				)
+					(reference "C14")
+					(unit 1)
+				)

Commit message: datasheets disappeared for some reason
Other:
- note removed: "check if psom pin is timer in/input capture"
Changed lines of the file:
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@@
-		)
-	)
-	(text "check if psom pin is timer in/input capture"
-		(exclude_from_sim no)
-		(at 182.626 41.91 0)
-		(effects
-			(font
-				(size 1.27 1.27)
-			)
 		)
 	)
@@
 		)
 	)
-	(text_box "CONTINGENCY PLANS"
+	(text_box "TESTING CIRCUITRY"
 		(exclude_from_sim no)
-		(at 205.74 102.235 0)
-		(size 22.86 3.81)
+		(at 208.28 102.235 0)
+		(size 20.32 3.81)
 		(margins 0.9525 0.9525 0.9525 0.9525)
 		(stroke

Commit message: fixed header
Parts:
- removed Q3: PSMN8R5-40MSDX, Package_TO_SOT_SMD:LFPAK33, symbol Transistor_FET:BUK7M27-80EX
- removed R29: 10k, Resistor_SMD:R_0603_1608Metric, symbol Device:R_US
- added Q7: PMOS, symbol Simulation_SPICE:PMOS
- added Q8: BUK6M61-60PX, BUK6M61-60PX:BUK9M34100EX, symbol BUK6M61-60PX:BUK6M61-60PX
- R27: value 0 -> 100
Connections:
- net +3.3V: now also Q7.3 (S), Q8.1 (S_1), Q8.2 (S_2), Q8.3 (S_3)
- net FLOW_SEN: now also Q7.1 (D), Q8.10 (D_6), Q8.11 (D_7), Q8.5 (D_1), Q8.6 (D_2), Q8.7 (D_3), Q8.8 (D_4), Q8.9 (D_5)
- net F_GATE: now reaches R27.2, R28.1
- net F_GATE: now also Q7.2 (G), Q8.4 (G)
Other:
- note added: "real nmos symbol with correct footprint"
- note added: "symbol for schematic clarity not populated on board"
- note removed: "pmos circuitry felt unnecessary, I'm just gonna invert in sw"
