File: PowerProtection.kicad_sch (KiCad schematic)
At the start: 28 parts, among them J5 Conn_01x02, Q4 PSMN8R5-40MSDX, U1 LM76202QPWPRQ1, U5 LM74501-Q1

Commit message: finalized schematic (pls be the last time)
Parts:
- removed C13: 220n, Capacitor_SMD:C_0603_1608Metric, symbol Device:C
- removed C14: 22n, Capacitor_SMD:C_0603_1608Metric, symbol Device:C
- removed C15: 10u, Capacitor_SMD:C_0603_1608Metric, symbol Device:C
- removed C16, C17: 0.1u, Capacitor_SMD:C_0603_1608Metric, symbol Device:C
- removed D9: BZT52-B12-QX, UTSVT_Passives:BZT52B12QX, symbol Device:D_Zener
- removed J5: Conn_01x02, UTSVT_Connectors:Molex_Nano-Fit_105309-xx02_1x02_P2.50mm_Vertical, symbol Connector_Generic:Conn_01x02
- removed LVGND_TP1: TestPoint, UTSVT_Special:TestPoint_HEX_3mmID, symbol Connector:TestPoint
- removed Q4: PSMN8R5-40MSDX, UTSVT_Power:BUK7M1780EX, symbol UTSVT_Power:PSMN8R5-40MSDX
- removed R28: 0, Resistor_SMD:R_0603_1608Metric, symbol Device:R_US
- removed U5: LM74501-Q1, UTSVT_ICs:LM74501QDDFRQ1, symbol UTSVT_ICs:LM74501-Q1
- renumbered C24 to C21, C25 to C22, C26 to C23, C27 to C24, C28 to C25, R43 to R37, R41 to R38, R38 to R39, R39 to R40, R40 to R41, R44 to R43, R46 to R44
Connections:
- no-connect marks 4 -> 2
Other:
- note removed: "24V Input Bypass Cap"

Commit message: changed rpp circuit to match vcu
Parts:
- removed C25: 10uF, Capacitor_SMD:C_0805_2012Metric_Pad1.18x1.45mm_HandSolder, symbol Device:C
- removed D12: TVS, Diode_SMD:D_SOD-323_HandSoldering, symbol Diode:SD12_SOD323
- removed D13: TVS, Diode_SMD:D_SOD-123F, symbol Device:D_Zener
- removed R37: 24m, Resistor_SMD:R_0603_1608Metric_Pad0.98x0.95mm_HandSolder, symbol Device:R
- removed R38, R43, R44: 10k, Resistor_SMD:R_0603_1608Metric_Pad0.98x0.95mm_HandSolder, symbol Device:R
- removed R39: 45.3k, Resistor_SMD:R_0603_1608Metric_Pad0.98x0.95mm_HandSolder, symbol Device:R
- removed R40: 590, Resistor_SMD:R_0603_1608Metric_Pad0.98x0.95mm_HandSolder, symbol Device:R
- removed R41: 2.1k, Resistor_SMD:R_0603_1608Metric_Pad0.98x0.95mm_HandSolder, symbol Device:R
- removed R42: 402k, Resistor_SMD:R_0603_1608Metric_Pad0.98x0.95mm_HandSolder, symbol Device:R
- removed R45: 100k, Resistor_SMD:R_0603_1608Metric_Pad0.98x0.95mm_HandSolder, symbol Device:R
- removed U1: LM76202QPWPRQ1, UTSVT_Power:LM76202QPWPRQ1, symbol utsvt_power:LM76202QPWPRQ1
- added IC3: LM74502HDDFR, LM74502HDDFR:SOT65P280X110-8N, symbol UTSVT_ICs:LM74502HDDFR
- added J6: Conn_01x02, UTSVT_Connectors:Molex_Nano-Fit_105309-xx02_1x02_P2.50mm_Vertical, symbol Connector_Generic:Conn_01x02
- added Q4: PSMN8R5-40MSDX, PSMN8R5-40MSDX:BUK7M1780EX, symbol UTSVT_Power:PSMN8R5-40MSDX
- added R37: 10k, Resistor_SMD:R_0603_1608Metric, symbol Device:R_US
- added R38: 200k, Resistor_SMD:R_0603_1608Metric, symbol Device:R_US
- added R39: 8k, Resistor_SMD:R_0603_1608Metric, symbol Device:R_US
- added Z1: SMAF4749A-TP, DO-221AC-2:SODFL5026X125N, symbol UTSVT_Power:SMAF4749A-TP
- C21: value 10uF -> 22n; footprint Capacitor_SMD:C_0805_2012Metric_Pad1.18x1.45mm_HandSolder -> Capacitor_SMD:C_0603_1608Metric; P/N GRM21BR61H106KE43K -> (none)
- C22: value 1uF -> 220u; footprint Capacitor_SMD:C_0603_1608Metric_Pad1.08x0.95mm_HandSolder -> Capacitor_SMD:C_0603_1608Metric; P/N MLASU168SB5105KTNA01 -> (none)
- C23: value 100nF -> 1u; footprint Capacitor_SMD:C_0603_1608Metric_Pad1.08x0.95mm_HandSolder -> Capacitor_SMD:C_0603_1608Metric; P/N MLASH168SB7104KTNA01 -> (none)
- C24: value 1uF -> 220n; footprint Capacitor_SMD:C_0603_1608Metric_Pad1.08x0.95mm_HandSolder -> Capacitor_SMD:C_0603_1608Metric; P/N MLASU168SB5105KTNA01 -> (none)
Connections:
- net +24V: now also C22.1, IC3.8 (SRC), Q4.10 (D_6), Q4.11 (D_7), Q4.5 (D_1), Q4.6 (D_2), Q4.7 (D_3), Q4.8 (D_4), Q4.9 (D_5); no longer C24.1
- net GND: now also C23.1, IC3.2 (GND), J6.1 (Pin_1), R39.2, Z1.2 (A); no longer C21.2, C24.2
- net 24V_Ext: no longer names the net of C21.1
- net 24V_Ext: now also IC3.6 (GATE), Q4.4 (G); no longer C22.1
- net RTN renamed RPP_EN
- net RPP_EN: now also C24.1, IC3.1 (EN/UVLO), IC3.5 (VS), R37.2, Z1.1 (K)
- new net: C24.2, IC3.4 (VCAP)
- new net: IC3.7 (OV), R38.2, R39.1
- new net +24V_IN: C21.2, Q4.1 (S_1), Q4.2 (S_2), Q4.3 (S_3), R37.1
- new net +3V3: J6.2 (Pin_2)
- new net LV+: R38.1
- no-connect marks 2 -> 0
Other:
- note added: "3v3 injector"
- note added: "RPP PROTECTION (taken from vcu)"
- note removed: "20.88 ms ramp time"
- note removed: "Current Monitoring"
- note removed: "DNP until validated"
- note removed: "Functional Mode Selection"
- note removed: "ILim(A) = 12/R(k) 1.2A = 12/10kΩ"
- note removed: "OVP set to 27v for buck max voltage of 28v"
- note removed: "Overcurrent Protection"
- note removed: "Pullups"
- note removed: "RTN!=GND Conecting GND to RTN turns off RPP!"
- note removed: "SHDN has weak internal pullup - pulled up to MCU voltage after initial power on"
- note removed: "Set to circuit breaker (latchoff) Use 0 ohm resistor for auto-retry (540ms)"
- note removed: "Typical gain: 78.28 uA/A Vout @ 1.3A = 2.407v R(imon) = 23.7 mΩ"
- note removed: "Under/Overvoltage Protection"

Commit message: everything done other than the routing for logic analyzers
Parts:
- renumbered J6 to 3.3V_In1
Connections:
- net LV+ is gone; now on net +24V_IN: R38.1
- net +3V3 renamed +3.3V
Changed lines of the file:
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@@
-	(wire
-		(pts
-			(xy 86.36 66.04) (xy 86.36 66.675)
-		)
-		(stroke
-			(width 0)
-			(type default)
-		)
-	)
 	(wire
 		(pts
@@
 		)
 	)
-	(label "LV+"
-		(at 86.36 66.04 0)
-		(effects
-			(font
-				(size 1.27 1.27)
-			)
-			(justify left bottom)
-		)
-	)
 	(symbol
 		(lib_id "UTSVT_Power:PSMN8R5-40MSDX")
@@
 			)
 		)
-		(property "Value" "+3V3"
+		(property "Value" "+3.3V"
 			(at 140.97 27.94 0)
 			(effects
@@
 	)
 	(symbol
+		(lib_id "power:+12V")
+		(at 86.36 66.675 0)
+		(unit 1)
+		(exclude_from_sim no)
+		(in_bom yes)
+		(on_board yes)
+		(dnp no)
+		(property "Reference" "#PWR071"
+			(at 86.36 70.485 0)
+			(effects
+				(font
+					(size 1.27 1.27)
+				)
+				(hide yes)
+			)
+		)
+		(property "Value" "+24V_IN"
+			(at 87.376 65.278 0)
+			(effects
+				(font
+					(size 1.27 1.27)
+				)
+				(justify left)
+			)
+		)
+		(property "Footprint" ""
+			(at 86.36 66.675 0)
+			(effects
+				(font
+					(size 1.27 1.27)
+				)
+				(hide yes)
+			)
+		)
+		(property "Datasheet" ""
+			(at 86.36 66.675 0)
+			(effects
+				(font
+					(size 1.27 1.27)
+				)
+				(hide yes)
+			)
+		)
+		(property "Description" "Power symbol creates a global label with name \"+12V\""
+			(at 86.36 66.675 0)
+			(effects
+				(font
+					(size 1.27 1.27)
+				)
+				(hide yes)
+			)
+		)
+		(pin "1"
+		)
+		(instances
+			(project "PTN-PumpControlBoard"
+				(path "/591f46f8-eb1d-42dc-a4cb-8182eac4ef58/7f721191-bbe1-432a-ba4a-c8116ab8eb09"
+					(reference "#PWR071")
+					(unit 1)
+				)
+			)
+		)
+	)
+	(symbol
 		(lib_id "Device:R_US")
 		(at 95.885 77.47 90)
@@
 		(dnp no)
 		(fields_autoplaced yes)
-		(property "Reference" "J6"
+		(property "Reference" "3.3V_In1"
 			(at 129.54 26.67 0)
 			(effects
@@
 			(project "PTN-PumpControlBoard"
 				(path "/591f46f8-eb1d-42dc-a4cb-8182eac4ef58/7f721191-bbe1-432a-ba4a-c8116ab8eb09"
-					(reference "J6")
-					(unit 1)
-				)
+					(reference "3.3V_In1")
+					(unit 1)
+				)

Commit message: rounded corners and added rpp bypass
Parts:
- added R40: 0, Resistor_SMD:R_0603_1608Metric, symbol Device:R_US
Connections:
- net +24V: now also R40.2
- net +24V_IN: now also R40.1
Changed lines of the file:
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@@
+	)
+	(junction
+		(at 90.17 43.18)
+		(diameter 0)
+		(color 0 0 0 0)
 	)
 	(junction
@@
 	)
 	(junction
+		(at 49.53 38.1)
+		(diameter 0)
+		(color 0 0 0 0)
+	)
+	(junction
 		(at 46.355 38.1)
 		(diameter 0)
@@
 	(wire
 		(pts
+			(xy 90.17 43.18) (xy 93.345 43.18)
+		)
+		(stroke
+			(width 0)
+			(type default)
+		)
+	)
+	(wire
+		(pts
+			(xy 64.77 27.94) (xy 49.53 27.94)
+		)
+		(stroke
+			(width 0)
+			(type default)
+		)
+	)
+	(wire
+		(pts
 			(xy 31.115 73.66) (xy 38.1 73.66)
 		)
@@
 	(wire
 		(pts
+			(xy 72.39 27.94) (xy 90.17 27.94)
+		)
+		(stroke
+			(width 0)
+			(type default)
+		)
+	)
+	(wire
+		(pts
 			(xy 81.915 53.34) (xy 81.915 60.96)
 		)
@@
 	(wire
 		(pts
+			(xy 49.53 38.1) (xy 53.34 38.1)
+		)
+		(stroke
+			(width 0)
+			(type default)
+		)
+	)
+	(wire
+		(pts
 			(xy 93.345 43.18) (xy 97.79 43.18)
 		)
@@
 	(wire
 		(pts
+			(xy 90.17 27.94) (xy 90.17 43.18)
+		)
+		(stroke
+			(width 0)
+			(type default)
+		)
+	)
+	(wire
+		(pts
 			(xy 86.36 77.47) (xy 92.075 77.47)
 		)
@@
 	(wire
 		(pts
-			(xy 86.995 43.18) (xy 93.345 43.18)
+			(xy 86.995 43.18) (xy 90.17 43.18)
+		)
+		(stroke
+			(width 0)
+			(type default)
+		)
+	)
+	(wire
+		(pts
+			(xy 49.53 27.94) (xy 49.53 38.1)
 		)
 		(stroke
@@
 	(wire
 		(pts
-			(xy 46.355 38.1) (xy 53.34 38.1)
+			(xy 46.355 38.1) (xy 49.53 38.1)
 		)
 		(stroke
@@
 					(unit 1)
 				)
+			)
+		)
+	)
+	(symbol
+		(lib_id "Device:R_US")
+		(at 68.58 27.94 90)
+		(unit 1)
+		(exclude_from_sim no)
+		(in_bom yes)
+		(on_board yes)
+		(dnp yes)
+		(property "Reference" "R40"
+			(at 70.6119 25.4 90)
+			(effects
+				(font
+					(size 1.27 1.27)
+				)
+				(justify left)
+			)
+		)
+		(property "Value" "0"
+			(at 69.85 23.876 90)
+			(effects
+				(font
+					(size 1.27 1.27)
+				)
+				(justify left)
+			)
+		)
+		(property "Footprint" "Resistor_SMD:R_0603_1608Metric"
+			(at 68.834 26.924 90)
+			(effects
+				(font
+					(size 1.27 1.27)
+				)
+				(hide yes)
+			)
+		)
+		(property "Datasheet" "~"
+			(at 68.58 27.94 0)
+			(effects
+				(font
+					(size 1.27 1.27)
+				)
+				(hide yes)
+			)
+		)
+		(property "Description" "Resistor, US symbol"
+			(at 68.58 27.94 0)
+			(effects
+				(font
+					(size 1.27 1.27)
+				)
+				(hide yes)
+			)
+		)
+		(pin "1"
+		)
+		(pin "2"
+		)
+		(instances
+			(project "PTN-PumpControlBoard"
+				(path "/591f46f8-eb1d-42dc-a4cb-8182eac4ef58/7f721191-bbe1-432a-ba4a-c8116ab8eb09"
+					(reference "R40")
+					(unit 1)
+				)

Commit message: fixed cap vals + made schem pretty
Parts:
- C21: value 22n -> 22nF
- C22: value 220u -> 10uF
- R39: value 8k -> 9k
Changed lines of the file:
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@@
 			)
 		)
-		(property "Value" "22n"
+		(property "Value" "22nF"
 			(at 50.8 43.434 0)
 			(effects
@@
 			)
 		)
-		(property "Value" "220u"
+		(property "Value" "10uF"
 			(at 90.17 53.9749 0)
 			(effects
@@
 			)
 		)
-		(property "Value" "8k"
+		(property "Value" "9k"
 			(at 95.885 73.66 90)
 			(effects

Commit message: fixed rpp
Parts:
- removed Q4: PSMN8R5-40MSDX, PSMN8R5-40MSDX:BUK7M1780EX, symbol UTSVT_Power:PSMN8R5-40MSDX
- added Q3: PSMN8R5-40MSDX, BUK7M1780EX, symbol UTSVT_Power:PSMN8R5-40MSDX
- C21: value 22nF -> .1u
Connections:
- net +24V: now also Q3.1 (S)
- net +24V_IN: now also Q3.3 (D)
- net GND: now also C21.1
- net at IC3.6 (GATE): now also Q3.2 (G); no longer C21.1
Other:
- moved on the sheet: C22, C23, C24, R37, R38, R39, Z1
