File: Fans+Pump.kicad_sch (KiCad schematic)
At the start: 15 parts, among them U1 EMC2305-1-AP-TR

Commit message: lakshays bs
Parts:
- removed JP1: P_Tach, Connector_PinHeader_2.54mm:PinHeader_1x03_P2.54mm_Vertical, symbol Jumper:Jumper_3_Open
Changed lines of the file:
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@@
 	(wire
 		(pts
-			(xy 54.61 92.71) (xy 54.61 88.9)
-		)
-		(stroke
-			(width 0)
-			(type default)
-		)
-	)
-	(wire
-		(pts
 			(xy 64.77 43.18) (xy 66.04 43.18)
 		)
@@
 	(wire
 		(pts
-			(xy 53.34 92.71) (xy 54.61 92.71)
+			(xy 41.91 88.9) (xy 43.18 88.9)
 		)
 		(stroke
@@
 	(wire
 		(pts
-			(xy 45.72 85.09) (xy 48.26 85.09)
+			(xy 58.42 88.9) (xy 55.88 88.9)
 		)
 		(stroke
@@
 			"////////////////////////////////////////////////////////////////////////////"
 			"////////////////////////////////////////////////////////////////////////////"
-			"/////////////////////////////////////w=="
+			"/////////////////////////////////////wAAAAAAAAAAAAAAAAAAAAAAAAAAAAAAAAAAAAAA"
+			"AAAAAAAAAAAAAAAAAAAAAAAAAAAAAAAAAAAAAAAAAAAAAAAAAAAAAAAAAAAAAAAAAAAAAAAAAAAA"
+			"AAAAAAAAAAAAAAAAAAAAAAAAAAAAAAAAAAAAAAAAAAAAAAAAAAAAAAAAAAAAAAAAAAAAAAAAAAAA"
+			"AAAAAAAAAAAAAAAAAAAAAAAAAAAAAAAAAAAAAAAAAAAAAAAAAAAAAAAAAAAAAAAAAAAAAAAAAAAA"
+			"AAAAAAAAAAAAAAAAAAAAAAAAAAAAAAAAAAAAAAAAAAAAAAAAAAAAAAAAAAAAAAAAAAAAAAAAAAAA"
+			"AAAAAAAAAAAAAAAAAAAAAAAAAAAAAAAAAAAAAAAAAAAAAAAAAAAAAAAAAAAAAAAAAAAAAAAAAAAA"
+			"AAAAAAAAAAAAAAAAAAAAAAAAAAAAAAAAAAAAAAAAAAAAAAAAAAAAAAAAAAAAAAAAAAAAAAAAAAAA"
+			"AAAAAAAAAAAAAAAAAAAAAAAAAAAAAAAAAAAAAAAAAAAAAAAAAAAAAAAAAAAAAAAAAAAAAAAAAAAA"
+			"AAAAAAAAAAAAAAAAAAAAAAAAAAAAAAAAAAAAAAAAAAAAAAAAAAAAAAAAAAAAAAAAAAAAAAAAAAAA"
+			"AAAAAAAAAAAAAAAAAAAAAAAAAAAAAAAAAAAAAAAAAAAAAAAAAAAAAAAAAAAAAAAAAAAAAAAAAAAA"
+			"AAAAAAAAAAAAAAAAAAAAAAAAAAAAAAAAAAAAAAAAAAAAAAAAAAAAAAAAAAAAAAAAAAAAAAAAAAAA"
+			"AAAAAAAAAAAAAAAAAAAAAAAAAAAAAAAAAAAAAAAAAAAAAAAAAAAAAAAAAAAAAAAAAAAAAAAAAAAA"
+			"AAAAAAAAAAAAAAAAAAAAAAAAAAAAAAAAAAAAAAAAAAAAAAAAAAAAAAAAAAAAAAAAAAAAAAAAAAAA"
+			"AAAAAAAAAAAAAAAAAAAAAAAAAAAAAAAAAAAAAAAAAAAAAAAAAAAAAAAAAAAAAAAAAAAAAAAAAAAA"
+			"AAAAAAAAAAAAAAAAAAAAAAAAAAAAAAAAAAAAAAAAAAAAAAAAAAAAAAAAAAAAAAAAAAAAAAAAAAAA"
+			"AAAAAAAAAAAAAAAAAAAAAAAAAAAAAAAAAAAAAAAAAAAAAAAAAAAAAAAAAAAAAAAAAAAAAAAAAAAA"
+			"AAAAAAAAAAAAAAAAAAAAAAAAAAAAAAAAAAAAAAAAAAAAAAAAAAAAAAAAAAAAAAAAAAAAAAAAAAAA"
+			"AAAAAAAAAAAAAAAAAAAAAAAAAAAAAAAAAAAAAAAAAAAAAAAAAAAAAAAAAAAAAAAAAAAAAAAAAAAA"
+			"AAAAAAAAAAAAAAAAAAAAAAAAAAAAAAAAAAAAAA=="
 		)
 	)
@@
 			"OTk3KSk7CiMxNDU5OTIgPSBTVVJGQUNFX1NUWUxFX1VTQUdFKC5CT1RILiwjMTQ1OTkzKTsKIzE0"
 			"NTk5MyA9IFNVUkZBQ0VfU0lERV9TVFlMRSgnJywoIzE0NTk5NCkpOwojMTQ1OTk0ID0gU1VSRkFD"
-			"RQ=="
+			"RQEAAACwS1ZGAQAAAH1RT5khAP1R8EtWRgEAAADwS1ZGAQAAAJyCjOFrUdVH8ExWRgEAAADwTFZG"
+			"AQAAAAcVP5aEzciwME1WRgEAAAAwTVZGAQAAAAMa46BusHkVcE1WRgEAAABwTVZGAQAAAHFEkly3"
+			"gAUesE1WRgEAAACwTVZGAQAAAKd+GshlLtGf8E1WRgEAAADwTVZGAQAAAC9l/vIC53cBcE5WRgEA"
+			"AABwTlZGAQAAAAQ7M0SZZ9b0sE5WRgEAAACwTlZGAQAAAGFxGpyGQTXD8E5WRgEAAADwTlZGAQAA"
+			"AB58kKsey65FME9WRgEAAAAwT1ZGAQAAAHrz7ZYjA9aQcE9WRgEAAABwT1ZGAQAAANx+VFa+k5IR"
+			"cEZWRgEAAABwRlZGAQAAAAW8D3NRaA+X8PBbRgEAAADw8FtGAQAAAKCIQh8u5pQ/MPFbRgEAAAAw"
+			"8VtGAQAAAAYzvDFAsmAlcPFbRgEAAABw8VtGAQAAADnPTqD+z2LfsPBbRgEAAACw8FtGAQAAAEVn"
+			"9S6MYQPTAAAAAAAAAAAAAAAAAAAAAJoEvgvr73KJ8PNbRgEAAADw81tGAQAAAA4jDFbrFo8/AAAA"
+			"AAAAAAAAAAAAAAAAAKrUjZajA4SlAAAAAAAAAAAAAAAAAAAAADkGY5jqXIPj8PVbRgEAAADw9VtG"
+			"AQAAAHu7VcLu6CCSsPZbRgEAAACw9ltGAQAAAMjxcc2V3m0eAAAAAAAAAAAAAAAAAAAAAIT6W/cI"
+			"KXm/AAAAAAAAAAAAAAAAAAAAAPxYdaWFUQ3EAAAAAAAAAAAAAAAAAAAAAMTHHGmgaZraAAAAAAAA"
+			"AAAAAAAAAAAAAJf2tdnyqqw0AAAAAAAAAAAAAAAAAAAAAMAF2RF6QqnXAAAAAAAAAAAAAAAAAAAA"
+			"AKJaadI39cdCAAAAAAAAAAAAAAAAAAAAAE/Jxvk7MmPTAAAAAAAAAAAAAAAAAAAAACL/xUajG61H"
+			"AAAAAAAAAAAAAAAAAAAAAPTV07kzriPMAAAAAAAAAAAAAAAAAAAAABhW8DCp1eNGAAAAAAAAAAAA"
+			"AAAAAAAAACvsoE4A7vbqAAAAAAAAAAAAAAAAAAAAAJO8q0ShN7fIAAAAAAAAAAAAAAAAAAAAAAHE"
+			"cTAKglbMAAAAAAAAAAAAAAAAAAAAADoI9WtJJqZ5AAAAAAAAAAAAAAAAAAAAAJ+MkZDOt6NPAAAA"
+			"AAAAAAAAAAAAAAAAADfxy6to/bpbAAAAAAAAAAAAAAAAAAAAAIHhx2QsDTf6AAAAAAAAAAAAAAAA"
+			"AAAAAPJouSYJJ6O7AAAAAAAAAAAAAAAAAAAAAAV4bfA5or3yAAAAAAAAAAAAAAAAAAAAAA+dv9cx"
+			"vg=="
 		)
 	)
@@
 	(hierarchical_label "PUMP_TACH"
 		(shape input)
-		(at 53.34 92.71 180)
+		(at 41.91 88.9 180)
 		(effects
 			(font
@@
 	(hierarchical_label "PUMP_TACH_PSOM"
 		(shape output)
-		(at 45.72 85.09 180)
+		(at 58.42 88.9 0)
 		(effects
 			(font
 				(size 1.27 1.27)
 			)
-			(justify right)
+			(justify left)
 		)
 	)
@@
 					(unit 1)
 				)
-			)
-		)
-	)
-	(symbol
-		(lib_id "Jumper:Jumper_3_Open")
-		(at 54.61 85.09 0)
-		(unit 1)
-		(exclude_from_sim no)
-		(in_bom no)
-		(on_board yes)
-		(dnp no)
-		(fields_autoplaced yes)
-		(property "Reference" "JP1"
-			(at 54.61 78.74 0)
-			(effects
-				(font
-					(size 1.27 1.27)
-				)
-			)
-		)
-		(property "Value" "P_Tach"
-			(at 54.61 81.28 0)
-			(effects
-				(font
-					(size 1.27 1.27)
-				)
-			)
-		)
-		(property "Footprint" "Connector_PinHeader_2.54mm:PinHeader_1x03_P2.54mm_Vertical"
-			(at 54.61 85.09 0)
-			(effects
-				(font
-					(size 1.27 1.27)
-				)
-				(hide yes)
-			)
-		)
-		(property "Datasheet" "~"
-			(at 54.61 85.09 0)
-			(effects
-				(font
-					(size 1.27 1.27)
-				)
-				(hide yes)
-			)
-		)
-		(property "Description" "Jumper, 3-pole, both open"
-			(at 54.61 85.09 0)
-			(effects
-				(font
-					(size 1.27 1.27)
-				)
-				(hide yes)
-			)
-		)
-		(pin "1"
-		)
-		(pin "2"
-		)
-		(pin "3"
-		)
-		(instances
-			(project "PTN-PumpControlBoard"
-				(path "/591f46f8-eb1d-42dc-a4cb-8182eac4ef58/d90f7da4-ca39-48c6-8d97-b8d1e37c7dd0"
-					(reference "JP1")
-					(unit 1)
-				)
