File: Fans+Pump.kicad_sch (KiCad schematic)
At the start: 14 parts, among them U1 EMC2305-1-AP-TR

Commit message: jic
Parts:
- removed JP2: P_PWM, Connector_PinHeader_2.54mm:PinHeader_1x03_P2.54mm_Vertical, symbol Jumper:Jumper_3_Open
- added R41, R48, R49, R50: 0, Resistor_SMD:R_0603_1608Metric_Pad0.98x0.95mm_HandSolder, symbol Device:R_US
Connections:
- net PUMP_PWM: now also R50.2
- net PUMP_PWM_CHIP: now also R49.2
- net PUMP_PWM_PSOM: now also R49.1, R50.1
- net PUMP_TACH: now also R41.1, R48.1
- net PUMP_TACH_CHIP: now also R41.2
- net PUMP_TACH_PSOM: now also R48.2

Commit message: almost there
Connections:
- net PUMP_PWM: now also R49.1, R50.1; no longer R50.2
- net PUMP_PWM_PSOM: now also R50.2; no longer R49.1, R50.1
Changed lines of the file:
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@@
 	(hierarchical_label "PUMP_PWM_PSOM"
 		(shape input)
-		(at 41.91 106.68 180)
+		(at 62.23 111.76 0)
 		(effects
 			(font
 				(size 1.27 1.27)
 			)
-			(justify right)
+			(justify left)
 		)
 	)
@@
 	(hierarchical_label "PUMP_PWM"
 		(shape output)
-		(at 62.23 111.76 0)
+		(at 41.91 106.68 180)
 		(effects
 			(font
 				(size 1.27 1.27)
 			)
-			(justify left)
+			(justify right)
 		)
 	)
