File: Power.kicad_sch (KiCad schematic)
At the start: 13 parts, among them U4 LMR33630ADDA

Commit message: major schem fixes
Parts:
- added C18: 1uF, Capacitor_SMD:C_0805_2012Metric_Pad1.18x1.45mm_HandSolder, symbol Device:C
- added C19: 220nF, Capacitor_SMD:C_0805_2012Metric_Pad1.18x1.45mm_HandSolder, symbol Device:C
- added C3: 100n, Capacitor_SMD:C_0603_1608Metric_Pad1.08x0.95mm_HandSolder, symbol Device:C
- added C3: 10uF, Capacitor_SMD:C_0805_2012Metric_Pad1.18x1.45mm_HandSolder, symbol Device:C
- added IC1: LM74502HDDFR, UTSVT_Power_SP:SOT65P280X110-8N, symbol UTSVT_ICs:LM74502HDDFR
- added Q2 (x2): NVMFWS1D7N04XMT1G, Controls_Pi:NVMFWS3D0P04M8LT1G, symbol NVMFWS1D7N04XMT1G:NVMFWS1D7N04XMT1G
- added R1: 200k, Resistor_SMD:R_0603_1608Metric_Pad0.98x0.95mm_HandSolder, symbol Device:R_US
- added R13: 10k, Resistor_SMD:R_0603_1608Metric_Pad0.98x0.95mm_HandSolder, symbol Device:R_US
Connections:
- net GND: now also C18.1, C3.1, C3.2, IC1.2 (GND), R13.2
- net +24V renamed 24V_IN
- net 24V_IN: now also C18.2, C19.1, C3.2, IC1.1 (EN/UVLO), IC1.5 (VS), Q2.5, Q2.6, Q2.7, Q2.8, Q2.9, R1.1
- net 12V_BUS renamed 12V_OUT
- new net: IC1.8 (SRC), Q2.1, Q2.1, Q2.2, Q2.2, Q2.3, Q2.3
- new net: IC1.6 (GATE), Q2.4, Q2.4
- new net: IC1.7 (OV), R1.2, R13.1
- new net: C19.2, IC1.4 (VCAP)
- new net 24V_OUT: C3.1, Q2.5, Q2.6, Q2.7, Q2.8, Q2.9
Other:
- note added: "1400 fsw"
- note added: "from moco interface"
- note added: "from pi board (from vcu)"
- note added: "~26V OVP"
- note removed: "Buck Converter 24V -> 12V 1400 fsw"
- note removed: "REDO LC CALCS"
- moved on the sheet: C12, C13, C14, C15, C20, C26, C27, C28, C29, L2, R24, R25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

Commit message: schem review changes
Parts:
- added C21: 1uF, Capacitor_SMD:C_0805_2012Metric_Pad1.18x1.45mm_HandSolder, symbol Device:C
- added C22: 220nF, Capacitor_SMD:C_0805_2012Metric_Pad1.18x1.45mm_HandSolder, symbol Device:C
- added C5: 100n, Capacitor_SMD:C_0603_1608Metric_Pad1.08x0.95mm_HandSolder, symbol Device:C
- added C8: 10uF, Capacitor_SMD:C_0805_2012Metric_Pad1.18x1.45mm_HandSolder, symbol Device:C
- added IC2: LM74502HDDFR, UTSVT_Power_SP:SOT65P280X110-8N, symbol UTSVT_ICs:LM74502HDDFR
- added J2: PowerDebug, Connector_PinHeader_2.54mm:PinHeader_2x03_P2.54mm_Vertical, symbol Connector_Generic:Conn_02x03_Top_Bottom
- added Q4, Q5: NVMFWS1D7N04XMT1G, Controls_Pi:NVMFWS3D0P04M8LT1G, symbol NVMFWS1D7N04XMT1G:NVMFWS1D7N04XMT1G
- added R2: 98k, Resistor_SMD:R_0603_1608Metric_Pad0.98x0.95mm_HandSolder, symbol Device:R_US
- added R33: 10k, Resistor_SMD:R_0603_1608Metric_Pad0.98x0.95mm_HandSolder, symbol Device:R_US
- added R34: 0, Resistor_SMD:R_0603_1608Metric, symbol Device:R_US
Connections:
- net 12V_OUT: now also C8.1, J2.5 (Pin_5), Q5.5, Q5.6, Q5.7, Q5.8, Q5.9, R34.2; no longer C20.1, C26.1, C27.1, C28.1, C29.1, L2.2, R24.1
- net 24V_IN: now also J2.1 (Pin_1); no longer C12.1, C13.1, U4.2 (VIN), U4.3 (EN)
- net 24V_OUT: now also C12.1, C13.1, U4.2 (VIN), U4.3 (EN), J2.4 (Pin_4)
- net GND: now also C21.1, C5.1, C8.2, IC2.2 (GND), J2.3 (Pin_3), J2.6 (Pin_6), R33.2
- new net: IC2.8 (SRC), Q4.1, Q4.2, Q4.3, Q5.1, Q5.2, Q5.3
- new net: IC2.6 (GATE), Q4.4, Q5.4
- new net: C22.2, IC2.4 (VCAP)
- new net: IC2.7 (OV), R2.2, R33.1
- new net 12V_BUCKED: C20.1, C21.2, C22.1, C26.1, C27.1, C28.1, C29.1, C5.2, IC2.1 (EN/UVLO), IC2.5 (VS), J2.2 (Pin_2), L2.2, Q4.5, Q4.6, Q4.7, Q4.8, Q4.9, R2.1, R24.1, R34.1
Other:
- note added: "from datasheet"
- note added: "~13.5V OVP (bc pump)"
- moved on the sheet: C12, C13, C14, C15, C18, C19, C20, C26, C27, C28, C29, C3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

Commit message: finalized schem
Parts:
- renumbered C15 to C10, C12 to C11, C13 to C12, C26 to C13, C27 to C14, C28 to C15, C29 to C16, C20 to C17, C14 to C18, C5 to C19, C8 to C20, C3 to C6, C3 to C7, C18 to C8, C19 to C9, J2 to J5, L2 to L1, Q2 to Q3, Q2 to Q4, Q4 to Q5, Q5 to Q6, R1 to R32, R13 to R33, R24 to R34, R25 to R35, R34 to R36, R2 to R37, R33 to R38, U4 to U3

Commit message: almost all footprints
Parts:
- C11, C13, C14, C15, C16, C20, C21, C22, C7, C8, C9: footprint Capacitor_SMD:C_0805_2012Metric_Pad1.18x1.45mm_HandSolder -> Capacitor_SMD:C_0603_1608Metric_Pad1.08x0.95mm_HandSolder
- IC1, IC2: footprint UTSVT_Power_SP:SOT65P280X110-8N -> UTSVT_Power:SOT65P280X110-8N
- Q3, Q4, Q5, Q6: footprint Controls_Pi:NVMFWS3D0P04M8LT1G -> PumpLib:NVMFWS3D0P04M8LT1G
- R36: footprint Resistor_SMD:R_0603_1608Metric -> Resistor_SMD:R_0603_1608Metric_Pad0.98x0.95mm_HandSolder

Commit message: subcircuit layout
Parts:
- L1: footprint easyeda2kicad:IND-SMD_L5.0-W5.0 -> PumpLib:IND-SMD_L5.0-W5.0
Changed lines of the file:
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@@
 			"AAAAAAAAAA0SAAAAAAAAJiIAAAAAAACwQAAAAAAAAFMcAAAAAAAAPS0AAAAAAACADQAAAAAAAAAA"
 			"AAAAAAAAdw4AAAAAAACROgAAAAAAAAAAAAAAAAAAXzQAAAAAAAAAAAAAAAAAAAAAAAAAAAAAYiEA"
-			"AAAAAAAAAAAAAAAAAGA6AA=="
+			"AAAAAAAAAAAAAAAAAGA6AAAAAAAAAAAAAAAAAAAAAAAAAAAAAAAAAAAAAAAAAAAAAAAAAAAAAAAA"
+			"AAAAAAAAAAAAAAAAAAAAAAAAAAAAAAAAAAAAAAAAAAAAAAAAAAAAAAAAAAAAAAAAAAAAAAAAAAAA"
+			"AAAAAAAAAAAAAAAAAAAAAAAAAAAAAAAAAAAAAAAAAAAAAAAAAAAAAAAAAAAAAAAAAAAAAAAAAAAA"
+			"AAAAAAAAAAAAAAAAAAAAAAAAAAAAAAAAAAAAAAAAAAAAAAAAAAAAAAAAAAAAAAAAAAAAAAAAAAAA"
+			"AAAAAAAAAAAAAAAAAAAAAAAAAAAAAAAAAAAAAAAAAAAAAAAAAAAAAAAAAAAAAAAAAAAAAAAAAAAA"
+			"AAAAAAAAAAAAAAAAAAAAAAAAAAAAAAAAAAAAAAAAAAAAAAAAAAAAAAAAAAAAAAAAAAAAAAAAAAAA"
+			"AAAAAAAAAAAAAAAAAAAAAAAAAAAAAAAAAAAAAAAAAAAAAAAAAAAAAAAAAAAAAAAAAAAAAAAAAAAA"
+			"AAAAAAAAAAAAAAAAAAAAAAAAAAAAAAAAAAAAAAAAAAAAAAAAAAAAAAAAAAAAAAAAAAAAAAAAAAAA"
+			"AAAAAAAAAAAAAAAAAAAAAAAAAAAAAAAAAAAAAAAAAAAAAAAAAAAAAAAAAAAAAAAAAAAAAAAAAAAA"
+			"AAAAAAAAAAAAAAAAAAAAAAAAAAAAAAAAAAAAAAAAAAAAAAAAAAAAAAAAAAAAAAAAAAAAAAAAAAAA"
+			"AAAAAAAAAAAAAAAAAAAAAAAAAAAAAAAAAAAAAAAAAAAAAAAAAAAAAAAAAAAAAAAAAAAAAAAAAAAA"
+			"AAAAAAAAAAAAAAAAAAAAAAAAAAAAAAAAAAAAAAAAAAAAAAAAAAAAAAAAAAAAAAAAAAAB/////wAA"
+			"AAAAAAAAAAAAAAAAAAAAAAAAAAAAAAAAAAAAAAAAAAAAAAAAAAAAAAAAAAAAAAAAAAAAAAAAAAAA"
+			"AAAAAAAAAAAAAAAAAAAAAAAAAAAAAAAAAAAAAAAAAAAAAAAAAAAAAAAAAAAAAAAAAAAAAAAAAAAA"
+			"AAAAAAAAAAAAAAAAAAAAAAAAAAAAAAAAAAAAAAAAAAAAAAAAAAAAAAAAAAAAAAAAAAAAAAAAAAAA"
+			"AAAAAAAAAAAAAAAAAAAAAAAAAAAAAAAAAAAAAAAAAAAAAAAAAAAAAAAAAAAAAAAAAAAAAAAAAAAA"
+			"AAAAAAAAAAAAAAAAAAAAAAAAAAAAAAAAAAAAAAAAAAAAAAAAAAAAAAAAAAAAAAAAAAAAAAAAAAAA"
+			"AAAAAAAAAAAAAAAAAAAAAAAAAAAAAAAAAAAAAAAAAAAAAAAAAAAAAAAAAAAAAAAAAAAAAAAAAAAA"
+			"AAAAAAAAAAAAAAAAAAAAAAAAAAAAAAAAAAAAAAAAAAAAAAAAAAAAAAAAAAAAAAAAAAAAAAAAAAAA"
+			"AAAAAAAAAAAAAAAAAAAAAAAAAAAAAAAAAAAAAAAAAAAAAAAAAAAAAAAAAAAAAAAAAAAAAAAAAAAA"
+			"AAAAAAAAAAAAAAAAAAAAAAAAAAAAAAAAAAAAAAAAAAAAAAAAAAAAAAAAAAAAAAAAAAAAAAAAAAAA"
+			"AAAAAAAAAAAAAAAAAAAAAAAAAAAAAAAAAAAAAAAAAAAAAAAAAAAAAAAAAAAAAAAAAAAAAAAAAAAA"
+			"AAAAAAAAAAAAAAAAAAAAAAAAAAAAAAAAAAAAAAAAAAAAAAAAAAAAAAAAAAAAAAAAAAAAAAAAAAAA"
+			"AAAAAAAAAAAAAAAAAAAAAAAAAAAAAAAAAAAAAAAAAAAAAAAAAAAAAAAAAAAAAAAAAAAAAAAAAAAA"
+			"AAAAAAAAAAAAAAAAAAAAAAAAAAAAAAAAAAAAAAAAAAAAAAAAAAAAAAAAAAAAAAAAAAAAAAAAAAAA"
+			"AAAAAAAAAAAAAAAAAAAAAAAAAAAAAAAAAAAAAAAAAAAAAAAAAAAAAAAAAAAAAAAAAAAAAAAAAAAA"
+			"AAAAAAAAAAAAAAAAAAAAAAAAAAAAAAAAAAAAAAAAAAAAAAAAAAAAAAAAAAAAAAAAAAAAAAAAAAAA"
+			"AAAAAAAAAAAAAAAAAAAAAAAAAAAAAAAAAAAAAAAAAAAAAAAAAAAAAAAAAAAAAAAAAAAAAAAAAAAA"
+			"AAAAAAAAAAAAAAAAAAAAAAAAAAAAAAAAAAAAAAAAAAAAAAAAAAAAAAAAAAAAAAAAAAAAAAAAAAAA"
+			"AAAAAAAAAAAAAAAAAAAAAAAAAAAAAAAAAAAAAAAAAAAAAAAAAAAAAAAAAAAAAAAAAAAAAAAAAAAA"
+			"AAAAAAAAAAAAAAAAAAAAAAAAAAAAAAAAAAAAAAAAAAAAAAAAAAAAAAAAAAAAAAAAAAAAAAAAAAAA"
+			"AAAAAAAAAAAAAAAAAAAAAAAAAAAAAAAAAAAAAAAAAAAAAAAAAAAAAAAAAAAAAAAAAAAAAAAAAAAA"
+			"AAAAAAAAAAAAAAAAAAAAAAAAAAAAAAAAAAAAAAAAAAAAAAAAAAAAAAAAAAAAAAAAAAAAAAAAAAAA"
+			"AAAAAAAAAAAAAAAAAAAAAAAAAAAAAAAAAAAAAAAAAAAAAAAAAAAAAAAAAAAAAAAAAAAAAAAAAAAA"
+			"AAAAAAAAAAAAAAAAAAAAAAAAAAAAAAAAAAAAAAAAAAAAAAAAAAAAAAAAAAAAAAAAAAAAAAAAAAAA"
+			"AAAAAAAAAAAAAAAAAAAAAAAAAAAAAAAAAAAAAAAAAAAAAAAAAAAAAAAAAAAAAAAAAAAAAAAAAAAA"
+			"AAAAAAAAAAAAAAAAAAAAAPr/+vr6//r6+v/6+vr/+vr6/7q6uv+6uroAAAAAAAAAAAAAAAAAAAAA"
+			"/7q6uv+6urr/4+Pj/+Pj4//j4+P/4+Pj/7q6uv+6urr/+vr6//r6+v/6+vr/+vr6//r6+v/6+vr/"
+			"+vr6//r6+v/6+vr/+vr6/7q6uv+6urr/+vr6//r6+v/6+vr/+vr6//r6+v/6+vr/+vr6//r6+v/6"
+			"+vr/+vr6/7q6uv+6urr/+vr6//r6+v/6+vr/+vr6//r6+v/6+vr/+vr6//r6+v/6+vr/+vr6/7q6"
+			"uv+6uroAAAAAAAAAAAAAAAAAAAAA/7q6uv+6urr/4+Pj/+Pj4//j4+P/4+Pj/7q6uv+6urr/+vr6"
+			"//r6+v/6+vr/+vr6//r6+v/6+vr/+vr6//r6+v/6+vr/+vr6/7q6uv+6urr/+vr6//r6+v/6+vr/"
+			"+vr6//r6+v/6+vr/+vr6//r6+v/6+vr/+vr6/7q6uv+6urr/+vr6//r6+v/6+vr/+vr6//r6+v/6"
+			"+vr/+vr6//r6+v/6+vr/+vr6/7q6uv+6uroAAAAAAAAAAAAAAAAAAAAA/7q6uv+6urr/4+Pj/+Pj"
+			"4//j4+P/4+Pj/7q6uv+6urr/+vr6//r6+v/6+vr/+vr6//r6+v/6+vr/+vr6//r6+v/6+vr/+vr6"
+			"/7q6uv+6urr/+vr6//r6+v/6+vr/+vr6//r6+v/6+vr/+vr6//r6+v/6+vr/+vr6/7q6uv+6urr/"
+			"+vr6//r6+v/6+vr/+vr6//r6+v/6+vr/+vr6//r6+v/6+vr/+vr6/7q6uv+6uroAAAAAAAAAAAAA"
+			"AAAAAAAA/7q6uv+6urr/4+Pj/+Pj4//j4+P/4+Pj/7q6uv+6urr/+vr6//r6+v/6+vr/+vr6//r6"
+			"+v/6+vr/+vr6//r6+v/6+vr/+vr6/7q6uv+6urr/+vr6//r6+v/6+vr/+vr6//r6+v/6+vr/+vr6"
+			"//r6+v/6+vr/+vr6/7q6uv+6urr/+vr6//r6+v/6+vr/+vr6//r6+v/6+vr/+vr6//r6+v/6+vr/"
+			"+vr6/7q6uv+6uroAAAAAAAAAAAAAAAAAAAAA/7q6uv+6urr/4+Pj/+Pj4//j4+P/4+Pj/7q6uv+6"
+			"urr/+vr6//r6+v/6+vr/+vr6//r6+v/6+vr/+vr6//r6+v/6+vr/+vr6/7q6uv+6urr/+vr6//r6"
+			"+v/6+vr/+vr6//r6+v/6+vr/+vr6//r6+v/6+vr/+vr6/7q6uv+6urr/+vr6//r6+v/6+vr/+vr6"
+			"//r6+v/6+vr/+vr6//r6+v/6+vr/+vr6/7q6uv+6uroAAAAAAAAAAAAAAAAAAAAA/7q6uv+6urr/"
+			"4+Pj/+Pj4//j4+P/4+Pj/w=="
 		)
 	)
@@
 			"d62GXo18T+R7QmdDZ0PjWx/f+tSKPrViNB6d47ETX3nWV6yygFUWfAr9KTQ7dWCrEXJgQA50qeVc"
 			"arnoMXQ+Rl+P0tej6D+D/jPwqRx8KodgJHpGQu+B3oM82caz2YaY94l5p8g57Zz/4n+8q3N/6Ve5"
-			"9DWuH32Ba6T9Blfm6smP/RaXvc5/kav0Cw=="
+			"9DWuH32Ba6T9Blfm6smP/RaXvc5/kav0CwAAAAAAAAAAAAAAAAAAAAAAAAAAAAAAAAAAAAAAAAAA"
+			"AAAAAAAAAAAAAAAAAAAAAAAAAAAAAAAAAAAAAAAAAAAAAAAAAAAAAAAAAAAAAAAAAAAAAAAAAAAA"
+			"AAAAAAAAAAAAAAAAAAAAAAAAAAAAAAAAAAAAAAAAAAAAAAAAAAAAAAAAAAAAAAAAAAAAAAAAAAAA"
+			"AAAAAAAAAAAAAAAAAAAAAAAAAAAAAAAAAAAAAAAAAAAAAAAAAAAAAAAAAAAAAAAAAAAAAAAAAAAA"
+			"AAAAAAAAAAAAAAAAAAAAAAAAAAAAAAAAAAAAAAAAAAAAAAAAAAAAAAAAAAAAAAAAAAAAAAAAAAAA"
+			"AAAAAAAAAAAAAAAAAAAAAAAAAAAAAAAAAAAAAAAAAAAAAAAAAAAAAAAAAAAAAAAAAAAAAAAAAAAA"
+			"AAAAAAAAAAAAAAAAAAAAAAAAAAAAAAAAAAAAAAAAAAAAAAAAAAAAAAAAAAAAAAAAAAAAAAAAAAAA"
+			"AAAAAAAAAAAAAAAAAAAAAAAAAAAAAAAAAAAAAAAAAAAAAAAAAAAAAAAAAAAAAAAAAAAAAAAAAAAA"
+			"AAAAAAAAAAAAAAAAAAAAAAAAAAAAAAAAAAAAAAAAAAAAAAAAAAAAAAAAAAAAAAAAAAAAAAAAAAAA"
+			"AAAAAAAAAAAAAAAAAAAAAAAAAAAAAAAAAAAAAAAAAAAAAAAAAAAAAAAAAAAAAAAAAAAAAAAAAAAA"
+			"AAAAAAAAAAAAAAAAAAAAAAAAAAAAAAAAAAAAAAAAAAAAAAAAAAAAAAAAAAAAAAAAAAAAAAAAAAAA"
+			"AAAAAAAAAAAAAAAAAAAAAAAAAAAAAAAAAAAAAAAAAAAAAAAAAAAAAAAAAAAAAAAAAAAAAAAAAAAA"
+			"AAAAAAAAAAAAAAAAAAAAAAAAAAAAAAAAAAAAAAAAAAAAAAAAAAAAAAAAAAAAAAAAAAAAAAAAAAAA"
+			"AAAAAAAAAAAAAAAAAAAAAAAAAAAAAAAAAAAAAAAAAAAAAAAAAAAAAAAAAAAAAAAAAAAAAAAAAAAA"
+			"AAAAAAAAAAAAAAAAAAAAAAAAAAAAAAAAAAAAAAAAAAAAAAAAAAAAAAAAAAAAAAAAAAAAAAAAAAAA"
+			"AAAAAAAAAAAAAAAAAAAAAAAAAAAAAAAAAAAAAAAAAAAAAAAAAAAAAAAAAAAAAAAAAAAAAAAAAAAA"
+			"AAAAAAAAAAAAAAAAAAAAAAAAAAAAAAAAAAAAAAAAAAAAAAAAAAAAAAAAAAAAAAAAAAAAAAAAAAAA"
+			"AAAAAAAAAAAAAAAAAAAAAAAAAAAAAAAAAAAAAAAAAAAAAAAAAAAAAAAAAAAAAAAAAAAAAAAAAAAA"
+			"AAAAAAAAAAAAAAAAAAAAAAAAAAAAAAAAAFNmck9aU2lUNUhCTUpVa1NTU3hSRUVwU2U4WkU4ME1P"
+			"U2ZSRGZ3blBoSHVpcG9pRWt1UEpHRnUwUVVaUXpFaE5UY0ZyK1FoQi8vLy8vMzAveExjVVBKazJL"
+			"bC9JaC8vK3VLNEhpLzd3OFBEdzMrUFM4ajB6WWV5MnRUMWljWkRGZENLaFVFZ1NKU1JrTWdseEVo"
+			"Tk43cEZRU0VoSWpCVzdRU1NFSkVreVBDUkRKRWx5aENFSlpWNHlTTkxqZE9TNDN6RVJYREFZRkVW"
+			"UkZNWEFRTjFCbmxnc0ZpSVhiT0EzM2NMRXJpUVdVeXcyamJaRmJCUFdNSWFGaFVYNDhqMGVianNp"
+			"RkNFMVJRdXBvWlpLU0Znb2tzRUpETjlVSGdwaEI0ZDVQMjNaclZYRklxS0VCTGtVUWR6WEdidVF5"
+			"V1pOWVp1b3hCY1JJV3hWZll3VUZQNFFJVUtFQ0NIZU5LUWhRZ2lGSVZRRmM3OTh5L1BRTVdoOCth"
+			"djZ2L0wvNTgvei9NWC91aTdIcGZEYlp5eU1KWTFhRnEzUnRDMVo4VEFqZXM4T2Z1Vy9Pd0VGR0J3"
+			"TUVHQUEvMTlTRVArcC82WmQyNlp0enVHd0hHelB6RGdVYkdabTZKa0pNMU8zN2JSdHBXeWpiVnZo"
+			"eFdJWnFRaEZSRUpFUkJJa3lHbXlKT21Da2VSSWt2UTk2emlPazNIY0Z1TzRjWlFtR0g4d0ZyR0lV"
+			"TWdVaEJBaHJxQnB1aEpLUkUzaWhrSVNmZG9lMndYKy8zOEl2TzhwOFAveWYrWjVudWRRb1BtKzJM"
+			"NXYvNDk0V1ArcmkzQjJoZjdQYjNrYUhzN3cveUU4aFAvK3ZPL2wvQjZQNitHM2JZOXJNVTNQWVRr"
+			"NCtKNlptWm54Wjl5MnJibTJyZmovL2Z1WDIxTWg2VXVNL2dQL2Yya2hPZzF0TktUTFdNUndXelhw"
+			"c0J6c1lVZEdLbTJGdUtoakpMVFdyUDBOa3hhSVVVQXdGay9rSUlZZ3BKQmowQWNUUUlGTGxXb3hu"
+			"dVFFaEJoQ0NER0dqSWpJU0NBeU1wSW02Y3l5K0hrb09HdDdrMVA5bGdOaGluQ1orK25ONjl3ZXp5"
+			"VGNyL1dWMCt6OG0wdE5uQkREKzNDT055UDU0M3M4VTJReENucENVekliem1yOTRxM1BwUENHaE5Y"
+			"K3EyNEtWS293cEM5V1J0MHNsREdjcStkcTBPRzQrVGRSMjJ1MzFmazNpNnA0SUliL3lVSEszMFRl"
+			"bEt5UEJLV1FsVTdEcGJSKzhhdG5VSGpROGlCdUZKL2F2L25YN3YxRFRDSEVRTkFKWlZJemNGeHRY"
+			"endHNTk5TWFtS01BUDhUcDVXL2VieFRzeEIvM31lOoESpP0gdx7bf7As+9ofrhe/7G637KhSJZt6"
+			"7H0hnb9XT6pKVSy58izO/5OeWTKccrfHzk9Qcv2p2494VYeg+tDnsz4R5z08RbhOeuxb71LzvVpI"
+			"M/47e5aUg0TUXYtWrenRJ5+mVnu30aNcYb8+FIT98378gW667ipZJs43GfzwENr/gK4uG1IR6PYj"
+			"r6DbAMTD5IkT6MP3p5MX3rr99cXNTmed24d697mAatWurUe7wnodgrbfVWDAgnTbj5unJk8cTyNf"
+			"elESbsr8mjVr0j+uGUhnnt3banMVh+fiP36nq/peIkVjJrxNeC+8nG4/dLgNvJBKn8zUBqkSKCtX"
+			"rqP9DjpTfAcXUNs2LWjUiAfo+P873DoU+b6HhtODj4yQlRt0/SU09PFbpB/6R/71QlqwcLFMt3jh"
+			"DCMAOoGi+lCq9g99ZgzdeudQatmiKa1Y9JHRBj1y1mdz6OSeA6R4ibC/jai/n9Pt99NjOSPACDAC"
+			"jIAYJ4jByR4GghFgBKKPgBqwBTH5xeqMmwdeI1Zu/OoApkOnfeip54fTjddeRUsXxwiGrKws2i0+"
+			"RvaIFQZwuFb3hVdHU6d993Ok1QP6oFnZnyoBVC2nAdWp3lgvzjPcSqyeua19bJI/6Je7LR18LG7e"
+			"scy4kkYnUIKyH0Y0qtORnunysLSn3//6U1HxNsu2k1r3ob4te1vh3OKttKloC7Wq3oxqVK0u5ZuF"
+			"/q0/3047C3MtPd2j2494VYcg+tBrI1+hsf9+1Sr2xZGjaZ/99qe5c76hu24eJLCNffVkZ2dTw0aN"
+			"JUlUXFws9UFCPPzEUNpPrBoyOb8+FIT9dgIINsDO8y68hC7p24+qiauvg3C6/cgzyDYA+XODeFex"
+			"mkl3uL67Rs1a8iBfnciFbtv2HWjIU8/IQ331tPawXocg7beXky5/uu1/a/ybNOL5Yb7mH37k0ZJc"
+			"rFmrlkOHCSCiIN5jB6hpCuh9CMWo9yBVAmXyu5/QeRfdLL9X5333tlzdY6/GQYefQ/MXLKKGDerR"
+			"8j9mypU2Kv6DmV/Q6WddJ4PrVnxmPBhaJ1CCsv+JoaPpjnuGUYf2ren3+dOVaSV6/jTvN7m6Ccq/"
+			"/zydOnTwJkERr9sPGTtGgBFgBBgBbwSYAPLGhaWMQOQQUAO2IAbNtw26nr7/7luJAX6pbt6iJa1Y"
+			"tlTe+NKgYUN5HTAm7Tfcejsddexfabe4Cebzzz6lF58ZStu2bhUT/c70wiv/Nm4l0QfNyv5UCaCj"
+			"mvekgW2dB2SWpTEH/DiQ8gvW+ybVCZSg7EeBfgRQnZot6YUDn5Irf5bEV/pstFb6VKH9m/wfXdfm"
+			"MqqfXYfm5y2iIfMTpJZeEd1+xKs6pNqH1g=="
 		)
 	)
@@
 			)
 		)
-		(property "Footprint" "easyeda2kicad:IND-SMD_L5.0-W5.0"
+		(property "Footprint" "PumpLib:IND-SMD_L5.0-W5.0"
 			(at 224.79 69.85 0)
 			(effects

Commit message: main circuitry done
Parts:
- renumbered J5 to J6
Changed lines of the file:
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@@
 		(dnp no)
 		(fields_autoplaced yes)
-		(property "Reference" "J5"
+		(property "Reference" "J6"
 			(at 171.45 118.11 0)
 			(effects
@@
 			(project ""
 				(path "/591f46f8-eb1d-42dc-a4cb-8182eac4ef58/7f721191-bbe1-432a-ba4a-c8116ab8eb09"
-					(reference "J5")
+					(reference "J6")
 					(unit 1)
 				)

Commit message: lakshays bs
Parts:
- L1: P/N (none) -> CKCS5040
Other:
- moved on the sheet: C19, C20, C21, C22, C6, C7, C8, C9, IC1, IC2, Q3, Q4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

Commit message: almost there
Parts:
- removed J6: PowerDebug, Connector_PinHeader_2.54mm:PinHeader_2x03_P2.54mm_Vertical, symbol Connector_Generic:Conn_02x03_Top_Bottom
- added TP1: 24V_IN, TestPoint:TestPoint_Pad_2.0x2.0mm, symbol Connector:TestPoint
- added TP2: 24V, TestPoint:TestPoint_Pad_2.0x2.0mm, symbol Connector:TestPoint
- added TP3: 12V_IN, TestPoint:TestPoint_Pad_2.0x2.0mm, symbol Connector:TestPoint
- added TP4: 12V_OUT, TestPoint:TestPoint_Pad_2.0x2.0mm, symbol Connector:TestPoint
- added TP5: GND, TestPoint:TestPoint_Pad_2.0x2.0mm, symbol Connector:TestPoint
Connections:
- net 12V_BUCKED: now also TP3.1
- net 12V_OUT: now also TP4.1
- net 24V_IN: now also TP1.1
- net 24V_OUT: now also TP2.1
- net GND: now also TP5.1
