File: hardware/PTN-PumpControlBoard.kicad_sch (KiCad schematic)
At the start: 33 parts, among them J1 PWR_CAN, J2 Pump_Temp, J3 Flow_Fan, J4 53307-2471, J5 SFH11-PBPC-D05-ST-BK

Commit message: better organization:
Other:
- note added: "PA0"
- note added: "PA12"
- note added: "PA6"
- note added: "PB0"
- note added: "PB10"
- note added: "PB14"
