File: hardware/PTN-PumpControlBoard.kicad_pcb (KiCad board)
At the start: 2 copper layers, 53.1 x 81.9 mm, 115 parts, among them IC1 LM74502HDDFR, IC2 LM74502HDDFR, J1 PWR_CAN, J2 Pump_Temp, J3 Flow_Fan, J4 53307-2471, J5 SFH11-PBPC-D05-ST-BK, Q1 IRLML0030TRPBF, Q2 IRLML0030TRPBF, Q3 NVMFWS1D7N04XMT1G, Q4 NVMFWS1D7N04XMT1G, Q5 NVMFWS1D7N04XMT1G, Q6 NVMFWS1D7N04XMT1G, U1 EMC2305-1-AP-TR, U2 TLV9002QDRQ1, U3 LMR33630ADDA

Commit message: Rev c (#4)
* making sure submodules are right

* deleting stuff

* more deletes

* last delete (?)

* hopefully fixed?

* gerbers

* fixed 3d models

* fix .gitignore

Add various entries to .gitignore for build files, Python environments, Mac specific files, Vim swap files, Nix lock files, documentation toolset, and VSCode settings.

* .gitmodules fix

* hopefully firmware setup works?
Parts:
- J3: footprint Connector_Molex:Molex_Nano-Fit_105310-xx12_2x06_P2.50mm_Vertical -> PumpLib:CONN_SD-105310-100_14_MOL
- moved D23 2.38 mm to (159.4, 123.7)
- moved TP4 2.38 mm to (155.9, 122.7)
- moved R47 2.38 mm to (159.4, 122.1)
- moved D22 2.06 mm to (148.7, 123.6)
- moved R46 2.06 mm to (148.7, 122.0)
- moved TP2 1.86 mm to (145.3, 122.7)
- turned J3 to -90 degrees
Connections:
- J3 pad 11: /FAN1_PWM -> GND
- J3 pad 12: /FAN2_PWM -> /FAN1_PWM
- J3 pad 7: GND -> +24V
- J3 pad 8: /FLOW2_SIG -> GND
- J3 pad 9: GND -> /FLOW2_SIG
Routing:
- net +24V: track 110.1 -> 116.2 mm
- net GND: track 74.8 -> 70.8 mm, vias 151 -> 148
- net /TEMP_IN1: track 39.2 -> 35.4 mm, vias 3 -> 4
- net +3.3V: track 91.5 -> 89.5 mm
- net /PUMP_TACH: track 111.5 -> 113.1 mm
Other:
- board text added: "AGND"
- board text added: "FAN2+ TACH2 TACH1 FAN1+ FLOW2+ FLOW1 FLOW1+"
- board text added: "FAN2- PWM2 PWM1 FAN1- FLOW2- FLOW2 FLOW1-"
- board text added: "TEMP1"
- board text added: "TEMP2"
- board text removed: "PWM2 PWM1 FANS- FLOW2- FLOW2 FLOW2+"
- board text removed: "TACH2 TACH1 FANS+ FLOW2+ FLOW1 FLOW1+"
